File: hardware/5v-solar-regulator.kicad_pcb (KiCad board)
At the start: 2 copper layers, 82.4 x 48.6 mm, 37 parts, among them P1 CONN_01X20, P2 CONN_01X20, P3 CONN_01X03, P4 CONN_01X04, P5 USB_A_2, Q2 Q_NMOS_GSD, Q3 Q_PMOS_GSD, U1 ESP-WROOM-32, U10 touchpad, U2 ZXCT1107, U3 LM2576, U5 SPX3819, U6 OPA344

Commit message: update
Parts:
- removed P1, P2: CONN_01X20, Pin_Headers:Pin_Header_Straight_1x20_Pitch2.54mm
- added J1: CONN_02X16, Pin_Headers:Pin_Header_Straight_2x16_Pitch2.54mm, F.Cu at (123.0, 76.8)
- C3, C4, R11, U5: moved to B.Cu
- R17, R18, R19, U6: moved to F.Cu
- moved P3 42.8 mm to (140.3, 116.2)
- moved U10 33.1 mm to (133.8, 86.3), turned to 180 degrees
- moved D3 14.9 mm to (166.6, 115.4), turned to 0 degrees
- moved U5 14.2 mm to (159.0, 102.7), turned to 180 degrees
- moved C4 14.1 mm to (159.2, 98.8), turned to 0 degrees
- moved R25 14.1 mm to (144.0, 109.2)
- moved C3 12.8 mm to (165.3, 102.6)
- moved R11 11.9 mm to (163.0, 102.6)
- moved U6 11.1 mm to (162.8, 115.4)
- moved C2 10.2 mm to (159.0, 105.7), turned to 90 degrees
- moved R18 8.38 mm to (158.4, 111.0), turned to 180 degrees
- moved P4 7.01 mm to (145.3, 112.4), turned to 270 degrees
- moved R17 4.79 mm to (162.7, 112.0), turned to 180 degrees
- moved R19 4.50 mm to (162.7, 110.0), turned to 180 degrees
- moved R5 4.08 mm to (143.2, 79.0)
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Connections:
- C1 pad 1: VIN -> Vin
- C2 pad 1: 5V -> 5v
- L1 pad 2: 5V -> 5v
- P4 pad 1: 5V -> 5v
- R2 pad 1: 3V3 -> 3v3
- R25 pad 2: 5V -> 5v
- R5 pad 2: VIN -> Vin
- U1 pad 2: 3V3 -> 3v3
- U2 pad 2: VIN -> Vin
- U3 pad 1: VIN -> Vin
- U3 pad 4: 5V -> 5v
