File: hardware/power.sch (KiCad schematic (older format))
At the start: 14 parts, among them U2 ZXCT1107, U3 LM2576, U5 SPX3819

Commit message: update
Parts:
- added J?: CONN_01X02, symbol CONN_01X02
Connections:
- net BATTERY: now also J?.1 (P1)
- net GND: now also J?.2 (P2)
Other:
- moved on the sheet: C1, C2, C3, C4, D1, R11, R3, R4, R5, R6, U2, U3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

Commit message: update
Parts:
- J2: renamed from J?; footprint (none) -> footprints:battery_input
- R6: Part Number RC0603JR-0710KL -> RC0402FR-074K99L
- U3: Part Number ZXCT1107SA-7 -> LM2576SX-5.0/NOPB
Connections:
- net 5v is gone; now on net 5V: C2.1, L1.2, U3.4 (Feedback)
- net VIN is gone; now on net Vin: R3.1
- net 3V3 renamed 3v3
Changed lines of the file:
@@
 LIBS:contrib
 LIBS:valves
-LIBS:5v-solar-regulator-cache
-EELAYER 26 0
+LIBS:open-automation
+LIBS:5v-smart-solar-regulator-cache
+EELAYER 25 0
 EELAYER END
 $Descr A4 11693 8268
@@
 $EndComp
 $Comp
-L GND #PWR18
+L GND #PWR012
 U 1 1 5909DD65
 P 7450 3050
-F 0 "#PWR18" H 7450 2800 50  0001 C CNN
+F 0 "#PWR012" H 7450 2800 50  0001 C CNN
 F 1 "GND" H 7450 2900 50  0000 C CNN
 F 2 "" H 7450 3050 50  0000 C CNN
@@
 $EndComp
 $Comp
-L GND #PWR17
+L GND #PWR013
 U 1 1 5909DD66
 P 6900 3100
-F 0 "#PWR17" H 6900 2850 50  0001 C CNN
+F 0 "#PWR013" H 6900 2850 50  0001 C CNN
 F 1 "GND" H 6900 2950 50  0000 C CNN
 F 2 "" H 6900 3100 50  0000 C CNN
@@
 $EndComp
 $Comp
-L GND #PWR19
+L GND #PWR014
 U 1 1 5909DD67
 P 8950 2850
-F 0 "#PWR19" H 8950 2600 50  0001 C CNN
+F 0 "#PWR014" H 8950 2600 50  0001 C CNN
 F 1 "GND" H 8950 2700 50  0000 C CNN
 F 2 "" H 8950 2850 50  0000 C CNN
@@
 5V
 Text GLabel 8950 2100 1    60   Input ~ 0
-3V3
+3v3
 $Comp
 L LM2576 U3
@@
 F 1 "LM2576" H 5300 4850 60  0000 C CNN
 F 2 "footprints:Regulator-LM2576" H 5650 5000 60  0001 C CNN
-F 3 "http://www.digikey.com/scripts/DkSearch/dksus.dll?Detail&itemSeq=233265175&uq=636356458892291311" H 5650 5000 60  0001 C CNN
-F 4 "ZXCT1107SA-7" H 5250 5050 60  0001 C CNN "Part Number"
+F 3 "http://www.digikey.com/scripts/DkSearch/dksus.dll?Detail&itemSeq=233232230&uq=636364877859867737" H 5650 5000 60  0001 C CNN
+F 4 "LM2576SX-5.0/NOPB" H 5250 5050 60  0001 C CNN "Part Number"
 	1    5250 5050
 	1    0    0    -1
@@
 Vin
 Text GLabel 6300 4800 1    60   Input ~ 0
-5v
+5V
 $Comp
 L CP C1
@@
 $EndComp
 $Comp
-L GND #PWR12
+L GND #PWR015
 U 1 1 5966A247
 P 2400 3050
-F 0 "#PWR12" H 2400 2800 50  0001 C CNN
+F 0 "#PWR015" H 2400 2800 50  0001 C CNN
 F 1 "GND" H 2400 2900 50  0000 C CNN
 F 2 "" H 2400 3050 50  0000 C CNN
@@
 $EndComp
 Text GLabel 2400 2000 1    60   Input ~ 0
-VIN
+Vin
 $Comp
 L CP C2
@@
 $EndComp
 $Comp
-L GND #PWR16
+L GND #PWR016
 U 1 1 59690AC9
 P 6350 5400
-F 0 "#PWR16" H 6350 5150 50  0001 C CNN
+F 0 "#PWR016" H 6350 5150 50  0001 C CNN
 F 1 "GND" H 6350 5250 50  0000 C CNN
 F 2 "" H 6350 5400 50  0000 C CNN
@@
 $EndComp
 $Comp
-L GND #PWR14
+L GND #PWR017
 U 1 1 59690B3F
 P 4700 5250
-F 0 "#PWR14" H 4700 5000 50  0001 C CNN
+F 0 "#PWR017" H 4700 5000 50  0001 C CNN
 F 1 "GND" H 4700 5100 50  0000 C CNN
 F 2 "" H 4700 5250 50  0000 C CNN
@@
 $EndComp
 $Comp
-L GND #PWR15
+L GND #PWR018
 U 1 1 59690D86
 P 5900 5450
-F 0 "#PWR15" H 5900 5200 50  0001 C CNN
+F 0 "#PWR018" H 5900 5200 50  0001 C CNN
 F 1 "GND" H 5900 5300 50  0000 C CNN
 F 2 "" H 5900 5450 50  0000 C CNN
@@
 $EndComp
 $Comp
-L GND #PWR13
+L GND #PWR019
 U 1 1 59691C20
 P 2750 5600
-F 0 "#PWR13" H 2750 5350 50  0001 C CNN
+F 0 "#PWR019" H 2750 5350 50  0001 C CNN
 F 1 "GND" H 2750 5450 50  0000 C CNN
 F 2 "" H 2750 5600 50  0000 C CNN
@@
 F 1 "5K" V 2750 5400 50  0000 C CNN
 F 2 "Resistors_SMD:R_0603_HandSoldering" V 2680 5400 50  0001 C CNN
-F 3 "http://www.digikey.com/en/resources/datasheets/yageo/rc-series-l-suffix-datasheet" H 2750 5400 50  0001 C CNN
-F 4 "RC0603JR-0710KL" V 2750 5400 60  0001 C CNN "Part Number"
+F 3 "https://www.digikey.com/product-detail/en/yageo/RC0402FR-074K99L/311-4.99KLRCT-ND/2827886" H 2750 5400 50  0001 C CNN
+F 4 "RC0402FR-074K99L" V 2750 5400 60  0001 C CNN "Part Number"
 	1    2750 5400
 	-1   0    0    1
@@
 	3100 4200 2900 4200
 $Comp
-L CONN_01X02 J?
+L CONN_01X02 J2
 U 1 1 597573B9
 P 5200 2550
-F 0 "J?" H 5278 2591 50  0000 L CNN
+F 0 "J2" H 5278 2591 50  0000 L CNN
 F 1 "CONN_01X02" H 5278 2500 50  0000 L CNN
-F 2 "" H 5200 2550 50  0001 C CNN
-F 3 "" H 5200 2550 50  0001 C CNN
+F 2 "footprints:battery_input" H 5200 2550 50  0001 C CNN
+F 3 "https://www.digikey.com/product-detail/en/phoenix-contact/1934861/277-1607-ND/568644" H 5200 2550 50  0001 C CNN
 	1    5200 2550
 	1    0    0    -1
@@
 	4900 2500 5000 2500
 $Comp
-L GND #PWR?
+L GND #PWR020
 U 1 1 59757643
 P 4950 2650
-F 0 "#PWR?" H 4950 2400 50  0001 C CNN
+F 0 "#PWR020" H 4950 2400 50  0001 C CNN
 F 1 "GND" H 4950 2500 50  0000 C CNN
 F 2 "" H 4950 2650 50  0000 C CNN

Commit message: update
Parts:
- U2: symbol ZXCT1107 -> ZXCT1107-RESCUE-5v-smart-solar-regulator
Changed lines of the file:
@@
 EESchema Schematic File Version 2
+LIBS:5v-smart-solar-regulator-rescue
 LIBS:power
 LIBS:device
@@
 LIBS:open-automation
 LIBS:5v-smart-solar-regulator-cache
-EELAYER 25 0
+EELAYER 26 0
 EELAYER END
 $Descr A4 11693 8268
@@
 $EndComp
 $Comp
-L ZXCT1107 U2
+L ZXCT1107-RESCUE-5v-smart-solar-regulator U2
 U 1 1 59691952
 P 2800 4800
+AR Path="/59691952" Ref="U2"  Part="1"
+AR Path="/5936D89B/59691952" Ref="U2"  Part="1"
 F 0 "U2" V 3000 4600 60  0000 C CNN
 F 1 "ZXCT1107" V 2550 5100 60  0000 C CNN
