File: hardware/power.sch (KiCad schematic (older format))
At the start: 25 parts, among them J2 CONN_01X02, Q1 Q_PMOS_GSD_BSS84, U11 SPX1117M3-L-3-3/TR, U2 ZXCT1107, U3 LM2576, U6 OPA344NA/3K

Commit message: update
Parts:
- removed Q1: Q_PMOS_GSD_BSS84, TO_SOT_Packages_SMD:SOT-23, symbol Q_PMOS_GSD_BSS84
- removed R10: 100K, Resistors_SMD:R_0603_HandSoldering, symbol R
- removed R11, R7: 82K, Resistors_SMD:R_0603_HandSoldering, symbol R
- removed R12, R13: 1K, Resistors_SMD:R_0603_HandSoldering, symbol R
- removed R8: 30K, Resistors_SMD:R_0603_HandSoldering, symbol R
- removed R9: 3M, Resistors_SMD:R_0603_HandSoldering, symbol R
- removed U6: OPA344NA/3K, TO_SOT_Packages_SMD:SOT-23-5, symbol OPA344NA/3K
Connections:
- net labels removed: IO33
- wire segments 68 -> 42
Other:
- moved on the sheet: R20

Commit message: update
Parts:
- removed R20: 1K, Resistors_SMD:R_0603_HandSoldering, symbol R
- removed R6: 10K, Resistors_SMD:R_0603_HandSoldering, symbol R
- removed U2: ZXCT1107, footprints:Current_sense-ZXCT1107, symbol ZXCT1107-RESCUE-5v-smart-solar-regulator
- added C7, C8: C_0.1uF, Capacitors_SMD:C_0603_HandSoldering, symbol C_0.1uF
- added PANEL1: CONN_01X02, open-automation:XT60, symbol CONN_01X02
- added Q1: Q_NMOS_GSD_PSMN038-100YLX, open-automation:SOT-669_PSMN038-100YLX, symbol Q_NMOS_GSD_PSMN038-100YLX
- added R8: R_10k, Resistors_SMD:R_0603_HandSoldering, symbol R_10k
- added U2, U5: Power-Monitor-INA219, TO_SOT_Packages_SMD:SOT-23-8_Handsoldering, symbol Power-Monitor-INA219
- BATTERY1: renamed from J2; footprint footprints:battery_input -> open-automation:XT60
- C1: footprint footprints:smd-cap-13.5 -> open-automation:CAP-RAD-5mm-UVR1H102MHD; Part Number EEV-FK1K101Q -> 860240675007
- C2: footprint footprints:smd-cap-13.5 -> open-automation:CAP-RAD-5mm-UVR1H102MHD; Part Number UUG1E102MNQ1MS -> UVR1H102MHD
- C3: footprint Capacitors_SMD:C_0603 -> Capacitors_SMD:C_0603_HandSoldering
- L1: footprint footprints:Inductor-SRR1210 -> open-automation:L-RAD-7.4mm; Part Number SRR1210-470M -> AIUR-06-470K
- R3: value 100K -> 1K; Part Number RC0603JR-07100KL -> RC0603JR-071KL
- R4: value 25K -> 50m; footprint Resistors_SMD:R_0603_HandSoldering -> Resistors_SMD:R_0805_HandSoldering; Part Number RC0603FR-0724K9L -> RL1220T-R050-J
- U11: footprint TO_SOT_Packages_SMD:SOT-223 -> open-automation:SPX1117M3; Part Number SPX1117M3-L-3-3/TR -> 1016-1848-1-ND
- U3: footprint footprints:Regulator-LM2576 -> open-automation:Regulator-LM2576
Connections:
- net BATTERY: now also Q1.2 (S); no longer R5.1
- net GND: now also C7.1, C8.1, PANEL1.2 (P2), R8.2, U2.3 (GND), U2.7 (A0), U2.8 (A1), U5.3 (GND), U5.8 (A1); no longer R4.1
- net power_EN: now also R8.1
- net 3v3 renamed 3V3
- net 3V3: now also R3.1, U5.7 (A0)
- net 5V renamed V_USB
- net IO4 renamed BAT_SW
- net BAT_SW: now also Q1.1 (G); no longer R4.2
- net Vin renamed V_MAIN
- net V_MAIN: now also R4.2, U2.2 (IN-), U5.2 (IN-); no longer R3.1
- new net: Q1.3 (D), R5.1, U5.1 (IN+)
- new net SCL: U2.5 (SCL), U5.5 (SCL)
- new net SDA: U2.6 (SDA), U5.6 (SDA)
- new net VCC_I2C: C7.2, C8.2, U2.4 (Vs), U5.4 (Vs)
- new net V_PANEL: PANEL1.1 (P1), R4.1, U2.1 (IN+)
Other:
- moved on the sheet: BATTERY1, C1, C2, C3, D1, D4, R2, R5, U11, U3

Commit message: update
Parts:
- removed C7: C_0.1uF, Capacitors_SMD:C_0603_HandSoldering, symbol C_0.1uF
- removed R2, R3: 1K, Resistors_SMD:R_0603_HandSoldering, symbol R
- removed R4: 50m, Resistors_SMD:R_0805_HandSoldering, symbol R
- removed U2: Power-Monitor-INA219, TO_SOT_Packages_SMD:SOT-23-8_Handsoldering, symbol Power-Monitor-INA219
- added R11: R_10k, Resistors_SMD:R_0603_HandSoldering, symbol R_10k
- added R7: 1K, Resistors_SMD:R_0603_HandSoldering, symbol R
- C2: footprint open-automation:CAP-RAD-5mm-UVR1H102MHD -> Capacitors_THT:CP_Radial_D10.0mm_P3.50mm
Connections:
- net 3V3: now also R7.1; no longer U5.7 (A0)
- net BATTERY: now also R5.1, U5.1 (IN+); no longer Q1.2 (S)
- net GND: now also R11.2
- net VCC_I2C: now also U5.7 (A0)
- net V_MAIN: now also Q1.3 (D)
- net V_PANEL: now also Q1.2 (S)
- net at D4.1 (K): now also R11.1
- net BAT_SW renamed PANEL_SW
- net PANEL_SW: now also R7.2

Commit message: update
Parts:
- C1: footprint open-automation:CAP-RAD-5mm-UVR1H102MHD -> Capacitors_THT:CP_Radial_D10.0mm_P3.50mm; Part Number 860240675007 -> UVR1H101MPD
- C2: Part Number UVR1H102MHD -> UVR0J102MPD1TD
Changed lines of the file:
@@
 F 0 "C1" V 7950 3525 50  0000 L CNN
 F 1 "100uF" V 7750 3375 50  0000 L CNN
-F 2 "open-automation:CAP-RAD-5mm-UVR1H102MHD" H 7938 3325 50  0001 C CNN
-F 3 "https://www.digikey.com/product-detail/en/wurth-electronics-inc/860240675007/732-9294-3-ND/5727524" H 7900 3475 50  0001 C CNN
-F 4 "860240675007" H 7900 3475 60  0001 C CNN "Part Number"
+F 2 "Capacitors_THT:CP_Radial_D10.0mm_P3.50mm" H 7938 3325 50  0001 C CNN
+F 3 "https://www.digikey.com/product-detail/en/nichicon/UVR1H101MPD/493-1107-ND/588848" H 7900 3475 50  0001 C CNN
+F 4 "UVR1H101MPD" H 7900 3475 60  0001 C CNN "Part Number"
 	1    7900 3475
 	0    1    1    0
@@
 F 1 "1000uF" H 9925 3725 50  0000 L CNN
 F 2 "Capacitors_THT:CP_Radial_D10.0mm_P3.50mm" H 9938 3675 50  0001 C CNN
-F 3 "https://www.digikey.com/product-detail/en/nichicon/UVR1H102MHD/493-1111-ND/588852" H 9900 3825 50  0001 C CNN
-F 4 "UVR1H102MHD" H 9900 3825 60  0001 C CNN "Part Number"
+F 3 "https://www.digikey.com/product-detail/en/nichicon/UVR0J102MPD1TD/493-12738-1-ND/4328447" H 9900 3825 50  0001 C CNN
+F 4 "UVR0J102MPD1TD" H 9900 3825 60  0001 C CNN "Part Number"
 	1    9900 3825
 	1    0    0    -1

Commit message: update
Parts:
- removed Q1: Q_NMOS_GSD_PSMN038-100YLX, open-automation:SOT-669_PSMN038-100YLX, symbol Q_NMOS_GSD_PSMN038-100YLX
- removed R5: 50m, Resistors_SMD:R_0805_HandSoldering, symbol R
- removed U11: SPX1117M3-L-3-3/TR, open-automation:SPX1117M3, symbol SPX1117M3-L-3-3/TR
- added Q1: Q_NMOS_GSD_AOD4184A, TO_SOT_Packages_SMD:TO-252-2_Rectifier, symbol Q_NMOS_GSD_AOD4184A
- added R1: R_10m, Resistors_SMD:R_2512_HandSoldering, symbol R_10m
- added U11: NCP1117LPST33T3G, TO_SOT_Packages_SMD:SOT-223, symbol NCP1117LPST33T3G
- D4: footprint Diodes_SMD:D_0603 -> LEDs:LED_0603_HandSoldering
Connections:
- net VCC_I2C is gone; now on net 3V3: C8.2, U5.4 (Vs), U5.7 (A0)
- net 3V3: now also U11.2 (Vout)
- net BATTERY: now also R1.1
- net GND: now also U11.1 (GND)
- net PANEL_SW: now also Q1.1 (G)
- net V_MAIN: now also Q1.3 (D), R1.2, U11.3 (Vin)
- net V_PANEL: now also Q1.2 (S)
Changed lines of the file:
@@
 	0    1    1    0
-$EndComp
-$Comp
-L R R5
-U 1 1 59691BB3
-P 4150 4725
-F 0 "R5" V 4230 4725 50  0000 C CNN
-F 1 "50m" V 4150 4725 50  0000 C CNN
-F 2 "Resistors_SMD:R_0805_HandSoldering" V 4080 4725 50  0001 C CNN
-F 3 "https://www.digikey.com/product-detail/en/susumu/RL1220T-R050-J/RL12T.05JCT-ND/567358" H 4150 4725 50  0001 C CNN
-F 4 "RL1220T-R050-J" V 4150 4725 60  0001 C CNN "Part Number"
-	1    4150 4725
-	1    0    0    -1
 $EndComp
 Text GLabel 4075 4525 0    60   Input ~ 0
@@
 Text GLabel 7750 3675 0    60   Input ~ 0
 power_EN
-$Comp
-L SPX1117M3-L-3-3/TR U11
-U 1 1 598F6A23
-P 8675 4950
-F 0 "U11" H 8800 4750 50  0000 C CNN
-F 1 "SPX1117M3-L-3-3/TR" H 8675 5200 50  0000 C CNN
-F 2 "open-automation:SPX1117M3" H 8675 4550 50  0001 C CIN
-F 3 "https://www.digikey.com/product-detail/en/exar-corporation/SPX1117M3-L-3-3-TR/1016-1848-1-ND/3586565" H 8725 4450 50  0001 C CNN
-F 4 "1016-1848-1-ND" H 8675 4950 60  0001 C CNN "Part Number"
-	1    8675 4950
-	1    0    0    -1
-$EndComp
 $Comp
 L GND #PWR015
@@
 F 0 "D4" H 9525 5300 50  0000 C CNN
 F 1 "LED" H 9525 5100 50  0000 C CNN
-F 2 "Diodes_SMD:D_0603" H 9525 5200 50  0001 C CNN
+F 2 "LEDs:LED_0603_HandSoldering" H 9525 5200 50  0001 C CNN
 F 3 "https://www.digikey.com/product-detail/en/rohm-semiconductor/SML-D12M8WT86/511-1578-1-ND/1641810" H 9525 5200 50  0001 C CNN
 F 4 "SML-D12M8WT86" H 9525 5200 60  0001 C CNN "Part Number"
@@
 $EndComp
 Text GLabel 4500 4275 2    60   Input ~ 0
-VCC_I2C
+3V3
 $Comp
 L C_0.1uF C8
@@
 Wire Wire Line
 	5700 4575 5700 4550
-$Comp
-L Q_NMOS_GSD_PSMN038-100YLX Q1
-U 1 1 59E3D0E0
-P 4875 3175
-F 0 "Q1" V 4775 3050 50  0000 L CNN
-F 1 "Q_NMOS_GSD_PSMN038-100YLX" V 5100 2475 50  0000 L CNN
-F 2 "open-automation:SOT-669_PSMN038-100YLX" H 5075 3275 50  0001 C CNN
-F 3 "https://www.digikey.com/product-detail/en/nexperia-usa-inc/PSMN038-100YLX/1727-1815-1-ND/4813999" H 5075 3225 50  0001 C CNN
-F 4 "PSMN038-100YLX" H 5175 3325 60  0001 C CNN "Part Number"
-	1    4875 3175
-	0    1    1    0
-$EndComp
 Wire Wire Line
 	4525 3275 4675 3275
@@
 $EndComp
 Text GLabel 5675 4675 2    60   Input ~ 0
-VCC_I2C
+3V3
 Wire Wire Line
 	5675 4675 5550 4675
+$Comp
+L NCP1117LPST33T3G U11
+U 1 1 5A105FD6
+P 8675 4950
+F 0 "U11" H 8800 4750 50  0000 C CNN
+F 1 "NCP1117LPST33T3G" H 8675 5200 50  0000 C CNN
+F 2 "TO_SOT_Packages_SMD:SOT-223" H 8625 4675 50  0001 C CIN
+F 3 "https://www.digikey.com/product-detail/en/on-semiconductor/NCP1117LPST33T3G/NCP1117LPST33T3GOSCT-ND/3462387" H 8650 4600 50  0001 C CNN
+F 4 "NCP1117LPST33T3G" H 8700 5275 60  0001 C CNN "Part Number"
+	1    8675 4950
+	1    0    0    -1
+$EndComp
+$Comp
+L R_10m R1
+U 1 1 5A108421
+P 4150 4750
+F 0 "R1" H 4125 4750 50  0000 C CNN
+F 1 "R_10m" H 4125 4650 50  0000 C CNN
+F 2 "Resistors_SMD:R_2512_HandSoldering" H 4125 4575 50  0001 C CNN
+F 3 "https://www.digikey.com/product-detail/en/bourns-inc/CRA2512-FZ-R010ELF/CRA2512-FZ-R010ELFCT-ND/1775054" H 4150 4500 50  0001 C CNN
+F 4 "CRA2512-FZ-R010ELF" H 4150 4825 60  0001 C CNN "Part Number"
+	1    4150 4750
+	0    1    1    0
+$EndComp
+$Comp
+L Q_NMOS_GSD_AOD4184A Q1
+U 1 1 5A109055
+P 4800 3250
+F 0 "Q1" V 4650 3225 50  0000 L CNN
+F 1 "Q_NMOS_GSD_AOD4184A" V 4950 2825 50  0000 L CNN
+F 2 "TO_SOT_Packages_SMD:TO-252-2_Rectifier" H 4850 2950 50  0001 C CNN
+F 3 "https://www.digikey.com/products/en?keywords=785-1221-1-ND" H 4850 3025 50  0001 C CNN
+F 4 "AOD4184A" H 4850 2875 60  0001 C CNN "Part Number"
+	1    4800 3250
+	0    1    1    0
+$EndComp
 $EndSCHEMATC

Commit message: regulator ya know
Parts:
- added U? (x3): LM2576, open-automation:Regulator-LM2576, symbol open-automation:LM2576
- BATTERY1, PANEL1: symbol CONN_01X02 -> Connector_Generic:Conn_01x02
- C1: symbol CP -> open-automation:C_100uF
- C2: symbol CP -> open-automation:C_1000uF
- C3: symbol C -> open-automation:C_4.7uF
- C8: symbol C_0.1uF -> open-automation:C_0.1uF
- D1: symbol D_Schottky -> Device:D_Schottky
- D4: symbol LED -> open-automation:LED-0603-R
- L1: symbol L -> open-automation:L_47uH
- Q1: symbol Q_NMOS_GSD_AOD4184A -> open-automation:Q_NMOS_GSD_AOD4184A
- R1: symbol R_10m -> open-automation:R_10m
- R11, R8: symbol R_10k -> open-automation:R_10k
- R7: symbol R -> open-automation:R_1k
- U3: symbol LM2576 -> open-automation:LM2576
- U5: symbol Power-Monitor-INA219 -> open-automation:Power-Monitor-INA219
Connections:
- net labels added: POWER_EN
- net labels removed: power_EN
- wire segments 56 -> 67

Commit message: update
Parts:
- added R? (x3): R_10m, Resistors_SMD:R_2512_HandSoldering, symbol open-automation:R_10m
Connections:
- wire segments 67 -> 70
Changed lines of the file:
@@
 	1    0    0    -1
 $EndComp
+$Comp
+L open-automation:R_10m R?
+U 1 1 5B3BA66D
+P 9650 2400
+F 0 "R?" H 9625 2607 50  0000 C CNN
+F 1 "R_10m" H 9625 2516 50  0000 C CNN
+F 2 "Resistors_SMD:R_2512_HandSoldering" H 9625 2225 50  0001 C CNN
+F 3 "https://www.digikey.com/product-detail/en/bourns-inc/CRA2512-FZ-R010ELF/CRA2512-FZ-R010ELFCT-ND/1775054" H 9650 2150 50  0001 C CNN
+F 4 "CRA2512-FZ-R010ELF" H 9650 2475 60  0001 C CNN "Part Number"
+	1    9650 2400
+	1    0    0    -1
+$EndComp
+$Comp
+L open-automation:R_10m R?
+U 1 1 5B3BA8B0
+P 9650 1725
+F 0 "R?" H 9625 1932 50  0000 C CNN
+F 1 "R_10m" H 9625 1841 50  0000 C CNN
+F 2 "Resistors_SMD:R_2512_HandSoldering" H 9625 1550 50  0001 C CNN
+F 3 "https://www.digikey.com/product-detail/en/bourns-inc/CRA2512-FZ-R010ELF/CRA2512-FZ-R010ELFCT-ND/1775054" H 9650 1475 50  0001 C CNN
+F 4 "CRA2512-FZ-R010ELF" H 9650 1800 60  0001 C CNN "Part Number"
+	1    9650 1725
+	1    0    0    -1
+$EndComp
+$Comp
+L open-automation:R_10m R?
+U 1 1 5B3BA943
+P 9650 1075
+F 0 "R?" H 9625 1282 50  0000 C CNN
+F 1 "R_10m" H 9625 1191 50  0000 C CNN
+F 2 "Resistors_SMD:R_2512_HandSoldering" H 9625 900 50  0001 C CNN
+F 3 "https://www.digikey.com/product-detail/en/bourns-inc/CRA2512-FZ-R010ELF/CRA2512-FZ-R010ELFCT-ND/1775054" H 9650 825 50  0001 C CNN
+F 4 "CRA2512-FZ-R010ELF" H 9650 1150 60  0001 C CNN "Part Number"
+	1    9650 1075
+	1    0    0    -1
+$EndComp
+Wire Wire Line
+	9475 1725 9400 1725
+Wire Wire Line
+	9475 2400 9400 2400
+Wire Wire Line
+	9475 1075 9400 1075
 $EndSCHEMATC

Commit message: dac and diodes
Parts:
- added D? (x3): D, Diode_SMD:D_SMC, symbol open-automation:D
Changed lines of the file:
@@
 Wire Wire Line
 	9475 1075 9400 1075
+$Comp
+L open-automation:D D?
+U 1 1 5B3D3C36
+P 9625 775
+F 0 "D?" H 9625 469 50  0000 C CNN
+F 1 "D" H 9625 560 50  0000 C CNN
+F 2 "Diode_SMD:D_SMC" H 9525 775 50  0001 C CNN
+F 3 "https://www.digikey.com/product-detail/en/diodes-incorporated/MURS320-13-F/MURS320-13FDICT-ND/3053318" H 9625 875 50  0001 C CNN
+F 4 "MURS320-13-F" H 9625 651 50  0000 C CNN "Part Number"
+	1    9625 775
+	-1   0    0    1
+$EndComp
+$Comp
+L open-automation:D D?
+U 1 1 5B3D9A39
+P 9650 1400
+F 0 "D?" H 9650 1094 50  0000 C CNN
+F 1 "D" H 9650 1185 50  0000 C CNN
+F 2 "Diode_SMD:D_SMC" H 9550 1400 50  0001 C CNN
+F 3 "https://www.digikey.com/product-detail/en/diodes-incorporated/MURS320-13-F/MURS320-13FDICT-ND/3053318" H 9650 1500 50  0001 C CNN
+F 4 "MURS320-13-F" H 9650 1276 50  0000 C CNN "Part Number"
+	1    9650 1400
+	-1   0    0    1
+$EndComp
+$Comp
+L open-automation:D D?
+U 1 1 5B3D9B00
+P 9625 2050
+F 0 "D?" H 9625 1744 50  0000 C CNN
+F 1 "D" H 9625 1835 50  0000 C CNN
+F 2 "Diode_SMD:D_SMC" H 9525 2050 50  0001 C CNN
+F 3 "https://www.digikey.com/product-detail/en/diodes-incorporated/MURS320-13-F/MURS320-13FDICT-ND/3053318" H 9625 2150 50  0001 C CNN
+F 4 "MURS320-13-F" H 9625 1926 50  0000 C CNN "Part Number"
+	1    9625 2050
+	-1   0    0    1
+$EndComp
 $EndSCHEMATC
