File: hardware/power.sch (KiCad schematic (older format))
At the start: 26 parts, among them Q1 Q_NMOS_GSD_AOD4184A, U11 NCP1117LPST33T3G, U3 LM2576, U5 Power-Monitor-INA219

Commit message: additional components
Parts:
- added R? (x6): R_10k, Resistor_SMD:R_0603_1608Metric_Pad0.99x1.00mm_HandSolder, symbol open-automation:R_10k
- added U?: ACS712ELCTR-05B-T_NRND, open-automation:ACS711, symbol dk_Current-Transducers:ACS712ELCTR-05B-T_NRND
Connections:
- wire segments 70 -> 91
Other:
- note added: "POWER"
- moved on the sheet: BATTERY1, C3, C8, D4, D?, PANEL1, R1, R11, R7, R8, R?, U5

Commit message: layout complete bitches
Parts:
- removed BATTERY1, PANEL1: CONN_01X02, open-automation:XT60, symbol Connector_Generic:Conn_01x02
- removed D? (x2): D, Diode_SMD:D_SMC, symbol open-automation:D
- removed R1, R? (x2): R_10m, Resistors_SMD:R_2512_HandSoldering, symbol open-automation:R_10m
- removed R? (x4): R_10k, Resistor_SMD:R_0603_1608Metric_Pad0.99x1.00mm_HandSolder, symbol open-automation:R_10k
- removed U11: NCP1117LPST33T3G, TO_SOT_Packages_SMD:SOT-223, symbol NCP1117LPST33T3G
- removed U? (x2): LM2576, open-automation:Regulator-LM2576, symbol open-automation:LM2576
- added C10, C3, C9: C_0.1uF, Capacitor_SMD:C_0603_1608Metric_Pad1.05x0.95mm_HandSolder, symbol open-automation:C_0.1uF
- added C4: C_10uF, Capacitor_SMD:C_0603_1608Metric_Pad1.05x0.95mm_HandSolder, symbol open-automation:C_10uF
- added C5, C6, C7: C_10uF, Capacitor_SMD:C_1206_3216Metric_Pad1.42x1.75mm_HandSolder, symbol open-automation:C_10uF
- added D4, D5: D, Diode_SMD:D_SMC, symbol open-automation:D
- added R11, R12, R13, R14: R_10k, Resistor_SMD:R_0603_1608Metric_Pad1.05x0.95mm_HandSolder, symbol open-automation:R_10k
- added R17, R18, R9: R_1k, Resistor_SMD:R_0603_1608Metric_Pad1.05x0.95mm_HandSolder, symbol open-automation:R_1k
- added R7, R8: R_10m, Resistor_SMD:R_2512_6332Metric_Pad1.52x3.35mm_HandSolder, symbol open-automation:R_10m
- added U10, U9: Power-Monitor-INA219, Package_TO_SOT_SMD:SOT-23-8_Handsoldering, symbol open-automation:Power-Monitor-INA219
- added U11: DAC, Package_DFN_QFN:DFN-14-1EP_3x3mm_P0.4mm_EP1.78x2.35mm, symbol open-automation:DAC
- added U12: ZLDO1117G33TA, Package_TO_SOT_SMD:SOT-223, symbol open-automation:ZLDO1117G33TA
- added U4, U5: LM2576, open-automation:Regulator-LM2576, symbol open-automation:LM2576
- C11: renamed from C1; footprint Capacitors_THT:CP_Radial_D10.0mm_P3.50mm -> Capacitor_THT:CP_Radial_D10.0mm_P3.50mm
- C12: renamed from C3; footprint Capacitors_SMD:C_0603_HandSoldering -> Capacitor_SMD:C_0603_1608Metric_Pad1.05x0.95mm_HandSolder
- C13: renamed from C2; footprint Capacitors_THT:CP_Radial_D10.0mm_P3.50mm -> Capacitor_THT:CP_Radial_D10.0mm_P3.50mm
- C8: footprint Capacitors_SMD:C_0603_HandSoldering -> Capacitor_SMD:C_0603_1608Metric_Pad1.05x0.95mm_HandSolder
- D7: renamed from D1; footprint Diodes_SMD:D_SMA -> Diode_SMD:D_SMA
- D8: renamed from D4; footprint LEDs:LED_0603_HandSoldering -> LED_SMD:LED_0603_1608Metric_Pad0.88x0.95mm_HandSolder
- Q1: footprint TO_SOT_Packages_SMD:TO-252-2_Rectifier -> Package_TO_SOT_SMD:TO-252-2
- R10: renamed from R?; footprint Resistors_SMD:R_2512_HandSoldering -> Resistor_SMD:R_2512_6332Metric_Pad1.52x3.35mm_HandSolder
- R15, R16: renamed from R?; footprint Resistor_SMD:R_0603_1608Metric_Pad0.99x1.00mm_HandSolder -> Resistor_SMD:R_0603_1608Metric_Pad1.05x0.95mm_HandSolder
- R19: renamed from R8; footprint Resistors_SMD:R_0603_HandSoldering -> Resistor_SMD:R_0603_1608Metric_Pad1.05x0.95mm_HandSolder
- R20: renamed from R11; footprint Resistors_SMD:R_0603_HandSoldering -> Resistor_SMD:R_0603_1608Metric_Pad1.05x0.95mm_HandSolder
- R21: renamed from R7; footprint Resistors_SMD:R_0603_HandSoldering -> Resistor_SMD:R_0603_1608Metric_Pad1.05x0.95mm_HandSolder
- U8: renamed from U5; footprint TO_SOT_Packages_SMD:SOT-23-8_Handsoldering -> Package_TO_SOT_SMD:SOT-23-8_Handsoldering
- gave numbers to parts that had none: 3
- renumbered U3 to U13
Connections:
- net labels added: +3V3, OUT1, OUT2, OUT3, PANEL, REG1_POST_CURR, REG1_PRE, REG2_POST_CURR, REG2_PRE, REG3_POST_CURR, REG3_PRE, REG_POWER
- net labels removed: BATTERY
- wire segments 91 -> 205
Other:
- moved on the sheet: C8, D6, R10, R15, R16, R21, U8

Commit message: multifile update
Parts:
- removed C11: 100uF, Capacitor_THT:CP_Radial_D10.0mm_P3.50mm, symbol open-automation:C_100uF
- removed C13: 1000uF, Capacitor_THT:CP_Radial_D10.0mm_P3.50mm, symbol open-automation:C_1000uF
- removed D7: D_Schottky, Diode_SMD:D_SMA, symbol Device:D_Schottky
- removed L1: 47uH, open-automation:L-RAD-7.4mm, symbol open-automation:L_47uH
- removed Q1: Q_NMOS_GSD_AOD4184A, Package_TO_SOT_SMD:TO-252-2, symbol open-automation:Q_NMOS_GSD_AOD4184A
- removed R21: 1K, Resistor_SMD:R_0603_1608Metric_Pad1.05x0.95mm_HandSolder, symbol open-automation:R_1k
- removed U13: LM2576, open-automation:Regulator-LM2576, symbol open-automation:LM2576
- added C11: C_10uF, Capacitor_SMD:C_0603_1608Metric_Pad1.05x0.95mm_HandSolder, symbol open-automation:C_10uF
- added C13: C_1uF, Capacitor_SMD:C_0603_1608Metric_Pad1.05x0.95mm_HandSolder, symbol open-automation:C_1uF
- added C16: C_10uF, Capacitor_SMD:C_1206_3216Metric_Pad1.42x1.75mm_HandSolder, symbol open-automation:C_10uF
- added R21, R?: R_10k, Resistor_SMD:R_0603_1608Metric_Pad1.05x0.95mm_HandSolder, symbol open-automation:R_10k
- added U3: LM2576, open-automation:Regulator-LM2576, symbol open-automation:LM2576
- C10, C8, C9: Part Number C0603C104K5RACTU -> CC0603ZRY5V9BB104
- C3: Part Number C1608X8R1H104K080AB -> CC0603ZRY5V9BB104
- D8: value LED -> LED-0603-R; Part Number SML-D12M8WT86 -> LS Q976-NR-1
- U4, U5, U6: Part Number IC29302WU-TR -> MIC29302WU-TR
Connections:
- net labels added: PACK1, PACK2, PACK3, USB_EN
- net labels removed: PANEL, PANEL_SW, POWER_EN
- wire segments 205 -> 222
Other:
- moved on the sheet: D4, D5, D6

Commit message: traces complete
Parts:
- gave numbers to parts that had none: 1
Changed lines of the file:
@@
 	7850 3900 7950 3900
 $Comp
-L open-automation:R_10k R?
+L open-automation:R_10k R22
 U 1 1 5B71B230
 P 7950 4075
-F 0 "R?" H 8020 4121 50  0000 L CNN
+F 0 "R22" H 8020 4121 50  0000 L CNN
 F 1 "R_10k" H 8020 4030 50  0000 L CNN
 F 2 "Resistor_SMD:R_0603_1608Metric_Pad1.05x0.95mm_HandSolder" V 7880 4075 50  0001 C CNN
@@
 	7950 4225 7950 4250
 $Comp
-L open-automation:GND #PWR?
+L open-automation:GND #PWR0115
 U 1 1 5B743D64
 P 7950 4250
-F 0 "#PWR?" H 7950 4000 50  0001 C CNN
+F 0 "#PWR0115" H 7950 4000 50  0001 C CNN
 F 1 "GND" H 7955 4077 50  0000 C CNN
 F 2 "" H 7950 4250 50  0000 C CNN

Commit message: parts
Parts:
- C10, C3, C8, C9: Part Number CC0603ZRY5V9BB104 -> GCM188R71C104KA37D
- C11: Part Number GRM188R61A106ME69D -> GRM188C80G106ME47D
- C12: Part Number CL10B475KQ8NQNC -> CL10A475KQ8NNNC
- C13: Part Number CL10B105KP8NNNC -> CL10B105MO8NNWC
- C16, C5, C6, C7: Part Number TCA1C106M8R -> GRM188C80G106ME47D
- C4: Part Number CL10A106MP8NNNC -> GRM188C80G106ME47D
- R11, R12, R13, R14, R15, R16, R19, R20, R21, R22: Part Number RC0603JR-0710KL -> RR0816P-103-D

Commit message: re-layout
Parts:
- removed U3, U4, U5, U6: LM2576, open-automation:Regulator-LM2576, symbol open-automation:LM2576
- added U3, U4, U5, U6: MIC29302, open-automation:Regulator-LM2576, symbol open-automation:MIC29302
- C16, C5, C6, C7: footprint Capacitor_SMD:C_1206_3216Metric_Pad1.42x1.75mm_HandSolder -> Capacitor_SMD:C_0603_1608Metric_Pad1.05x0.95mm_HandSolder
Changed lines of the file:
@@
 V_MAIN
-$Comp
-L open-automation:LM2576 U6
-U 1 1 5B3BDAB3
-P 1500 3425
-F 0 "U6" H 1550 3862 60  0000 C CNN
-F 1 "LM2576" H 1550 3756 60  0000 C CNN
-F 2 "open-automation:Regulator-LM2576" H 1900 3375 60  0001 C CNN
-F 3 "https://www.digikey.com/product-detail/en/microchip-technology/MIC29302WU-TR/576-1125-1-ND/771851" H 1900 3375 60  0001 C CNN
-F 4 "MIC29302WU-TR" H 1550 3658 50  0001 C CNN "Part Number"
-	1    1500 3425
-	1    0    0    -1
-$EndComp
 $Comp
 L open-automation:R_10m R10
@@
 	5300 5825 5550 5825
 $Comp
-L open-automation:LM2576 U4
-U 1 1 5B5754B6
-P 1450 4675
-F 0 "U4" H 1500 5112 60  0000 C CNN
-F 1 "LM2576" H 1500 5006 60  0000 C CNN
-F 2 "open-automation:Regulator-LM2576" H 1850 4625 60  0001 C CNN
-F 3 "https://www.digikey.com/product-detail/en/microchip-technology/MIC29302WU-TR/576-1125-1-ND/771851" H 1850 4625 60  0001 C CNN
-F 4 "MIC29302WU-TR" H 1500 4908 50  0001 C CNN "Part Number"
-	1    1450 4675
-	1    0    0    -1
-$EndComp
-$Comp
 L open-automation:R_10m R7
 U 1 1 5B5754BE
@@
 Wire Wire Line
 	525  4575 950  4575
-$Comp
-L open-automation:LM2576 U5
-U 1 1 5B584421
-P 1475 5950
-F 0 "U5" H 1525 6387 60  0000 C CNN
-F 1 "LM2576" H 1525 6281 60  0000 C CNN
-F 2 "open-automation:Regulator-LM2576" H 1875 5900 60  0001 C CNN
-F 3 "https://www.digikey.com/product-detail/en/microchip-technology/MIC29302WU-TR/576-1125-1-ND/771851" H 1875 5900 60  0001 C CNN
-F 4 "MIC29302WU-TR" H 1525 6183 50  0001 C CNN "Part Number"
-	1    1475 5950
-	1    0    0    -1
-$EndComp
 $Comp
 L open-automation:R_10m R8
@@
 F 0 "C7" H 3740 3646 50  0000 L CNN
 F 1 "C_10uF" H 3740 3555 50  0000 L CNN
-F 2 "Capacitor_SMD:C_1206_3216Metric_Pad1.42x1.75mm_HandSolder" H 3725 3900 50  0001 C CNN
+F 2 "Capacitor_SMD:C_0603_1608Metric_Pad1.05x0.95mm_HandSolder" H 3725 3900 50  0001 C CNN
 F 3 "https://www.digikey.com/product-detail/en/murata-electronics-north-america/GRM188C80G106ME47D/490-10470-1-ND/5026387" H 3625 3350 50  0001 C CNN
 F 4 "GRM188C80G106ME47D" H 3750 3800 60  0001 C CNN "Part Number"
@@
 F 0 "C5" H 3690 4896 50  0000 L CNN
 F 1 "C_10uF" H 3690 4805 50  0000 L CNN
-F 2 "Capacitor_SMD:C_1206_3216Metric_Pad1.42x1.75mm_HandSolder" H 3675 5150 50  0001 C CNN
+F 2 "Capacitor_SMD:C_0603_1608Metric_Pad1.05x0.95mm_HandSolder" H 3675 5150 50  0001 C CNN
 F 3 "https://www.digikey.com/product-detail/en/murata-electronics-north-america/GRM188C80G106ME47D/490-10470-1-ND/5026387" H 3575 4600 50  0001 C CNN
 F 4 "GRM188C80G106ME47D" H 3700 5050 60  0001 C CNN "Part Number"
@@
 F 0 "C6" H 3715 6171 50  0000 L CNN
 F 1 "C_10uF" H 3715 6080 50  0000 L CNN
-F 2 "Capacitor_SMD:C_1206_3216Metric_Pad1.42x1.75mm_HandSolder" H 3700 6425 50  0001 C CNN
+F 2 "Capacitor_SMD:C_0603_1608Metric_Pad1.05x0.95mm_HandSolder" H 3700 6425 50  0001 C CNN
 F 3 "https://www.digikey.com/product-detail/en/murata-electronics-north-america/GRM188C80G106ME47D/490-10470-1-ND/5026387" H 3600 5875 50  0001 C CNN
 F 4 "GRM188C80G106ME47D" H 3725 6325 60  0001 C CNN "Part Number"
 	1    3600 6125
-	1    0    0    -1
-$EndComp
-$Comp
-L open-automation:LM2576 U3
-U 1 1 5B4FC426
-P 8750 3900
-F 0 "U3" H 8800 4337 60  0000 C CNN
-F 1 "LM2576" H 8800 4231 60  0000 C CNN
-F 2 "open-automation:Regulator-LM2576" H 9150 3850 60  0001 C CNN
-F 3 "https://www.digikey.com/product-detail/en/microchip-technology/MIC29302WU-TR/576-1125-1-ND/771851" H 9150 3850 60  0001 C CNN
-F 4 "MIC29302WU-TR" H 8800 4133 50  0001 C CNN "Part Number"
-	1    8750 3900
 	1    0    0    -1
 $EndComp
@@
 F 0 "C16" H 10340 4121 50  0000 L CNN
 F 1 "C_10uF" H 10340 4030 50  0000 L CNN
-F 2 "Capacitor_SMD:C_1206_3216Metric_Pad1.42x1.75mm_HandSolder" H 10325 4375 50  0001 C CNN
+F 2 "Capacitor_SMD:C_0603_1608Metric_Pad1.05x0.95mm_HandSolder" H 10325 4375 50  0001 C CNN
 F 3 "https://www.digikey.com/product-detail/en/murata-electronics-north-america/GRM188C80G106ME47D/490-10470-1-ND/5026387" H 10225 3825 50  0001 C CNN
 F 4 "GRM188C80G106ME47D" H 10350 4275 60  0001 C CNN "Part Number"
@@
 	1    0    0    -1
 $EndComp
+$Comp
+L open-automation:MIC29302 U6
+U 1 1 5B6453AA
+P 8750 3900
+F 0 "U6" H 8800 4337 60  0000 C CNN
+F 1 "MIC29302" H 8800 4231 60  0000 C CNN
+F 2 "open-automation:Regulator-LM2576" H 8750 3500 60  0001 C CNN
+F 3 "https://www.digikey.com/product-detail/en/microchip-technology/MIC29302WU-TR/576-1125-1-ND/771851" H 8700 3600 60  0001 C CNN
+F 4 "IC29302WU-TR" H 8800 4133 50  0000 C CNN "Part Number"
+	1    8750 3900
+	1    0    0    -1
+$EndComp
+$Comp
+L open-automation:MIC29302 U4
+U 1 1 5B645600
+P 1475 5950
+F 0 "U4" H 1525 6387 60  0000 C CNN
+F 1 "MIC29302" H 1525 6281 60  0000 C CNN
+F 2 "open-automation:Regulator-LM2576" H 1475 5550 60  0001 C CNN
+F 3 "https://www.digikey.com/product-detail/en/microchip-technology/MIC29302WU-TR/576-1125-1-ND/771851" H 1425 5650 60  0001 C CNN
+F 4 "IC29302WU-TR" H 1525 6183 50  0000 C CNN "Part Number"
+	1    1475 5950
+	1    0    0    -1
+$EndComp
+$Comp
+L open-automation:MIC29302 U3
+U 1 1 5B645766
+P 1450 4675
+F 0 "U3" H 1500 5112 60  0000 C CNN
+F 1 "MIC29302" H 1500 5006 60  0000 C CNN
+F 2 "open-automation:Regulator-LM2576" H 1450 4275 60  0001 C CNN
+F 3 "https://www.digikey.com/product-detail/en/microchip-technology/MIC29302WU-TR/576-1125-1-ND/771851" H 1400 4375 60  0001 C CNN
+F 4 "IC29302WU-TR" H 1500 4908 50  0000 C CNN "Part Number"
+	1    1450 4675
+	1    0    0    -1
+$EndComp
+$Comp
+L open-automation:MIC29302 U5
+U 1 1 5B6532CD
+P 1500 3425
+F 0 "U5" H 1550 3862 60  0000 C CNN
+F 1 "MIC29302" H 1550 3756 60  0000 C CNN
+F 2 "open-automation:Regulator-LM2576" H 1500 3025 60  0001 C CNN
+F 3 "https://www.digikey.com/product-detail/en/microchip-technology/MIC29302WU-TR/576-1125-1-ND/771851" H 1450 3125 60  0001 C CNN
+F 4 "IC29302WU-TR" H 1550 3658 50  0000 C CNN "Part Number"
+	1    1500 3425
+	1    0    0    -1
+$EndComp

Commit message: traces complete
Parts:
- added D7, D9: D, open-automation:SOD128, symbol open-automation:D
- added R23, R24, R25: R_10k, Resistor_SMD:R_0603_1608Metric_Pad1.05x0.95mm_HandSolder, symbol open-automation:R_10k
- D4, D5, D6: footprint Diode_SMD:D_SMC -> open-automation:SOD128; Part Number MURS320-13-F -> PMEG3030EP,115
Connections:
- net labels added: REG1, REG1_EN, REG2, REG2_EN, REG3, REG3_EN
- net labels removed: +3V3
- wire segments 222 -> 237
Changed lines of the file:
@@
 $Descr A4 11693 8268
 encoding utf-8
-Sheet 4 5
+Sheet 3 5
 Title ""
 Date ""
@@
 	9475 5450 9475 5400
 Wire Wire Line
-	8525 5300 8625 5300
+	7850 5150 7950 5150
 Wire Wire Line
 	8575 5500 8625 5500
@@
 Text HLabel 6900 3925 2    50   Input ~ 0
 SDA
-Text HLabel 8525 5300 0    50   Input ~ 0
+Text HLabel 7850 5150 0    50   Input ~ 0
 V_MAIN
 $Comp
@@
 Wire Wire Line
 	2175 3425 2150 3425
-$Comp
-L open-automation:D D6
-U 1 1 5B3D3C36
-P 2525 3000
-F 0 "D6" H 2525 2784 50  0000 C CNN
-F 1 "D" H 2525 2875 50  0000 C CNN
-F 2 "Diode_SMD:D_SMC" H 2425 3000 50  0001 C CNN
-F 3 "https://www.digikey.com/product-detail/en/diodes-incorporated/MURS320-13-F/MURS320-13FDICT-ND/3053318" H 2525 3100 50  0001 C CNN
-F 4 "MURS320-13-F" H 2525 2876 50  0001 C CNN "Part Number"
-	1    2525 3000
-	-1   0    0    1
-$EndComp
 Text Notes 7100 6950 0    197  ~ 0
 POWER
@@
 Wire Wire Line
 	1850 975  1675 975
-$Comp
-L open-automation:+3V3 #PWR015
-U 1 1 5B3FDB9A
-P 1675 750
-F 0 "#PWR015" H 1675 600 50  0001 C CNN
-F 1 "+3V3" H 1690 923 50  0000 C CNN
-F 2 "" H 1675 750 50  0000 C CNN
-F 3 "" H 1675 750 50  0000 C CNN
-	1    1675 750
-	1    0    0    -1
-$EndComp
 Wire Wire Line
 	1675 975  1675 1000
@@
 Wire Wire Line
 	2125 4675 2100 4675
-$Comp
-L open-automation:D D4
-U 1 1 5B5754C7
-P 2425 4350
-F 0 "D4" H 2425 4134 50  0000 C CNN
-F 1 "D" H 2425 4225 50  0000 C CNN
-F 2 "Diode_SMD:D_SMC" H 2325 4350 50  0001 C CNN
-F 3 "https://www.digikey.com/product-detail/en/diodes-incorporated/MURS320-13-F/MURS320-13FDICT-ND/3053318" H 2425 4450 50  0001 C CNN
-F 4 "MURS320-13-F" H 2425 4226 50  0001 C CNN "Part Number"
-	1    2425 4350
-	-1   0    0    1
-$EndComp
 Wire Wire Line
 	2050 4575 3000 4575
@@
 Wire Wire Line
 	2150 5950 2125 5950
-$Comp
-L open-automation:D D5
-U 1 1 5B584432
-P 2400 5650
-F 0 "D5" H 2400 5434 50  0000 C CNN
-F 1 "D" H 2400 5525 50  0000 C CNN
-F 2 "Diode_SMD:D_SMC" H 2300 5650 50  0001 C CNN
-F 3 "https://www.digikey.com/product-detail/en/diodes-incorporated/MURS320-13-F/MURS320-13FDICT-ND/3053318" H 2400 5750 50  0001 C CNN
-F 4 "MURS320-13-F" H 2400 5526 50  0001 C CNN "Part Number"
-	1    2400 5650
-	-1   0    0    1
-$EndComp
 Wire Wire Line
 	2075 5850 3025 5850
@@
 Text Label 550  5850 0    50   ~ 0
 REG_POWER
-Wire Wire Line
-	550  5850 975  5850
 Wire Wire Line
 	2575 4350 2650 4350
@@
 REG_POWER
 Wire Wire Line
-	1000 3425 925  3425
-Wire Wire Line
-	925  3425 925  3525
-Connection ~ 925  3525
-Wire Wire Line
-	950  4675 875  4675
-Wire Wire Line
-	875  4675 875  4775
-Connection ~ 875  4775
-Wire Wire Line
-	975  5950 900  5950
-Wire Wire Line
-	900  5950 900  6050
-Connection ~ 900  6050
-Wire Wire Line
 	9350 3800 9650 3800
 Wire Wire Line
@@
 	1    0    0    -1
 $EndComp
+$Comp
+L open-automation:R_10k R23
+U 1 1 5B62A9A9
+P 5200 975
+F 0 "R23" H 5270 1021 50  0000 L CNN
+F 1 "R_10k" H 5270 930 50  0000 L CNN
+F 2 "Resistor_SMD:R_0603_1608Metric_Pad1.05x0.95mm_HandSolder" V 5130 975 50  0001 C CNN
+F 3 "https://www.digikey.com/product-detail/en/susumu/RR0816P-103-D/RR08P10.0KDCT-ND/432748" V 5280 975 50  0001 C CNN
+F 4 "RR0816P-103-D" V 5380 1075 60  0001 C CNN "Part Number"
+	1    5200 975
+	0    1    1    0
+$EndComp
+$Comp
+L open-automation:R_10k R24
+U 1 1 5B6384E6
+P 5200 1475
+F 0 "R24" H 5270 1521 50  0000 L CNN
+F 1 "R_10k" H 5270 1430 50  0000 L CNN
+F 2 "Resistor_SMD:R_0603_1608Metric_Pad1.05x0.95mm_HandSolder" V 5130 1475 50  0001 C CNN
+F 3 "https://www.digikey.com/product-detail/en/susumu/RR0816P-103-D/RR08P10.0KDCT-ND/432748" V 5280 1475 50  0001 C CNN
+F 4 "RR0816P-103-D" V 5380 1575 60  0001 C CNN "Part Number"
+	1    5200 1475
+	0    1    1    0
+$EndComp
+$Comp
+L open-automation:R_10k R25
+U 1 1 5B64605B
+P 5200 2050
+F 0 "R25" H 5270 2096 50  0000 L CNN
+F 1 "R_10k" H 5270 2005 50  0000 L CNN
+F 2 "Resistor_SMD:R_0603_1608Metric_Pad1.05x0.95mm_HandSolder" V 5130 2050 50  0001 C CNN
+F 3 "https://www.digikey.com/product-detail/en/susumu/RR0816P-103-D/RR08P10.0KDCT-ND/432748" V 5280 2050 50  0001 C CNN
+F 4 "RR0816P-103-D" V 5380 2150 60  0001 C CNN "Part Number"
+	1    5200 2050
+	0    1    1    0
+$EndComp
+Wire Wire Line
+	875  5950 975  5950
+Wire Wire Line
+	850  4675 950  4675
+Wire Wire Line
+	550  5850 975  5850
+Wire Wire Line
+	1000 3425 900  3425
+Wire Wire Line
+	5350 1475 5375 1475
+Wire Wire Line
+	5350 975  5375 975
+Wire Wire Line
+	5350 2050 5375 2050
+Wire Wire Line
+	5050 2050 4950 2050
+Wire Wire Line
+	5050 1475 4950 1475
+Wire Wire Line
+	5050 975  4975 975
+Text Label 5425 975  0    50   ~ 0
+REG1
+Text Label 5425 1475 0    50   ~ 0
+REG2
+Text Label 5425 2050 0    50   ~ 0
+REG3
+Text Label 900  3425 2    50   ~ 0
+REG1
+Text Label 850  4675 2    50   ~ 0
+REG2
+Text Label 875  5950 2    50   ~ 0
+REG3
+Text Label 4975 975  2    50   ~ 0
+REG_POWER
+Text Label 4950 1475 2    50   ~ 0
+REG_POWER
+Text Label 4950 2050 2    50   ~ 0
+REG_POWER
+Wire Wire Line
+	5375 2050 5375 2000
+Wire Wire Line
+	5375 1475 5375 1425
+Connection ~ 5375 1475
+Wire Wire Line
+	5375 1475 5425 1475
+Wire Wire Line
+	5375 925  5375 975
+Connection ~ 5375 975
+Wire Wire Line
+	5375 975  5425 975
+Text HLabel 5375 925  1    50   Input ~ 0
+REG1_EN
+Text HLabel 5375 1425 1    50   Input ~ 0
+REG2_EN
+Text HLabel 5375 2000 1    50   Input ~ 0
+REG3_EN
+Wire Wire Line
+	5425 2050 5375 2050
+Connection ~ 5375 2050
+$Comp
+L open-automation:D D7
+U 1 1 5B805AA1
+P 8100 5150
+F 0 "D7" H 8100 4934 50  0000 C CNN
+F 1 "D" H 8100 5025 50  0000 C CNN
+F 2 "open-automation:SOD128" H 8000 5150 50  0001 C CNN
+F 3 "https://www.digikey.com/product-detail/en/diodes-incorporated/MURS320-13-F/MURS320-13FDICT-ND/3053318" H 8100 5250 50  0001 C CNN
+F 4 "PMEG3030EP,115" H 8100 5026 50  0001 C CNN "Part Number"
+	1    8100 5150
+	-1   0    0    1
+$EndComp
+Wire Wire Line
+	8250 5150 8425 5150
+Wire Wire Line
+	8425 5150 8425 5300
+Wire Wire Line
+	8425 5300 8625 5300
+Wire Wire Line
+	8425 5300 8425 5475
+Wire Wire Line
+	8425 5475 8250 5475
+Connection ~ 8425 5300
+Wire Wire Line
+	7950 5475 7875 5475
+Text Label 7875 5475 2    50   ~ 0
+REG_POWER
+$Comp
+L open-automation:D D9
+U 1 1 5B8629F6
+P 8100 5475
+F 0 "D9" H 8100 5259 50  0000 C CNN
+F 1 "D" H 8100 5350 50  0000 C CNN
+F 2 "open-automation:SOD128" H 8000 5475 50  0001 C CNN
+F 3 "https://www.digikey.com/product-detail/en/diodes-incorporated/MURS320-13-F/MURS320-13FDICT-ND/3053318" H 8100 5575 50  0001 C CNN
+F 4 "PMEG3030EP,115" H 8100 5351 50  0001 C CNN "Part Number"
+	1    8100 5475
+	-1   0    0    1
+$EndComp
+$Comp
+L open-automation:D D6
+U 1 1 5B872546
+P 2525 3000
+F 0 "D6" H 2525 2784 50  0000 C CNN
+F 1 "D" H 2525 2875 50  0000 C CNN
+F 2 "open-automation:SOD128" H 2425 3000 50  0001 C CNN
+F 3 "https://www.digikey.com/product-detail/en/diodes-incorporated/MURS320-13-F/MURS320-13FDICT-ND/3053318" H 2525 3100 50  0001 C CNN
+F 4 "PMEG3030EP,115" H 2525 2876 50  0001 C CNN "Part Number"
+	1    2525 3000
+	-1   0    0    1
+$EndComp
+$Comp
+L open-automation:D D5
+U 1 1 5B881DD6
+P 2425 4350
+F 0 "D5" H 2425 4134 50  0000 C CNN
+F 1 "D" H 2425 4225 50  0000 C CNN
+F 2 "open-automation:SOD128" H 2325 4350 50  0001 C CNN
+F 3 "https://www.digikey.com/product-detail/en/diodes-incorporated/MURS320-13-F/MURS320-13FDICT-ND/3053318" H 2425 4450 50  0001 C CNN
+F 4 "PMEG3030EP,115" H 2425 4226 50  0001 C CNN "Part Number"
+	1    2425 4350
+	-1   0    0    1
+$EndComp
+$Comp
+L open-automation:D D4
+U 1 1 5B8916A8
+P 2400 5650
+F 0 "D4" H 2400 5434 50  0000 C CNN
+F 1 "D" H 2400 5525 50  0000 C CNN
+F 2 "open-automation:SOD128" H 2300 5650 50  0001 C CNN
+F 3 "https://www.digikey.com/product-detail/en/diodes-incorporated/MURS320-13-F/MURS320-13FDICT-ND/3053318" H 2400 5750 50  0001 C CNN
+F 4 "PMEG3030EP,115" H 2400 5526 50  0001 C CNN "Part Number"
+	1    2400 5650
+	-1   0    0    1
+$EndComp
+Text GLabel 1675 750  1    50   Input ~ 0
+3V3
 $EndSCHEMATC
