File: hardware/power.sch (KiCad schematic (older format))
At the start: 47 parts, among them U10 Power-Monitor-INA219, U11 DAC, U12 ZLDO1117G33TA, U3 MIC29302, U4 MIC29302, U5 MIC29302, U6 MIC29302, U7 ACS712ELCTR-05B-T_NRND, U8 Power-Monitor-INA219, U9 Power-Monitor-INA219

Commit message: rewire
Connections:
- net labels added: MAIN_CURRENT_SENSE
Changed lines of the file:
@@
 	1    0    0    -1
 $EndComp
-Text GLabel 6900 3825 2    60   Input ~ 0
-3V3
 Wire Wire Line
 	6900 3825 6775 3825
@@
 	1    6925 3700
 	-1   0    0    1
-$EndComp
-$Comp
-L open-automation:GND #PWR025
-U 1 1 5B3B26E4
-P 5300 3425
-F 0 "#PWR025" H 5300 3175 50  0001 C CNN
-F 1 "GND" V 5305 3297 50  0000 R CNN
-F 2 "" H 5300 3425 50  0000 C CNN
-F 3 "" H 5300 3425 50  0000 C CNN
-	1    5300 3425
-	0    1    1    0
 $EndComp
 $Comp
@@
 Wire Wire Line
 	2600 3425 3225 3425
-Text Label 2975 2025 0    50   ~ 0
-REG_POWER
 Text Label 575  3325 0    50   ~ 0
 REG_POWER
@@
 Wire Wire Line
 	6925 4725 6925 4700
-Text GLabel 6900 4825 2    60   Input ~ 0
+Text GLabel 6900 5975 2    60   Input ~ 0
 3V3
 Wire Wire Line
@@
 L open-automation:GND #PWR035
 U 1 1 5B55FD46
-P 6925 4700
-F 0 "#PWR035" H 6925 4450 50  0001 C CNN
-F 1 "GND" H 6930 4527 50  0000 C CNN
-F 2 "" H 6925 4700 50  0000 C CNN
-F 3 "" H 6925 4700 50  0000 C CNN
-	1    6925 4700
-	-1   0    0    1
-$EndComp
-$Comp
-L open-automation:GND #PWR026
-U 1 1 5B55FD4C
-P 5300 4425
-F 0 "#PWR026" H 5300 4175 50  0001 C CNN
-F 1 "GND" V 5305 4297 50  0000 R CNN
-F 2 "" H 5300 4425 50  0000 C CNN
-F 3 "" H 5300 4425 50  0000 C CNN
-	1    5300 4425
-	0    1    1    0
+P 6900 4825
+F 0 "#PWR035" H 6900 4575 50  0001 C CNN
+F 1 "GND" H 6905 4652 50  0000 C CNN
+F 2 "" H 6900 4825 50  0000 C CNN
+F 3 "" H 6900 4825 50  0000 C CNN
+	1    6900 4825
+	0    -1   -1   0
 $EndComp
 Text HLabel 6900 5025 2    50   Input ~ 0
@@
 Wire Wire Line
 	6925 5875 6925 5850
-Text GLabel 6900 5975 2    60   Input ~ 0
-3V3
 Wire Wire Line
 	6900 5975 6775 5975
@@
 	1    6925 5850
 	-1   0    0    1
-$EndComp
-$Comp
-L open-automation:GND #PWR027
-U 1 1 5B56935F
-P 5300 5575
-F 0 "#PWR027" H 5300 5325 50  0001 C CNN
-F 1 "GND" V 5305 5447 50  0000 R CNN
-F 2 "" H 5300 5575 50  0000 C CNN
-F 3 "" H 5300 5575 50  0000 C CNN
-	1    5300 5575
-	0    1    1    0
 $EndComp
 Text HLabel 6900 6175 2    50   Input ~ 0
@@
 Text GLabel 1675 750  1    50   Input ~ 0
 3V3
+Text GLabel 2975 2025 2    50   Input ~ 0
+MAIN_CURRENT_SENSE
+Text GLabel 5300 4425 0    60   Input ~ 0
+3V3
+Text GLabel 5300 3425 0    60   Input ~ 0
+3V3
+Text GLabel 5300 5575 0    60   Input ~ 0
+3V3
+Text HLabel 6900 3825 2    50   Input ~ 0
+SDA
+Text GLabel 6925 4700 1    60   Input ~ 0
+3V3
 $EndSCHEMATC
