File: hardware/_autosave-5v-smart-solar-regulator.kicad_pcb (KiCad board)
At the start: 2 copper layers, 82.5 x 48.6 mm, 37 parts, among them J1 CONN_02X16, J2 CONN_01X02, P3 CONN_01X03, P4 CONN_01X04, P5 USB_A_2, Q2 Q_NMOS_GSD, Q3 Q_PMOS_GSD, U1 ESP-WROOM-32, U10 touchpad, U2 ZXCT1107, U3 LM2576, U4 housing-mounts, U5 SPX3819, U6 OPA344

Commit message: update
Changed lines of the file:
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@@
   (module footprints:battery_input (layer F.Cu)
     (at 96.774 97.028)
-    (fp_text reference J2 (at 1.4 1.25 180) (layer F.SilkS)
+    (fp_text reference J2 (at 1.27 1.778 180) (layer F.SilkS)
       (effects (font (size 1 1) (thickness 0.15)))
     )
