File: hardware/5v-smart-solar-regulator.kicad_pcb (KiCad board)
At the start: 2 copper layers, 82.5 x 48.6 mm, 38 parts, among them J1 CONN_02X16, J2 CONN_01X02, P3 CONN_01X03, P4 CONN_01X04, P5 USB_A_2, Q2 Q_NMOS_GSD, Q3 Q_PMOS_GSD, U1 ESP-WROOM-32, U10 touchpad, U2 ZXCT1107, U3 LM2576, U4 housing-mounts, U5 SPX3819, U6 OPA344

Commit message: update
Parts:
- removed R2: 10K, Resistors_SMD:R_0603_HandSoldering
- P5: footprint footprints:USB_A_2 -> open-automation:USB_A_2
- moved P5 0.79 mm to (169.8, 106.2)
Routing:
- net 3v3: track 93.5 -> 60.0 mm, vias 6 -> 2
- net IO2: track 9.50 -> 0.00 mm
- net 5V: track 235.3 -> 228.2 mm
- net GND: track 140.1 -> 139.4 mm

Commit message: update
Parts:
- moved J2 2.76 mm to (96.8, 97.0), turned to 0 degrees
Routing:
- net BATTERY: track 7.61 -> 16.3 mm
- net IO35: track 79.9 -> 73.5 mm, vias 5 -> 4
Changed lines of the file:
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@@
-(kicad_pcb (version 20170123) (host pcbnew no-vcs-found-67ae593~59~ubuntu17.04.1)
+(kicad_pcb (version 4) (host pcbnew 4.0.6+dfsg1-1)
   (general
+    (links 113)
+    (no_connects 2)
+    (area 93.142999 77.533999 175.743001 126.284001)
     (thickness 1.6)
     (drawings 24)
@@
       (hpglpenspeed 20)
       (hpglpendiameter 15)
+      (hpglpenoverlay 2)
       (psnegative false)
       (psa4output false)
@@
     (tags SOT-23)
     (attr smd)
-    (fp_text reference U2 (at 1.175 2.75 180) (layer F.SilkS)
+    (fp_text reference U2 (at 1.175 2.75 540) (layer F.SilkS)
       (effects (font (size 1 1) (thickness 0.15)))
     )
@@
   (module footprints:Regulator-LM2576 (layer F.Cu)
     (at 106.52 99.69 270)
-    (fp_text reference U3 (at -5.36 -0.19) (layer F.SilkS)
+    (fp_text reference U3 (at -5.36 -0.19 360) (layer F.SilkS)
       (effects (font (size 1 1) (thickness 0.15)))
     )
@@
     (tags SOT-23)
     (attr smd)
-    (fp_text reference Q2 (at 2.6 0) (layer B.SilkS)
+    (fp_text reference Q2 (at 2.6 0 360) (layer B.SilkS)
       (effects (font (size 1 1) (thickness 0.15)) (justify mirror))
     )
@@
   (module footprints:smd-cap-13.5 (layer F.Cu)
     (at 127.96 90.74 270)
-    (fp_text reference C2 (at 11.31 4.88) (layer F.SilkS)
+    (fp_text reference C2 (at 11.31 4.88 360) (layer F.SilkS)
       (effects (font (size 1 1) (thickness 0.15)))
     )
@@
     (tags "capacitor 0603")
     (attr smd)
-    (fp_text reference C3 (at 2.77731 0.572 180) (layer B.SilkS)
+    (fp_text reference C3 (at 2.77731 0.572 540) (layer B.SilkS)
       (effects (font (size 1 1) (thickness 0.15)) (justify mirror))
     )
@@
     (tags "capacitor 0603")
     (attr smd)
-    (fp_text reference C5 (at -2.831 -0.434) (layer B.SilkS)
+    (fp_text reference C5 (at -2.831 -0.434 360) (layer B.SilkS)
       (effects (font (size 1 1) (thickness 0.15)) (justify mirror))
     )
@@
     (descr "LED, diameter 3.0mm, 2 pins")
     (tags "LED diameter 3.0mm 2 pins")
-    (fp_text reference D3 (at 1.294 2.964) (layer F.SilkS)
+    (fp_text reference D3 (at 1.294 2.964 360) (layer F.SilkS)
       (effects (font (size 1 1) (thickness 0.15)))
     )
@@
     (tags "resistor 0603")
     (attr smd)
-    (fp_text reference R11 (at -2.80231 0.201) (layer B.SilkS)
+    (fp_text reference R11 (at -2.80231 0.201 360) (layer B.SilkS)
       (effects (font (size 1 1) (thickness 0.15)) (justify mirror))
     )
@@
     (tags "resistor 0603")
     (attr smd)
-    (fp_text reference R14 (at -2.994 0.326) (layer B.SilkS)
+    (fp_text reference R14 (at -2.994 0.326 360) (layer B.SilkS)
       (effects (font (size 1 1) (thickness 0.15)) (justify mirror))
     )
@@
     (tags "resistor 0603")
     (attr smd)
-    (fp_text reference R15 (at -2.806 0.36) (layer B.SilkS)
+    (fp_text reference R15 (at -2.806 0.36 360) (layer B.SilkS)
       (effects (font (size 1 1) (thickness 0.15)) (justify mirror))
     )
@@
     (fp_line (start 10.55 -9.4) (end 10.55 1.8) (layer B.CrtYd) (width 0.05))
     (fp_line (start 10.55 1.8) (end -1.8 1.8) (layer B.CrtYd) (width 0.05))
-    (fp_text user %R (at 2.77 -3.81) (layer B.Fab)
+    (fp_text user %R (at 2.77 -3.81 360) (layer B.Fab)
       (effects (font (size 1 1) (thickness 0.15)) (justify mirror))
     )
@@
     )
   )
-  (module footprints:battery_input (layer F.Cu)
-    (at 98.1 99.45 180)
-    (fp_text reference J2 (at 1.1 1.25) (layer F.SilkS)
-      (effects (font (size 1 1) (thickness 0.15)))
-    )
-    (fp_text value CONN_01X02 (at 1.05 7 180) (layer F.Fab)
-      (effects (font (size 1 1) (thickness 0.15)))
-    )
-    (fp_text user + (at 3.65 -2.5 180) (layer F.SilkS)
-      (effects (font (size 1 1) (thickness 0.15)))
-    )
-    (fp_text user - (at 3.8 4.9 180) (layer F.SilkS)
-      (effects (font (size 1 1) (thickness 0.15)))
-    )
-    (pad 1 thru_hole circle (at 1.1 -2.3 180) (size 3.5 3.5) (drill 2) (layers *.Cu *.Mask)
-      (net 46 BATTERY))
-    (pad 2 thru_hole rect (at 1.1 4.7 180) (size 3.5 3.5) (drill 2) (layers *.Cu *.Mask)
-      (net 1 GND))
-  )
   (module footprints:touch-pad (layer F.Cu)
     (at 140.175 111.075)
@@
     (pad 2 thru_hole circle (at 0.65 -8.45 90) (size 1.5 1.5) (drill 1.1) (layers *.Cu *.Mask)
       (net 2 5V))
+  )
+  (module footprints:battery_input (layer F.Cu)
+    (at 96.774 97.028)
+    (fp_text reference J2 (at 1.4 1.25 180) (layer F.SilkS)
+      (effects (font (size 1 1) (thickness 0.15)))
+    )
+    (fp_text value CONN_01X02 (at 1.05 7) (layer F.Fab)
+      (effects (font (size 1 1) (thickness 0.15)))
+    )
+    (fp_text user + (at -1.778 -2.54) (layer F.SilkS)
+      (effects (font (size 1 1) (thickness 0.15)))
+    )
+    (fp_text user - (at -1.524 4.572) (layer F.SilkS)
+      (effects (font (size 1 1) (thickness 0.15)))
+    )
+    (pad 1 thru_hole circle (at 1.1 -2.3) (size 4 4) (drill 2.75) (layers *.Cu *.Mask)
+      (net 46 BATTERY))
+    (pad 2 thru_hole rect (at 1.1 4.7) (size 3.5 3.5) (drill 2.75) (layers *.Cu *.Mask)
+      (net 1 GND))
   )
   (gr_line (start 93.218 111.709) (end 93.218 92.109) (layer Edge.Cuts) (width 0.15))
@@
   (segment (start 154.462999 108.968999) (end 155.638 110.144) (width 0.25) (layer F.Cu) (net 9) (status 20))
   (segment (start 113.198 91.62) (end 117.94 86.878) (width 0.5) (layer F.Cu) (net 9))
+  (segment (start 98.25 110.225) (end 98.9 110.225) (width 0.25) (layer F.Cu) (net 10))
+  (segment (start 98.9 110.225) (end 100.825 108.3) (width 0.25) (layer F.Cu) (net 10))
+  (segment (start 100.825 108.3) (end 100.825 104.699264) (width 0.25) (layer F.Cu) (net 10))
+  (segment (start 100.825 104.699264) (end 100.825 104.275) (width 0.25) (layer F.Cu) (net 10))
   (segment (start 141.685287 103.456524) (end 141.685287 103.865212) (width 0.25) (layer B.Cu) (net 10))
   (segment (start 137.524979 97.824979) (end 140.499999 100.799999) (width 0.25) (layer B.Cu) (net 10))
@@
   (segment (start 100.825 104.275) (end 101.6 103.5) (width 0.25) (layer F.Cu) (net 10))
   (segment (start 101.6 103.5) (end 104.125 103.5) (width 0.25) (layer F.Cu) (net 10))
-  (segment (start 95.025 104) (end 95.324999 104.299999) (width 0.25) (layer B.Cu) (net 10))
-  (segment (start 95.324999 104.299999) (end 100.800001 104.299999) (width 0.25) (layer B.Cu) (net 10))
   (segment (start 100.800001 104.299999) (end 100.825 104.275) (width 0.25) (layer B.Cu) (net 10))
   (via (at 100.825 104.275) (size 0.6) (drill 0.4) (layers F.Cu B.Cu) (net 10))
-  (segment (start 98.25 110.225) (end 97.6 110.225) (width 0.25) (layer F.Cu) (net 10) (status 10))
-  (segment (start 97.6 110.225) (end 95.025 107.65) (width 0.25) (layer F.Cu) (net 10))
-  (segment (start 95.025 107.65) (end 95.025 104) (width 0.25) (layer F.Cu) (net 10))
-  (via (at 95.025 104) (size 0.6) (drill 0.4) (layers F.Cu B.Cu) (net 10))
   (segment (start 118.85 102.914) (end 122.108 106.172) (width 0.25) (layer B.Cu) (net 10) (status 20))
   (segment (start 104.125 103.5) (end 104.549264 103.5) (width 0.25) (layer B.Cu) (net 10))
@@
   (segment (start 116.26 115.2) (end 117.16 115.2) (width 0.5) (layer B.Cu) (net 45) (status 10))
   (segment (start 117.16 115.2) (end 118.48 113.88) (width 0.5) (layer B.Cu) (net 45) (status 20))
-  (segment (start 96.55 105.725) (end 96.55 107.475) (width 1) (layer F.Cu) (net 46) (status 10))
-  (segment (start 96.55 107.475) (end 97.3 108.225) (width 1) (layer F.Cu) (net 46) (status 20))
-  (segment (start 97 101.75) (end 97 105.275) (width 1) (layer F.Cu) (net 46) (status 30))
-  (segment (start 97 105.275) (end 96.55 105.725) (width 1) (layer F.Cu) (net 46) (status 30))
-  (segment (start 96.55 102.2) (end 97 101.75) (width 0.25) (layer F.Cu) (net 46) (status 30))
+  (segment (start 96.55 105.725) (end 96.55 107.475) (width 2) (layer F.Cu) (net 46))
+  (segment (start 96.55 107.475) (end 97.3 108.225) (width 2) (layer F.Cu) (net 46))
+  (segment (start 96.55 105.725) (end 95.850998 105.725) (width 2) (layer F.Cu) (net 46))
+  (segment (start 95.850998 105.725) (end 94.723999 104.598001) (width 2) (layer F.Cu) (net 46))
+  (segment (start 94.723999 104.598001) (end 94.723999 97.878001) (width 2) (layer F.Cu) (net 46))
+  (segment (start 94.723999 97.878001) (end 95.874001 96.727999) (width 2) (layer F.Cu) (net 46))
+  (segment (start 95.874001 96.727999) (end 97.874 94.728) (width 2) (layer F.Cu) (net 46))
   (segment (start 113.644999 84.569999) (end 114.425 85.35) (width 0.5) (layer F.Cu) (net 47))
   (segment (start 114.425 85.35) (end 114.425 89.301002) (width 0.5) (layer F.Cu) (net 47))

Commit message: update
Parts:
- removed C4: 1uF, Capacitors_SMD:C_0603_HandSoldering
- added D4: LED, Diodes_SMD:D_0603, F.Cu at (122.5, 89.0)
- added R10: 100K, Resistors_SMD:R_0603_HandSoldering, B.Cu at (117.6, 97.1)
- added R2: 1K, Resistors_SMD:R_0603_HandSoldering, F.Cu at (123.6, 91.6)
- added R7: 82K, Resistors_SMD:R_0603_HandSoldering, B.Cu at (106.6, 96.9)
- added R8: 30K, Resistors_SMD:R_0603_HandSoldering, B.Cu at (115.5, 97.0)
- added R9: 3M, Resistors_SMD:R_0603_HandSoldering, B.Cu at (109.8, 99.9)
- added U11: SPX1117M3-L-3-3/TR, TO_SOT_Packages_SMD:SOT-223, B.Cu at (130.7, 87.4)
- added U12: AP2204K-5.0TRG1, TO_SOT_Packages_SMD:SOT-23-5, B.Cu at (103.5, 96.9)
- C3: value 1uF -> 4.7uF; footprint Capacitors_SMD:C_0603_HandSoldering -> Capacitors_SMD:C_0603; moved to F.Cu
- P3: moved to F.Cu
- R11: value 10K -> 82K
- U5: value SPX3819 -> OPA344NA/3K
- U6: value OPA344 -> OPA344NA/3K; moved to B.Cu
- moved U6 15.1 mm to (111.7, 96.9), turned to 90 degrees
- moved C3 12.6 mm to (124.7, 89.0)
- moved U5 11.0 mm to (112.8, 85.8)
- moved R19 7.67 mm to (116.6, 86.4), turned to 270 degrees
- moved R11 7.41 mm to (108.6, 96.8)
- moved R1 5.31 mm to (144.1, 90.4), turned to 0 degrees
- moved R17 3.05 mm to (113.2, 87.2)
- moved R18 2.96 mm to (113.2, 85.1)
- moved D3 2.02 mm to (114.0, 81.2)
- moved P3 0.61 mm to (133.8, 92.1), turned to 180 degrees
Connections:
- C3 pad 1: 5V -> 3v3
- R11 pad 1: GND -> Net-(R11-Pad1)
- R11 pad 2: 5V -> GND
- U3 pad 5: GND -> power_EN
- U5 pad 1: 5V -> IO34
- U5 pad 3: 5V -> Net-(D3-Pad1)
- U5 pad 4: Net-(U5-Pad4) -> Net-(R17-Pad1)
- U5 pad 5: 3v3 -> 5V
- U6 pad 1: IO34 -> power_EN
- U6 pad 3: Net-(D3-Pad1) -> Net-(R11-Pad1)
- U6 pad 4: Net-(R17-Pad1) -> Net-(R10-Pad2)
- U6 pad 5: 5V -> 5V_ref
Routing:
- net GND: track 139.4 -> 109.4 mm, vias 19 -> 16
- net Vin: track 0.07 -> 28.6 mm, vias 0 -> 2
- net 5V: track 228.2 -> 205.6 mm
- net 3v3: track 60.0 -> 74.8 mm, vias 2 -> 5
- net power_EN: track 0.00 -> 14.6 mm, vias 0 -> 1
- net 5V_ref: track 0.00 -> 10.9 mm, vias 0 -> 2
- net SD2: track 36.4 -> 27.2 mm, vias 0 -> 1
- net Net-(R10-Pad2): track 0.00 -> 8.92 mm
- net Net-(R17-Pad1): track 16.6 -> 8.82 mm, vias 0 -> 2
- net SD0: track 27.1 -> 20.5 mm
- net Net-(R11-Pad1): track 0.00 -> 6.22 mm
- net IO34: track 70.8 -> 66.3 mm
- net Net-(D1-Pad1): track 44.1 -> 48.2 mm
- net Net-(D3-Pad1): track 11.9 -> 8.67 mm, vias 0 -> 1
- net SD3: track 32.7 -> 29.5 mm
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