File: hardware/_saved_power.sch (KiCad schematic (older format))
At the start: 22 parts, among them J2 CONN_01X02, U11 SPX1117M3-L-3-3/TR, U12 AP2204K-5.0TRG1, U2 ZXCT1107, U3 LM2576, U6 OPA344NA/3K

Commit message: update
Parts:
- added R?: 100K, Resistors_SMD:R_0603_HandSoldering, symbol 100K
Changed lines of the file:
@@
+	1    0    0    -1
+$EndComp
+$Comp
+L 100K R?
+U 1 1 5991CC02
+P 6000 3850
+F 0 "R?" V 6080 3850 50  0000 C CNN
+F 1 "100K" V 6000 3850 50  0000 C CNN
+F 2 "Resistors_SMD:R_0603_HandSoldering" V 5930 3850 50  0001 C CNN
+F 3 "https://www.digikey.com/product-detail/en/yageo/RC0603JR-07100KL/311-100KGRCT-ND/729645" V 6080 3850 50  0001 C CNN
+F 4 "RC0603JR-07###L" V 6180 3950 60  0001 C CNN "Part Number"
+	1    6000 3850
 	1    0    0    -1
 $EndComp
