File: hardware/microcontroller.sch (KiCad schematic (older format))
At the start: 5 parts, among them P1 CONN_01X20, P2 CONN_01X20, U1 ESP-WROOM-32

Commit message: update
Parts:
- removed P1, P2: CONN_01X20, Pin_Headers:Pin_Header_Straight_1x20_Pitch2.54mm, symbol CONN_01X20
- added J1: CONN_02X16, Pin_Headers:Pin_Header_Straight_2x16_Pitch2.54mm, symbol CONN_02X16
Connections:
- wire segments 79 -> 74
Other:
- moved on the sheet: R1, R2, U1

Commit message: update
Connections:
- net IO14: no longer J1.23 (P23)
Changed lines of the file:
@@
 LIBS:contrib
 LIBS:valves
-LIBS:5v-solar-regulator-cache
-EELAYER 26 0
+LIBS:open-automation
+LIBS:5v-smart-solar-regulator-cache
+EELAYER 25 0
 EELAYER END
 $Descr A4 11693 8268
@@
 $EndDescr
 $Comp
-L GND #PWR2
+L GND #PWR01
 U 1 1 59097974
 P 4500 2600
-F 0 "#PWR2" H 4500 2350 50  0001 C CNN
+F 0 "#PWR01" H 4500 2350 50  0001 C CNN
 F 1 "GND" H 4500 2450 50  0000 C CNN
 F 2 "" H 4500 2600 50  0000 C CNN
@@
 $EndComp
 $Comp
-L GND #PWR1
+L GND #PWR02
 U 1 1 590979AD
 P 2600 3850
-F 0 "#PWR1" H 2600 3600 50  0001 C CNN
+F 0 "#PWR02" H 2600 3600 50  0001 C CNN
 F 1 "GND" H 2600 3700 50  0000 C CNN
 F 2 "" H 2600 3850 50  0000 C CNN
@@
 IO17
 $Comp
-L GND #PWR3
+L GND #PWR03
 U 1 1 590979B0
 P 8400 2850
-F 0 "#PWR3" H 8400 2600 50  0001 C CNN
+F 0 "#PWR03" H 8400 2600 50  0001 C CNN
 F 1 "GND" H 8400 2700 50  0000 C CNN
 F 2 "" H 8400 2850 50  0000 C CNN
@@
 Text GLabel 8350 4100 0    60   Input ~ 0
 IO12
-Text GLabel 8350 4000 0    60   Input ~ 0
-IO14
 Text GLabel 8350 3900 0    60   Input ~ 0
 IO27
@@
 EN
 $Comp
-L GND #PWR4
+L GND #PWR04
 U 1 1 590979B2
 P 9000 2850
-F 0 "#PWR4" H 9000 2600 50  0001 C CNN
+F 0 "#PWR04" H 9000 2600 50  0001 C CNN
 F 1 "GND" H 9000 2700 50  0000 C CNN
 F 2 "" H 9000 2850 50  0000 C CNN
@@
 	8350 3700 8450 3700
 Wire Wire Line
-	8350 4000 8450 4000
-Wire Wire Line
 	8350 3900 8450 3900

Commit message: update
Parts:
- removed R2: 10K, Resistors_SMD:R_0603_HandSoldering, symbol R
Other:
- moved on the sheet: R1
Changed lines of the file:
@@
 EESchema Schematic File Version 2
+LIBS:5v-smart-solar-regulator-rescue
 LIBS:power
 LIBS:device
@@
 LIBS:open-automation
 LIBS:5v-smart-solar-regulator-cache
-EELAYER 25 0
+EELAYER 26 0
 EELAYER END
 $Descr A4 11693 8268
@@
 	-1   0    0    1
 $EndComp
-Text GLabel 2600 3300 1    60   Input ~ 0
+Text GLabel 3350 3250 1    60   Input ~ 0
 IO15
 Text GLabel 5050 4600 3    60   Input ~ 0
@@
 L R R1
 U 1 1 590979AC
-P 2600 3600
-F 0 "R1" V 2680 3600 50  0000 C CNN
-F 1 "10K" V 2600 3600 50  0000 C CNN
-F 2 "Resistors_SMD:R_0603_HandSoldering" V 2530 3600 50  0001 C CNN
-F 3 "http://www.digikey.com/en/resources/datasheets/yageo/rc-series-l-suffix-datasheet" H 2600 3600 50  0001 C CNN
-F 4 "RC0603JR-0710KL" V 2600 3600 60  0001 C CNN "Part Number"
-	1    2600 3600
+P 3350 3550
+F 0 "R1" V 3430 3550 50  0000 C CNN
+F 1 "10K" V 3350 3550 50  0000 C CNN
+F 2 "Resistors_SMD:R_0603_HandSoldering" V 3280 3550 50  0001 C CNN
+F 3 "http://www.digikey.com/en/resources/datasheets/yageo/rc-series-l-suffix-datasheet" H 3350 3550 50  0001 C CNN
+F 4 "RC0603JR-0710KL" V 3350 3550 60  0001 C CNN "Part Number"
+	1    3350 3550
 	1    0    0    -1
 $EndComp
@@
 L GND #PWR02
 U 1 1 590979AD
-P 2600 3850
-F 0 "#PWR02" H 2600 3600 50  0001 C CNN
-F 1 "GND" H 2600 3700 50  0000 C CNN
-F 2 "" H 2600 3850 50  0000 C CNN
-F 3 "" H 2600 3850 50  0000 C CNN
-	1    2600 3850
+P 3350 3800
+F 0 "#PWR02" H 3350 3550 50  0001 C CNN
+F 1 "GND" H 3350 3650 50  0000 C CNN
+F 2 "" H 3350 3800 50  0000 C CNN
+F 3 "" H 3350 3800 50  0000 C CNN
+	1    3350 3800
 	1    0    0    -1
 $EndComp
 Text GLabel 5750 4600 3    60   Input ~ 0
 IO15
-Text GLabel 2850 3850 3    60   Input ~ 0
-IO2
-$Comp
-L R R2
-U 1 1 590979AE
-P 2850 3600
-F 0 "R2" V 2930 3600 50  0000 C CNN
-F 1 "10K" V 2850 3600 50  0000 C CNN
-F 2 "Resistors_SMD:R_0603_HandSoldering" V 2780 3600 50  0001 C CNN
-F 3 "http://www.digikey.com/en/resources/datasheets/yageo/rc-series-l-suffix-datasheet" H 2850 3600 50  0001 C CNN
-F 4 "RC0603JR-0710KL" V 2850 3600 60  0001 C CNN "Part Number"
-	1    2850 3600
-	1    0    0    -1
-$EndComp
-Text GLabel 2850 3250 1    60   Input ~ 0
-3v3
 $Comp
 L ESP-WROOM-32 U1
@@
 	4500 2600 4500 2650
 Wire Wire Line
-	2850 3250 2850 3450
-Wire Wire Line
-	2850 3850 2850 3750
-Wire Wire Line
-	2600 3750 2600 3850
-Wire Wire Line
-	2600 3300 2600 3450
+	3350 3700 3350 3800
+Wire Wire Line
+	3350 3250 3350 3400
 Wire Wire Line
 	4450 4050 4550 4050

Commit message: update
Connections:
- net IO27: no longer J1.21 (P21)
Changed lines of the file:
@@
 LIBS:open-automation
 LIBS:5v-smart-solar-regulator-cache
-EELAYER 26 0
+EELAYER 25 0
 EELAYER END
 $Descr A4 11693 8268
@@
 $EndDescr
 $Comp
-L GND #PWR01
+L GND #PWR2
 U 1 1 59097974
 P 4500 2600
-F 0 "#PWR01" H 4500 2350 50  0001 C CNN
+F 0 "#PWR2" H 4500 2350 50  0001 C CNN
 F 1 "GND" H 4500 2450 50  0000 C CNN
 F 2 "" H 4500 2600 50  0000 C CNN
@@
 $EndComp
 $Comp
-L GND #PWR02
+L GND #PWR1
 U 1 1 590979AD
 P 3350 3800
-F 0 "#PWR02" H 3350 3550 50  0001 C CNN
+F 0 "#PWR1" H 3350 3550 50  0001 C CNN
 F 1 "GND" H 3350 3650 50  0000 C CNN
 F 2 "" H 3350 3800 50  0000 C CNN
@@
 IO17
 $Comp
-L GND #PWR03
+L GND #PWR3
 U 1 1 590979B0
 P 8400 2850
-F 0 "#PWR03" H 8400 2600 50  0001 C CNN
+F 0 "#PWR3" H 8400 2600 50  0001 C CNN
 F 1 "GND" H 8400 2700 50  0000 C CNN
 F 2 "" H 8400 2850 50  0000 C CNN
@@
 Text GLabel 8350 4100 0    60   Input ~ 0
 IO12
-Text GLabel 8350 3900 0    60   Input ~ 0
-IO27
 Text GLabel 8350 3800 0    60   Input ~ 0
 IO26
@@
 EN
 $Comp
-L GND #PWR04
+L GND #PWR4
 U 1 1 590979B2
 P 9000 2850
-F 0 "#PWR04" H 9000 2600 50  0001 C CNN
+F 0 "#PWR4" H 9000 2600 50  0001 C CNN
 F 1 "GND" H 9000 2700 50  0000 C CNN
 F 2 "" H 9000 2850 50  0000 C CNN
@@
 	8350 3700 8450 3700
 Wire Wire Line
-	8350 3900 8450 3900
-Wire Wire Line
 	8450 3100 8350 3100
