File: hardware/microcontroller.sch (KiCad schematic (older format))
At the start: 8 parts, among them J1 Conn_02x05_Odd_Even, U1 ESP-WROOM-32

Commit message: layout complete bitches
Parts:
- removed U?: DAC, Package_DFN_QFN:DFN-14-1EP_3x3mm_P0.4mm_EP1.78x2.35mm, symbol open-automation:DAC
- C1: renamed from C4; footprint Capacitor_SMD:C_0603_1608Metric_Pad0.99x1.00mm_HandSolder -> Capacitor_SMD:C_0603_1608Metric_Pad1.05x0.95mm_HandSolder
- C2: renamed from C6; footprint Capacitor_SMD:C_0603_1608Metric_Pad0.99x1.00mm_HandSolder -> Capacitor_SMD:C_0603_1608Metric_Pad1.05x0.95mm_HandSolder
- J1: footprint Pin_Headers:Pin_Header_Straight_2x05_Pitch2.54mm -> Connector_PinHeader_2.54mm:PinHeader_2x05_P2.54mm_Vertical
- R1: renamed from R9; footprint Resistor_SMD:R_0603_1608Metric_Pad0.99x1.00mm_HandSolder -> Resistor_SMD:R_0603_1608Metric_Pad1.05x0.95mm_HandSolder
- R2: renamed from R10; footprint Resistor_SMD:R_0603_1608Metric_Pad0.99x1.00mm_HandSolder -> Resistor_SMD:R_0603_1608Metric_Pad1.05x0.95mm_HandSolder
- R3: renamed from R6; footprint Resistor_SMD:R_0603_1608Metric_Pad0.99x1.00mm_HandSolder -> Resistor_SMD:R_0603_1608Metric_Pad1.05x0.95mm_HandSolder
Connections:
- wire segments 51 -> 42
Changed lines of the file:
@@
 Microcontroller
 $Comp
-L open-automation:C_1uF C6
+L open-automation:C_1uF C2
 U 1 1 59C55B03
 P 2825 3775
-F 0 "C6" H 2825 3875 50  0000 L CNN
+F 0 "C2" H 2825 3875 50  0000 L CNN
 F 1 "C_1uF" H 2575 3675 50  0000 L CNN
-F 2 "Capacitor_SMD:C_0603_1608Metric_Pad0.99x1.00mm_HandSolder" H 2925 4075 50  0001 C CNN
+F 2 "Capacitor_SMD:C_0603_1608Metric_Pad1.05x0.95mm_HandSolder" H 2925 4075 50  0001 C CNN
 F 3 "https://www.digikey.com/product-detail/en/yageo/CC0603ZRY5V7BB105/311-1372-1-ND/2103156" H 2825 3525 50  0001 C CNN
 F 4 "CL10B105KA8VPNC" H 2950 3975 60  0001 C CNN "Part Number"
@@
 	8100 3750 8200 3750
 $Comp
-L open-automation:R_10k R6
+L open-automation:R_10k R3
 U 1 1 59C609F8
 P 6400 4700
-F 0 "R6" V 6400 4700 50  0000 C CNN
+F 0 "R3" V 6400 4700 50  0000 C CNN
 F 1 "R_10k" V 6325 4700 50  0000 C CNN
-F 2 "Resistor_SMD:R_0603_1608Metric_Pad0.99x1.00mm_HandSolder" V 6330 4700 50  0001 C CNN
+F 2 "Resistor_SMD:R_0603_1608Metric_Pad1.05x0.95mm_HandSolder" V 6330 4700 50  0001 C CNN
 F 3 "https://www.digikey.com/product-detail/en/yageo/RC0603JR-0710KL/311-10KGRCT-ND/729647" V 6480 4700 50  0001 C CNN
 F 4 "RC0603JR-0710KL" V 6580 4800 60  0001 C CNN "Part Number"
@@
 F 0 "J1" H 8450 4050 50  0000 C CNN
 F 1 "Conn_02x05_Odd_Even" H 8450 3450 50  0000 C CNN
-F 2 "Pin_Headers:Pin_Header_Straight_2x05_Pitch2.54mm" H 8400 3750 50  0001 C CNN
+F 2 "Connector_PinHeader_2.54mm:PinHeader_2x05_P2.54mm_Vertical" H 8400 3750 50  0001 C CNN
 F 3 "" H 8400 3750 50  0001 C CNN
 	1    8400 3750
@@
 $EndComp
 $Comp
-L open-automation:R_10k R10
+L open-automation:R_10k R2
 U 1 1 59C83F25
 P 3450 3700
-F 0 "R10" V 3450 3700 50  0000 C CNN
+F 0 "R2" V 3450 3700 50  0000 C CNN
 F 1 "R_10k" H 3325 3850 50  0000 C CNN
-F 2 "Resistor_SMD:R_0603_1608Metric_Pad0.99x1.00mm_HandSolder" V 3380 3700 50  0001 C CNN
+F 2 "Resistor_SMD:R_0603_1608Metric_Pad1.05x0.95mm_HandSolder" V 3380 3700 50  0001 C CNN
 F 3 "https://www.digikey.com/product-detail/en/yageo/RC0603JR-0710KL/311-10KGRCT-ND/729647" V 3530 3700 50  0001 C CNN
 F 4 "RC0603JR-0710KL" V 3630 3800 60  0001 C CNN "Part Number"
@@
 $EndComp
 $Comp
-L open-automation:R_10k R9
+L open-automation:R_10k R1
 U 1 1 59C83F7C
 P 3350 3700
-F 0 "R9" V 3350 3700 50  0000 C CNN
+F 0 "R1" V 3350 3700 50  0000 C CNN
 F 1 "R_10k" H 3475 3850 50  0000 C CNN
-F 2 "Resistor_SMD:R_0603_1608Metric_Pad0.99x1.00mm_HandSolder" V 3280 3700 50  0001 C CNN
+F 2 "Resistor_SMD:R_0603_1608Metric_Pad1.05x0.95mm_HandSolder" V 3280 3700 50  0001 C CNN
 F 3 "https://www.digikey.com/product-detail/en/yageo/RC0603JR-0710KL/311-10KGRCT-ND/729647" V 3430 3700 50  0001 C CNN
 F 4 "RC0603JR-0710KL" V 3530 3800 60  0001 C CNN "Part Number"
@@
 3V3
 $Comp
-L open-automation:C_10uF C4
+L open-automation:C_10uF C1
 U 1 1 5A10664F
 P 2425 3775
-F 0 "C4" H 2450 3875 50  0000 L CNN
+F 0 "C1" H 2450 3875 50  0000 L CNN
 F 1 "C_10uF" H 2125 3675 50  0000 L CNN
-F 2 "Capacitor_SMD:C_0603_1608Metric_Pad0.99x1.00mm_HandSolder" H 2525 4075 50  0001 C CNN
+F 2 "Capacitor_SMD:C_0603_1608Metric_Pad1.05x0.95mm_HandSolder" H 2525 4075 50  0001 C CNN
 F 3 "https://www.digikey.com/product-detail/en/murata-electronics-north-america/GRM188R61A106ME69D/490-10475-1-ND/5026393" H 2425 3525 50  0001 C CNN
 F 4 "GRM188R61A106ME69D" H 2550 3975 60  0001 C CNN "Part Number"
@@
 	2625 3525 2825 3525
 $Comp
-L open-automation:GND #PWR?
+L open-automation:GND #PWR01
 U 1 1 5B3C970C
 P 2625 4025
-F 0 "#PWR?" H 2625 3775 50  0001 C CNN
+F 0 "#PWR01" H 2625 3775 50  0001 C CNN
 F 1 "GND" H 2630 3852 50  0000 C CNN
 F 2 "" H 2625 4025 50  0000 C CNN
@@
 $EndComp
 $Comp
-L open-automation:GND #PWR?
+L open-automation:GND #PWR02
 U 1 1 5B3CA255
 P 4825 2750
-F 0 "#PWR?" H 4825 2500 50  0001 C CNN
+F 0 "#PWR02" H 4825 2500 50  0001 C CNN
 F 1 "GND" H 4830 2577 50  0000 C CNN
 F 2 "" H 4825 2750 50  0000 C CNN
@@
 $EndComp
 $Comp
-L open-automation:GND #PWR?
+L open-automation:GND #PWR04
 U 1 1 5B3CAD4B
 P 8150 3500
-F 0 "#PWR?" H 8150 3250 50  0001 C CNN
+F 0 "#PWR04" H 8150 3250 50  0001 C CNN
 F 1 "GND" H 8155 3327 50  0000 C CNN
 F 2 "" H 8150 3500 50  0000 C CNN
@@
 $EndComp
 $Comp
-L open-automation:GND #PWR?
+L open-automation:GND #PWR05
 U 1 1 5B3CB673
 P 8750 3500
-F 0 "#PWR?" H 8750 3250 50  0001 C CNN
+F 0 "#PWR05" H 8750 3250 50  0001 C CNN
 F 1 "GND" H 8755 3327 50  0000 C CNN
 F 2 "" H 8750 3500 50  0000 C CNN
@@
 $EndComp
 $Comp
-L open-automation:GND #PWR?
+L open-automation:GND #PWR03
 U 1 1 5B3CC21F
 P 6600 4700
-F 0 "#PWR?" H 6600 4450 50  0001 C CNN
+F 0 "#PWR03" H 6600 4450 50  0001 C CNN
 F 1 "GND" V 6605 4572 50  0000 R CNN
 F 2 "" H 6600 4700 50  0000 C CNN
@@
 Text HLabel 8100 3750 0    50   Input ~ 0
 PROG
-Wire Wire Line
-	7550 1650 7100 1650
-Wire Wire Line
-	7550 1750 7100 1750
-Text HLabel 7100 1650 0    50   Input ~ 0
-SDA
-Text HLabel 7100 1750 0    50   Input ~ 0
-SCL
-Wire Wire Line
-	8350 2150 7925 2150
-Wire Wire Line
-	7225 1850 7225 1950
-$Comp
-L open-automation:GND #PWR?
-U 1 1 5B3E686F
-P 7225 1950
-F 0 "#PWR?" H 7225 1700 50  0001 C CNN
-F 1 "GND" H 7230 1777 50  0000 C CNN
-F 2 "" H 7225 1950 50  0000 C CNN
-F 3 "" H 7225 1950 50  0000 C CNN
-	1    7225 1950
-	1    0    0    -1
-$EndComp
-Wire Wire Line
-	7550 1850 7225 1850
-Wire Wire Line
-	7925 1850 7550 1850
-Connection ~ 7550 1850
-$Comp
-L open-automation:DAC U?
-U 1 1 5B3E2E45
-P 8050 1850
-F 0 "U?" H 7950 2405 50  0000 C CNN
-F 1 "DAC" H 7950 2314 50  0000 C CNN
-F 2 "Package_DFN_QFN:DFN-14-1EP_3x3mm_P0.4mm_EP1.78x2.35mm" H 7900 1850 50  0001 C CNN
-F 3 "https://www.digikey.com/product-detail/en/maxim-integrated/DS4424N/DS4424N-ND/2045475" H 7900 1850 50  0001 C CNN
-F 4 "DS4424N+" H 7950 2223 50  0000 C CNN "Part Number"
-	1    8050 1850
-	1    0    0    -1
-$EndComp
-Wire Wire Line
-	8350 1950 7925 1950
-Wire Wire Line
-	7925 1850 7925 1950
-Connection ~ 7925 1950
-Wire Wire Line
-	7925 1950 7925 2150
 Text Notes 7025 6950 0    197  ~ 0
 MICRO

Commit message: multifile update
Parts:
- removed J1: Conn_02x05_Odd_Even, Connector_PinHeader_2.54mm:PinHeader_2x05_P2.54mm_Vertical, symbol Connector_Generic:Conn_02x05_Odd_Even
- added J2: Conn_02x20_Top_Bottom, Connector_PinSocket_2.54mm:PinSocket_2x20_P2.54mm_Vertical, symbol Connector_Generic:Conn_02x20_Top_Bottom
- added J?: Conn_02x20_Odd_Even, symbol Connector_Generic:Conn_02x20_Odd_Even
- C2: Part Number CL10B105KA8VPNC -> CL10B105KP8NNNC
Connections:
- net labels added: MISO, MOSI, SCLK, USB_EN
- net labels removed: PANEL_SW, POWER_EN
- wire segments 42 -> 72

Commit message: traces complete
Parts:
- removed J2: Conn_02x20_Top_Bottom, Connector_PinSocket_2.54mm:PinSocket_2x20_P2.54mm_Vertical, symbol Connector_Generic:Conn_02x20_Top_Bottom
- J2: renamed from J?; footprint (none) -> Connector_PinSocket_2.54mm:PinSocket_2x20_P2.54mm_Vertical; Part Number (none) -> SFH11-PBPC-D20-ST-BK
Changed lines of the file:
@@
 Text Notes 7025 6950 0    197  ~ 0
 MICRO
-$Comp
-L Connector_Generic:Conn_02x20_Top_Bottom J2
-U 1 1 5B5DD319
-P 8675 3800
-F 0 "J2" H 8725 4917 50  0000 C CNN
-F 1 "Conn_02x20_Top_Bottom" H 8725 4826 50  0000 C CNN
-F 2 "Connector_PinSocket_2.54mm:PinSocket_2x20_P2.54mm_Vertical" H 8675 3800 50  0001 C CNN
-F 3 "~" H 8675 3800 50  0001 C CNN
-F 4 "SFH11-PBPC-D20-ST-BK" H 8675 3800 50  0001 C CNN "Part Number"
-	1    8675 3800
-	1    0    0    -1
-$EndComp
 Wire Wire Line
 	10000 2950 10100 2950
@@
 MOSI
 $Comp
-L Connector_Generic:Conn_02x20_Odd_Even J?
+L Connector_Generic:Conn_02x20_Odd_Even J2
 U 1 1 5B768BB7
 P 10300 3850
-F 0 "J?" H 10350 4967 50  0000 C CNN
+F 0 "J2" H 10350 4967 50  0000 C CNN
 F 1 "Conn_02x20_Odd_Even" H 10350 4876 50  0000 C CNN
-F 2 "" H 10300 3850 50  0001 C CNN
+F 2 "Connector_PinSocket_2.54mm:PinSocket_2x20_P2.54mm_Vertical" H 10300 3850 50  0001 C CNN
 F 3 "~" H 10300 3850 50  0001 C CNN
+F 4 "SFH11-PBPC-D20-ST-BK" H 10300 3850 50  0001 C CNN "Part Number"
 	1    10300 3850
 	1    0    0    -1

Commit message: parts
Parts:
- C1: Part Number GRM188R61A106ME69D -> GRM188C80G106ME47D
- C2: Part Number CL10B105KP8NNNC -> CL10B105MO8NNWC
- R1, R2, R3: Part Number RC0603JR-0710KL -> RR0816P-103-D
Changed lines of the file:
@@
 F 1 "C_1uF" H 2575 3675 50  0000 L CNN
 F 2 "Capacitor_SMD:C_0603_1608Metric_Pad1.05x0.95mm_HandSolder" H 2925 4075 50  0001 C CNN
-F 3 "https://www.digikey.com/product-detail/en/yageo/CC0603ZRY5V7BB105/311-1372-1-ND/2103156" H 2825 3525 50  0001 C CNN
-F 4 "CL10B105KP8NNNC" H 2950 3975 60  0001 C CNN "Part Number"
+F 3 "https://www.digikey.com/product-detail/en/samsung-electro-mechanics/CL10B105MO8NNWC/1276-6524-1-ND/5961383" H 2825 3525 50  0001 C CNN
+F 4 "CL10B105MO8NNWC" H 2950 3975 60  0001 C CNN "Part Number"
 	1    2825 3775
 	1    0    0    -1
@@
 F 1 "R_10k" V 6325 4700 50  0000 C CNN
 F 2 "Resistor_SMD:R_0603_1608Metric_Pad1.05x0.95mm_HandSolder" V 6330 4700 50  0001 C CNN
-F 3 "https://www.digikey.com/product-detail/en/yageo/RC0603JR-0710KL/311-10KGRCT-ND/729647" V 6480 4700 50  0001 C CNN
-F 4 "RC0603JR-0710KL" V 6580 4800 60  0001 C CNN "Part Number"
+F 3 "https://www.digikey.com/product-detail/en/susumu/RR0816P-103-D/RR08P10.0KDCT-ND/432748" V 6480 4700 50  0001 C CNN
+F 4 "RR0816P-103-D" V 6580 4800 60  0001 C CNN "Part Number"
 	1    6400 4700
 	0    1    1    0
@@
 F 1 "R_10k" H 3325 3850 50  0000 C CNN
 F 2 "Resistor_SMD:R_0603_1608Metric_Pad1.05x0.95mm_HandSolder" V 3380 3700 50  0001 C CNN
-F 3 "https://www.digikey.com/product-detail/en/yageo/RC0603JR-0710KL/311-10KGRCT-ND/729647" V 3530 3700 50  0001 C CNN
-F 4 "RC0603JR-0710KL" V 3630 3800 60  0001 C CNN "Part Number"
+F 3 "https://www.digikey.com/product-detail/en/susumu/RR0816P-103-D/RR08P10.0KDCT-ND/432748" V 3530 3700 50  0001 C CNN
+F 4 "RR0816P-103-D" V 3630 3800 60  0001 C CNN "Part Number"
 	1    3450 3700
 	-1   0    0    1
@@
 F 1 "R_10k" H 3475 3850 50  0000 C CNN
 F 2 "Resistor_SMD:R_0603_1608Metric_Pad1.05x0.95mm_HandSolder" V 3280 3700 50  0001 C CNN
-F 3 "https://www.digikey.com/product-detail/en/yageo/RC0603JR-0710KL/311-10KGRCT-ND/729647" V 3430 3700 50  0001 C CNN
-F 4 "RC0603JR-0710KL" V 3530 3800 60  0001 C CNN "Part Number"
+F 3 "https://www.digikey.com/product-detail/en/susumu/RR0816P-103-D/RR08P10.0KDCT-ND/432748" V 3430 3700 50  0001 C CNN
+F 4 "RR0816P-103-D" V 3530 3800 60  0001 C CNN "Part Number"
 	1    3350 3700
 	-1   0    0    1
@@
 F 1 "C_10uF" H 2125 3675 50  0000 L CNN
 F 2 "Capacitor_SMD:C_0603_1608Metric_Pad1.05x0.95mm_HandSolder" H 2525 4075 50  0001 C CNN
-F 3 "https://www.digikey.com/product-detail/en/murata-electronics-north-america/GRM188R61A106ME69D/490-10475-1-ND/5026393" H 2425 3525 50  0001 C CNN
-F 4 "GRM188R61A106ME69D" H 2550 3975 60  0001 C CNN "Part Number"
+F 3 "https://www.digikey.com/product-detail/en/murata-electronics-north-america/GRM188C80G106ME47D/490-10470-1-ND/5026387" H 2425 3525 50  0001 C CNN
+F 4 "GRM188C80G106ME47D" H 2550 3975 60  0001 C CNN "Part Number"
 	1    2425 3775
 	1    0    0    -1

Commit message: traces complete
Connections:
- net labels added: REG1_EN, REG2_EN, REG3_EN
- wire segments 72 -> 75
Changed lines of the file:
@@
 $Descr A4 11693 8268
 encoding utf-8
-Sheet 2 5
+Sheet 5 5
 Title ""
 Date ""
@@
 Text Label 10000 4050 2    50   ~ 0
 SCLK
+Wire Wire Line
+	4875 3700 4750 3700
+Text HLabel 4750 3600 0    50   Input ~ 0
+REG1_EN
+Text HLabel 4750 3700 0    50   Input ~ 0
+REG2_EN
+Wire Wire Line
+	4875 3600 4750 3600
+Wire Wire Line
+	4875 3400 4750 3400
+Text HLabel 4750 3400 0    50   Input ~ 0
+REG3_EN
 $EndSCHEMATC

Commit message: rewire
Connections:
- net labels added: MAIN_CURRENT_SENSE
- wire segments 75 -> 76
Changed lines of the file:
@@
 SCLK
 Wire Wire Line
-	4875 3700 4750 3700
+	4875 3500 4750 3500
 Text HLabel 4750 3600 0    50   Input ~ 0
 REG1_EN
-Text HLabel 4750 3700 0    50   Input ~ 0
+Text HLabel 4750 3500 0    50   Input ~ 0
 REG2_EN
 Wire Wire Line
@@
 Text HLabel 4750 3400 0    50   Input ~ 0
 REG3_EN
+Wire Wire Line
+	4875 3700 4750 3700
+Text GLabel 4750 3700 0    50   Input ~ 0
+MAIN_CURRENT_SENSE
 $EndSCHEMATC
