File: hardware/switches.sch (KiCad schematic (older format))
At the start: 11 parts, among them P5 USB_A_2, Q2 Q_NMOS_GSD, Q3 Q_PMOS_GSD, U10 touchpad, U4 housing-mounts

Commit message: update
Parts:
- removed R16: 1K, Resistors_SMD:R_0603_HandSoldering, symbol R
- added PROG?: SW_PUSH, Buttons_Switches_SMD:SW_SPST_KMR2, symbol SW_PUSH
Connections:
- net 5V: no longer D2.2 (A)
- net IO0: now also Q2.3 (D)
- new net 3V3: D2.2 (A)
Changed lines of the file:
@@
 EESchema Schematic File Version 2
-LIBS:5v-smart-solar-regulator-rescue
 LIBS:power
 LIBS:device
@@
 LIBS:contrib
 LIBS:valves
-LIBS:open-automation
 LIBS:5v-smart-solar-regulator-cache
 EELAYER 25 0
@@
 $EndComp
 $Comp
-L R R16
-U 1 1 59092D22
-P 5200 4450
-F 0 "R16" V 5280 4450 50  0000 C CNN
-F 1 "1K" V 5200 4450 50  0000 C CNN
-F 2 "Resistors_SMD:R_0603_HandSoldering" V 5130 4450 50  0001 C CNN
-F 3 "http://www.digikey.com/en/resources/datasheets/yageo/rc-series-l-suffix-datasheet" H 5200 4450 50  0001 C CNN
-F 4 "RC0603JR-071KL" V 5200 4450 60  0001 C CNN "Part Number"
-	1    5200 4450
-	0    1    1    0
-$EndComp
-$Comp
 L C C5
 U 1 1 59092D23
@@
 	4900 2400 4900 2550
 Wire Wire Line
-	5350 4450 5500 4450
+	4650 4450 5500 4450
 Wire Wire Line
 	4900 4100 4900 4600
-Wire Wire Line
-	4650 4450 5050 4450
 Wire Wire Line
 	4200 4100 4450 4100
@@
 $EndComp
 Text GLabel 4900 2400 1    60   Input ~ 0
-5V
+3V3
 $Comp
 L USB_A_2 P5
@@
 	1    0    0    -1
 $EndComp
+$Comp
+L SW_PUSH PROG?
+U 1 1 59BEC83F
+P 6700 3550
+F 0 "PROG?" H 6850 3660 50  0000 C CNN
+F 1 "SW_PUSH" H 6700 3470 50  0000 C CNN
+F 2 "Buttons_Switches_SMD:SW_SPST_KMR2" H 6700 3550 50  0001 C CNN
+F 3 "http://www.mouser.com/ds/2/60/KMR2_9aug12-25127.pdf" H 6700 3550 50  0001 C CNN
+F 4 "KMR211NG LFS" H 6700 3550 60  0001 C CNN "Part Number"
+	1    6700 3550
+	0    1    1    0
+$EndComp
 $EndSCHEMATC
