File: hardware/switches.sch (KiCad schematic (older format))
At the start: 11 parts, among them P5 USB_A_2, Q2 Q_NMOS_GSD, Q3 Q_PMOS_GSD, U10 touchpad, U4 housing-mounts

Commit message: update
Parts:
- removed PROG?: SW_PUSH, Buttons_Switches_SMD:SW_SPST_KMR2, symbol SW_PUSH
- added FACTORY1: SW_PUSH, Buttons_Switches_SMD:SW_SPST_KMR2, symbol SW_PUSH
- U10: footprint footprints:touch-pad -> open-automation:touch-pad
- U4: footprint footprints:enclosure-25x38 -> open-automation:enclosure-25x38
Connections:
- net 5V is gone; now on net V_USB: P5.2 (VBUS)
- net GND: now also FACTORY1.2
- net 3V3 renamed V_USB
- net IO0 renamed PROG
- net IO14 renamed FACTORY
- net FACTORY: now also FACTORY1.1
Other:
- moved on the sheet: C5, D2, P5, PROG1, Q2, Q3, R14, R15, U10, U4

Commit message: update
Connections:
- net V_USB: no longer D2.2 (A)
- new net 3V3: D2.2 (A)
Changed lines of the file:
@@
 $EndComp
 Text GLabel 5525 2625 1    60   Input ~ 0
-V_USB
+3V3
 $Comp
 L USB_A_2 P5

Commit message: update
Parts:
- removed C5: 4.7uF, Capacitors_SMD:C_0603_HandSoldering, symbol C
- removed Q2: Q_NMOS_GSD, TO_SOT_Packages_SMD:SOT-23, symbol Q_NMOS_GSD
- removed Q3: Q_PMOS_GSD, TO_SOT_Packages_SMD:SOT-23, symbol Q_PMOS_GSD
- removed R14, R15: 1K, Resistors_SMD:R_0603_HandSoldering, symbol R
- added D3, D5: LED, LEDs:LED_0603, symbol LED
- added R2, R3, R4: R_10k, Resistors_SMD:R_0603_HandSoldering, symbol R_10k
- added REBOOT1: SW_PUSH, Buttons_Switches_SMD:SW_SPST_KMR2, symbol SW_PUSH
Connections:
- net 3V3: now also D3.2 (A), D5.2 (A)
- net EN: now also R3.2, REBOOT1.1; no longer PROG1.1
- net FACTORY: now also R2.2
- net GND: now also REBOOT1.2
- net PROG: now also PROG1.1, R4.2
- net at D2.1 (K): now also R2.1
- net TXD: now reaches P5.3 (D-)
- net TXD: now also P5.5 (D-)
- net RXD: now reaches P5.4 (D+)
- net RXD: now also P5.6 (D+)
- new net: D3.1 (K), R3.1
- new net: D5.1 (K), R4.1
Other:
- moved on the sheet: D2, FACTORY1, P5, U10, U4

Commit message: update
Parts:
- D2, D3, D5: footprint LEDs:LED_0603 -> LEDs:LED_0603_HandSoldering
Changed lines of the file:
@@
 F 0 "D2" V 3700 3225 50  0000 C CNN
 F 1 "LED" V 3825 3050 50  0000 C CNN
-F 2 "LEDs:LED_0603" H 3725 3125 50  0001 C CNN
+F 2 "LEDs:LED_0603_HandSoldering" H 3725 3125 50  0001 C CNN
 F 3 "http://www.osram-os.com/Graphics/XPic9/00128792_0.pdf" H 3725 3125 50  0001 C CNN
 F 4 "475-2512-2-ND" H 3725 3125 60  0001 C CNN "Part Number"
@@
 F 0 "D3" V 4650 3225 50  0000 C CNN
 F 1 "LED" V 4775 3050 50  0000 C CNN
-F 2 "LEDs:LED_0603" H 4675 3125 50  0001 C CNN
+F 2 "LEDs:LED_0603_HandSoldering" H 4675 3125 50  0001 C CNN
 F 3 "http://www.osram-os.com/Graphics/XPic9/00128792_0.pdf" H 4675 3125 50  0001 C CNN
 F 4 "475-2512-2-ND" H 4675 3125 60  0001 C CNN "Part Number"
@@
 F 0 "D5" V 5425 3225 50  0000 C CNN
 F 1 "LED" V 5550 3050 50  0000 C CNN
-F 2 "LEDs:LED_0603" H 5450 3125 50  0001 C CNN
+F 2 "LEDs:LED_0603_HandSoldering" H 5450 3125 50  0001 C CNN
 F 3 "http://www.osram-os.com/Graphics/XPic9/00128792_0.pdf" H 5450 3125 50  0001 C CNN
 F 4 "475-2512-2-ND" H 5450 3125 60  0001 C CNN "Part Number"

Commit message: regulator ya know
Parts:
- removed D2, D3, D5: LED, LEDs:LED_0603_HandSoldering, symbol LED
- removed FACTORY1, PROG1, REBOOT1: SW_PUSH, Buttons_Switches_SMD:SW_SPST_KMR2, symbol SW_PUSH
- removed R2, R3, R4: R_10k, Resistors_SMD:R_0603_HandSoldering, symbol R_10k
- added D2, D3, D5: LED-0603-R, LED_SMD:LED_0603_1608Metric_Pad0.82x1.00mm_HandSolder, symbol open-automation:LED-0603-R
- added R2, R3, R4: R_10k, Resistor_SMD:R_0603_1608Metric_Pad0.99x1.00mm_HandSolder, symbol open-automation:R_10k
- added SW? (x3): SW_PUSH, symbol open-automation:SW_PUSH
- P5: symbol USB_A_2 -> open-automation:USB_A_2
- U10: symbol touchpad -> open-automation:touch-pad
- U4: symbol housing-mounts -> open-automation:housing-mounts
Connections:
- wire segments 25 -> 29

Commit message: additional components
Other:
- note added: "SWITCHES"
Changed lines of the file:
@@
 	1    0    0    -1
 $EndComp
+Text Notes 7000 6950 0    197  ~ 0
+SWITCHES
 $EndSCHEMATC

Commit message: layout complete bitches
Parts:
- removed SW? (x2): SW_PUSH, symbol open-automation:SW_PUSH
- added BATTERY1, PANEL1: CONN_01X02, open-automation:XT60, symbol Connector_Generic:Conn_01x02
- added SW1, SW2: SW_PUSH, Button_Switch_SMD:SW_SPST_KMR2, symbol open-automation:SW_PUSH
- D1: renamed from D2; footprint LED_SMD:LED_0603_1608Metric_Pad0.82x1.00mm_HandSolder -> LED_SMD:LED_0603_1608Metric_Pad0.88x0.95mm_HandSolder
- D2: renamed from D3; footprint LED_SMD:LED_0603_1608Metric_Pad0.82x1.00mm_HandSolder -> LED_SMD:LED_0603_1608Metric_Pad0.88x0.95mm_HandSolder
- D3: renamed from D5; footprint LED_SMD:LED_0603_1608Metric_Pad0.82x1.00mm_HandSolder -> LED_SMD:LED_0603_1608Metric_Pad0.88x0.95mm_HandSolder
- R4: renamed from R2; footprint Resistor_SMD:R_0603_1608Metric_Pad0.99x1.00mm_HandSolder -> Resistor_SMD:R_0603_1608Metric_Pad1.05x0.95mm_HandSolder
- R5: renamed from R3; footprint Resistor_SMD:R_0603_1608Metric_Pad0.99x1.00mm_HandSolder -> Resistor_SMD:R_0603_1608Metric_Pad1.05x0.95mm_HandSolder
- R6: renamed from R4; footprint Resistor_SMD:R_0603_1608Metric_Pad0.99x1.00mm_HandSolder -> Resistor_SMD:R_0603_1608Metric_Pad1.05x0.95mm_HandSolder
- SW3: renamed from SW?; footprint (none) -> Button_Switch_SMD:SW_SPST_KMR2; Part Number (none) -> KMR211NG LFS
- renumbered P5 to P1, U4 to U2, U10 to U3
Connections:
- net labels added: BATTERY, V_PANEL
- wire segments 29 -> 35
Changed lines of the file:
@@
 	7975 4600 8075 4600
 $Comp
-L open-automation:touch-pad U10
+L open-automation:touch-pad U3
 U 1 1 590F8D3B
 P 8475 4600
-F 0 "U10" H 8625 4400 60  0000 C CNN
+F 0 "U3" H 8625 4400 60  0000 C CNN
 F 1 "touchpad" H 8475 4800 60  0000 C CNN
 F 2 "open-automation:touch-pad" H 8475 4600 60  0001 C CNN
@@
 3V3
 $Comp
-L open-automation:USB_A_2 P5
+L open-automation:USB_A_2 P1
 U 1 1 59693837
 P 8350 2800
-F 0 "P5" H 8600 2600 50  0000 C CNN
+F 0 "P1" H 8600 2600 50  0000 C CNN
 F 1 "USB_A_2" H 8300 3000 50  0000 C CNN
 F 2 "open-automation:USB_A_2" V 8300 2700 50  0001 C CNN
@@
 	7900 3200 7850 3200
 $Comp
-L open-automation:housing-mounts U4
+L open-automation:housing-mounts U2
 U 1 1 5978A2A6
 P 8425 4025
-F 0 "U4" H 8575 3925 60  0000 C CNN
+F 0 "U2" H 8575 3925 60  0000 C CNN
 F 1 "housing-mounts" H 8425 4225 60  0000 C CNN
 F 2 "open-automation:enclosure-25x38" H 8425 4075 60  0001 C CNN
@@
 PROG
 $Comp
-L open-automation:LED-0603-R D5
+L open-automation:LED-0603-R D3
 U 1 1 5B3AD696
 P 5450 3125
-F 0 "D5" V 5488 3008 50  0000 R CNN
+F 0 "D3" V 5488 3008 50  0000 R CNN
 F 1 "LED-0603-R" V 5397 3008 50  0000 R CNN
-F 2 "LED_SMD:LED_0603_1608Metric_Pad0.82x1.00mm_HandSolder" H 5350 3125 50  0001 C CNN
+F 2 "LED_SMD:LED_0603_1608Metric_Pad0.88x0.95mm_HandSolder" H 5350 3125 50  0001 C CNN
 F 3 "https://www.digikey.com/products/en?keywords=475-2512-2-ND" H 5450 3225 50  0001 C CNN
 F 4 "LS Q976-NR-1" H 5550 3325 50  0001 C CNN "Part Number"
@@
 $EndComp
 $Comp
-L open-automation:LED-0603-R D3
+L open-automation:LED-0603-R D2
 U 1 1 5B3AD76A
 P 4675 3125
-F 0 "D3" V 4713 3008 50  0000 R CNN
+F 0 "D2" V 4713 3008 50  0000 R CNN
 F 1 "LED-0603-R" V 4622 3008 50  0000 R CNN
-F 2 "LED_SMD:LED_0603_1608Metric_Pad0.82x1.00mm_HandSolder" H 4575 3125 50  0001 C CNN
+F 2 "LED_SMD:LED_0603_1608Metric_Pad0.88x0.95mm_HandSolder" H 4575 3125 50  0001 C CNN
 F 3 "https://www.digikey.com/products/en?keywords=475-2512-2-ND" H 4675 3225 50  0001 C CNN
 F 4 "LS Q976-NR-1" H 4775 3325 50  0001 C CNN "Part Number"
@@
 $EndComp
 $Comp
-L open-automation:LED-0603-R D2
+L open-automation:LED-0603-R D1
 U 1 1 5B3AD860
 P 3725 3125
-F 0 "D2" V 3763 3008 50  0000 R CNN
+F 0 "D1" V 3763 3008 50  0000 R CNN
 F 1 "LED-0603-R" V 3672 3008 50  0000 R CNN
-F 2 "LED_SMD:LED_0603_1608Metric_Pad0.82x1.00mm_HandSolder" H 3625 3125 50  0001 C CNN
+F 2 "LED_SMD:LED_0603_1608Metric_Pad0.88x0.95mm_HandSolder" H 3625 3125 50  0001 C CNN
 F 3 "https://www.digikey.com/products/en?keywords=475-2512-2-ND" H 3725 3225 50  0001 C CNN
 F 4 "LS Q976-NR-1" H 3825 3325 50  0001 C CNN "Part Number"
@@
 $EndComp
 $Comp
-L open-automation:R_10k R4
+L open-automation:R_10k R6
 U 1 1 5B3ADCC0
 P 5450 3475
-F 0 "R4" H 5520 3521 50  0000 L CNN
+F 0 "R6" H 5520 3521 50  0000 L CNN
 F 1 "R_10k" H 5520 3430 50  0000 L CNN
-F 2 "Resistor_SMD:R_0603_1608Metric_Pad0.99x1.00mm_HandSolder" V 5380 3475 50  0001 C CNN
+F 2 "Resistor_SMD:R_0603_1608Metric_Pad1.05x0.95mm_HandSolder" V 5380 3475 50  0001 C CNN
 F 3 "https://www.digikey.com/product-detail/en/yageo/RC0603JR-0710KL/311-10KGRCT-ND/729647" V 5530 3475 50  0001 C CNN
 F 4 "RC0603JR-0710KL" V 5630 3575 60  0001 C CNN "Part Number"
@@
 $EndComp
 $Comp
-L open-automation:R_10k R2
+L open-automation:R_10k R4
 U 1 1 5B3ADD56
 P 3725 3475
-F 0 "R2" H 3795 3521 50  0000 L CNN
+F 0 "R4" H 3795 3521 50  0000 L CNN
 F 1 "R_10k" H 3795 3430 50  0000 L CNN
-F 2 "Resistor_SMD:R_0603_1608Metric_Pad0.99x1.00mm_HandSolder" V 3655 3475 50  0001 C CNN
+F 2 "Resistor_SMD:R_0603_1608Metric_Pad1.05x0.95mm_HandSolder" V 3655 3475 50  0001 C CNN
 F 3 "https://www.digikey.com/product-detail/en/yageo/RC0603JR-0710KL/311-10KGRCT-ND/729647" V 3805 3475 50  0001 C CNN
 F 4 "RC0603JR-0710KL" V 3905 3575 60  0001 C CNN "Part Number"
@@
 $EndComp
 $Comp
-L open-automation:R_10k R3
+L open-automation:R_10k R5
 U 1 1 5B3ADDBF
 P 4675 3475
-F 0 "R3" H 4745 3521 50  0000 L CNN
+F 0 "R5" H 4745 3521 50  0000 L CNN
 F 1 "R_10k" H 4745 3430 50  0000 L CNN
-F 2 "Resistor_SMD:R_0603_1608Metric_Pad0.99x1.00mm_HandSolder" V 4605 3475 50  0001 C CNN
+F 2 "Resistor_SMD:R_0603_1608Metric_Pad1.05x0.95mm_HandSolder" V 4605 3475 50  0001 C CNN
 F 3 "https://www.digikey.com/product-detail/en/yageo/RC0603JR-0710KL/311-10KGRCT-ND/729647" V 4755 3475 50  0001 C CNN
 F 4 "RC0603JR-0710KL" V 4855 3575 60  0001 C CNN "Part Number"
@@
 $EndComp
 $Comp
-L open-automation:SW_PUSH SW?
-U 1 1 5B3AE0CC
-P 3725 3975
-F 0 "SW?" V 3679 4093 50  0000 L CNN
-F 1 "SW_PUSH" V 3770 4093 50  0000 L CNN
-F 2 "" H 3725 3975 50  0000 C CNN
-F 3 "" H 3725 3975 50  0000 C CNN
-	1    3725 3975
-	0    1    1    0
-$EndComp
-$Comp
-L open-automation:SW_PUSH SW?
-U 1 1 5B3AE227
-P 4675 3975
-F 0 "SW?" V 4629 4093 50  0000 L CNN
-F 1 "SW_PUSH" V 4720 4093 50  0000 L CNN
-F 2 "" H 4675 3975 50  0000 C CNN
-F 3 "" H 4675 3975 50  0000 C CNN
-	1    4675 3975
-	0    1    1    0
-$EndComp
-$Comp
-L open-automation:SW_PUSH SW?
+L open-automation:SW_PUSH SW3
 U 1 1 5B3AE2A4
 P 5450 3975
-F 0 "SW?" V 5404 4093 50  0000 L CNN
+F 0 "SW3" V 5404 4093 50  0000 L CNN
 F 1 "SW_PUSH" V 5495 4093 50  0000 L CNN
-F 2 "" H 5450 3975 50  0000 C CNN
-F 3 "" H 5450 3975 50  0000 C CNN
+F 2 "Button_Switch_SMD:SW_SPST_KMR2" H 5450 3975 50  0001 C CNN
+F 3 "http://www.mouser.com/ds/2/60/KMR2_9aug12-25127.pdf" H 5450 3975 50  0001 C CNN
+F 4 "KMR211NG LFS" V 5450 3975 50  0001 C CNN "Part Number"
 	1    5450 3975
 	0    1    1    0
 $EndComp
 $Comp
-L open-automation:GND #PWR?
+L open-automation:GND #PWR06
 U 1 1 5B3AE587
 P 3725 4350
-F 0 "#PWR?" H 3725 4100 50  0001 C CNN
+F 0 "#PWR06" H 3725 4100 50  0001 C CNN
 F 1 "GND" H 3730 4177 50  0000 C CNN
 F 2 "" H 3725 4350 50  0000 C CNN
@@
 $EndComp
 $Comp
-L open-automation:GND #PWR?
+L open-automation:GND #PWR07
 U 1 1 5B3AE5CD
 P 4675 4350
-F 0 "#PWR?" H 4675 4100 50  0001 C CNN
+F 0 "#PWR07" H 4675 4100 50  0001 C CNN
 F 1 "GND" H 4680 4177 50  0000 C CNN
 F 2 "" H 4675 4350 50  0000 C CNN
@@
 $EndComp
 $Comp
-L open-automation:GND #PWR?
+L open-automation:GND #PWR08
 U 1 1 5B3AE613
 P 5450 4350
-F 0 "#PWR?" H 5450 4100 50  0001 C CNN
+F 0 "#PWR08" H 5450 4100 50  0001 C CNN
 F 1 "GND" H 5455 4177 50  0000 C CNN
 F 2 "" H 5450 4350 50  0000 C CNN
@@
 FACTORY
 $Comp
-L open-automation:GND #PWR?
+L open-automation:GND #PWR011
 U 1 1 5B3AECFF
 P 8500 3200
-F 0 "#PWR?" H 8500 2950 50  0001 C CNN
+F 0 "#PWR011" H 8500 2950 50  0001 C CNN
 F 1 "GND" H 8505 3027 50  0000 C CNN
 F 2 "" H 8500 3200 50  0000 C CNN
@@
 Text Notes 7000 6950 0    197  ~ 0
 SWITCHES
+$Comp
+L Connector_Generic:Conn_01x02 BATTERY?
+U 1 1 5B7A43D7
+P 8400 5250
+AR Path="/5936D89B/5B7A43D7" Ref="BATTERY?"  Part="1"
+AR Path="/5936D8F6/5B7A43D7" Ref="BATTERY1"  Part="1"
+F 0 "BATTERY1" H 8478 5291 50  0000 L CNN
+F 1 "CONN_01X02" H 8478 5200 50  0000 L CNN
+F 2 "open-automation:XT60" H 8400 5250 50  0001 C CNN
+F 3 "https://www.digikey.com/product-detail/en/phoenix-contact/1934861/277-1607-ND/568644" H 8400 5250 50  0001 C CNN
+	1    8400 5250
+	1    0    0    -1
+$EndComp
+Wire Wire Line
+	8150 5400 8150 5350
+Wire Wire Line
+	8150 5350 8200 5350
+Wire Wire Line
+	8100 5250 8200 5250
+$Comp
+L Connector_Generic:Conn_01x02 PANEL?
+U 1 1 5B7A43E1
+P 8425 5750
+AR Path="/5936D89B/5B7A43E1" Ref="PANEL?"  Part="1"
+AR Path="/5936D8F6/5B7A43E1" Ref="PANEL1"  Part="1"
+F 0 "PANEL1" H 8503 5791 50  0000 L CNN
+F 1 "CONN_01X02" H 8503 5700 50  0000 L CNN
+F 2 "open-automation:XT60" H 8425 5750 50  0001 C CNN
+F 3 "https://www.digikey.com/product-detail/en/phoenix-contact/1934861/277-1607-ND/568644" H 8425 5750 50  0001 C CNN
+	1    8425 5750
+	1    0    0    -1
+$EndComp
+Wire Wire Line
+	8175 5900 8175 5850
+Wire Wire Line
+	8175 5850 8225 5850
+Wire Wire Line
+	8125 5750 8225 5750
+$Comp
+L open-automation:GND #PWR?
+U 1 1 5B7A43EB
+P 8150 5400
+AR Path="/5936D89B/5B7A43EB" Ref="#PWR?"  Part="1"
+AR Path="/5936D8F6/5B7A43EB" Ref="#PWR09"  Part="1"
+F 0 "#PWR09" H 8150 5150 50  0001 C CNN
+F 1 "GND" H 8155 5227 50  0000 C CNN
+F 2 "" H 8150 5400 50  0000 C CNN
+F 3 "" H 8150 5400 50  0000 C CNN
+	1    8150 5400
+	1    0    0    -1
+$EndComp
+$Comp
+L open-automation:GND #PWR?
+U 1 1 5B7A43F1
+P 8175 5900
+AR Path="/5936D89B/5B7A43F1" Ref="#PWR?"  Part="1"
+AR Path="/5936D8F6/5B7A43F1" Ref="#PWR010"  Part="1"
+F 0 "#PWR010" H 8175 5650 50  0001 C CNN
+F 1 "GND" H 8180 5727 50  0000 C CNN
+F 2 "" H 8175 5900 50  0000 C CNN
+F 3 "" H 8175 5900 50  0000 C CNN
+	1    8175 5900
+	1    0    0    -1
+$EndComp
+Text HLabel 8100 5250 0    50   Input ~ 0
+BATTERY
+Text HLabel 8125 5750 0    50   Input ~ 0
+V_PANEL
+$Comp
+L open-automation:SW_PUSH SW1
+U 1 1 5B7A977E
+P 3725 3975
+F 0 "SW1" V 3679 4093 50  0000 L CNN
+F 1 "SW_PUSH" V 3770 4093 50  0000 L CNN
+F 2 "Button_Switch_SMD:SW_SPST_KMR2" H 3725 3975 50  0001 C CNN
+F 3 "http://www.mouser.com/ds/2/60/KMR2_9aug12-25127.pdf" H 3725 3975 50  0001 C CNN
+F 4 "KMR211NG LFS" V 3725 3975 50  0001 C CNN "Part Number"
+	1    3725 3975
+	0    1    1    0
+$EndComp
+$Comp
+L open-automation:SW_PUSH SW2
+U 1 1 5B7A9D32
+P 4675 3975
+F 0 "SW2" V 4629 4093 50  0000 L CNN
+F 1 "SW_PUSH" V 4720 4093 50  0000 L CNN
+F 2 "Button_Switch_SMD:SW_SPST_KMR2" H 4675 3975 50  0001 C CNN
+F 3 "http://www.mouser.com/ds/2/60/KMR2_9aug12-25127.pdf" H 4675 3975 50  0001 C CNN
+F 4 "KMR211NG LFS" V 4675 3975 50  0001 C CNN "Part Number"
+	1    4675 3975
+	0    1    1    0
+$EndComp
 $EndSCHEMATC
