File: hardware/thermometer.sch (KiCad schematic (older format))
At the start: 2 parts, among them P4 CONN_01X04

Commit message: update
Parts:
- P4: footprint Pin_Headers:Pin_Header_Straight_1x04_Pitch2.54mm -> Pin_Headers:Pin_Header_Angled_1x04_Pitch2.54mm
Connections:
- net 5v renamed 5V
Changed lines of the file:
@@
 LIBS:contrib
 LIBS:valves
-LIBS:5v-solar-regulator-cache
-EELAYER 26 0
+LIBS:open-automation
+LIBS:5v-smart-solar-regulator-cache
+EELAYER 25 0
 EELAYER END
 $Descr A4 11693 8268
@@
 F 0 "P4" H 6150 3100 50  0000 C CNN
 F 1 "CONN_01X04" V 6250 2850 50  0000 C CNN
-F 2 "Pin_Headers:Pin_Header_Straight_1x04_Pitch2.54mm" H 6150 2850 50  0001 C CNN
+F 2 "Pin_Headers:Pin_Header_Angled_1x04_Pitch2.54mm" H 6150 2850 50  0001 C CNN
 F 3 "" H 6150 2850 50  0000 C CNN
 	1    6150 2850
@@
 $EndComp
 $Comp
-L GND #PWR11
+L GND #PWR011
 U 1 1 5962DDD8
 P 5900 3050
-F 0 "#PWR11" H 5900 2800 50  0001 C CNN
+F 0 "#PWR011" H 5900 2800 50  0001 C CNN
 F 1 "GND" H 5900 2900 50  0000 C CNN
 F 2 "" H 5900 3050 50  0000 C CNN
@@
 $EndComp
 Text GLabel 5900 2650 1    60   Input ~ 0
-5v
-Wire Wire Line
-	5900 3050 5900 3000
-Wire Wire Line
-	5900 3000 5950 3000
-Wire Wire Line
-	5900 2650 5900 2700
-Wire Wire Line
-	5750 2700 5950 2700
+5V
 $Comp
 L R R25
@@
 	0    -1   -1   0
 $EndComp
+Text Label 5550 2300 0    60   ~ 0
+humidy_and_temperature
+Wire Wire Line
+	5900 2650 5900 2700
+Wire Wire Line
+	5750 2700 5950 2700
 Wire Wire Line
 	5400 2800 5950 2800
@@
 Connection ~ 5900 2700
 Connection ~ 5450 2800
-Text Label 5550 2300 0    60   ~ 0
-humidy_and_temperature
+Wire Wire Line
+	5900 3000 5950 3000
+Wire Wire Line
+	5900 3050 5900 3000
 $EndSCHEMATC
