File: hardware/smart-regulator.kicad_pcb (KiCad board)
At the start: 2 copper layers, 82.5 x 48.6 mm, 45 parts, among them J1 Conn_02x05_Odd_Even, P5 USB_A_2, Q1 Q_NMOS_GSD_PSMN038-100YLX, Q2 Q_NMOS_GSD, Q3 Q_PMOS_GSD, U1 ESP-WROOM-32, U10 touchpad, U11 SPX1117M3-L-3-3/TR, U2 Power-Monitor-INA219, U3 LM2576, U4 housing-mounts, U5 Power-Monitor-INA219, U6 SI7020-A20, U7 OPT3001

Commit message: update
Connections:
- R10 pad 2: GND -> 3V3
- R9 pad 2: GND -> 3V3
Routing:
- net 3V3: track 113.4 -> 134.8 mm, vias 8 -> 9
- net SCL: track 82.2 -> 82.7 mm
Changed lines of the file:
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@@
   (general
     (links 122)
-    (no_connects 0)
-    (area 93.142999 77.533999 175.743001 126.284001)
+    (no_connects 4)
+    (area 82.795 63.317618 184.875001 150.475428)
     (thickness 1.6)
     (drawings 21)
-    (tracks 460)
+    (tracks 471)
     (zones 0)
     (modules 45)
@@
       (net 38 SDA))
     (pad 2 smd rect (at 1.1 0) (size 1.2 0.9) (layers F.Cu F.Paste F.Mask)
-      (net 1 GND))
+      (net 18 3V3))
     (model ${KISYS3DMOD}/Resistors_SMD.3dshapes/R_0603.wrl
       (at (xyz 0 0 0))
@@
       (net 37 SCL))
     (pad 2 smd rect (at 1.1 0) (size 1.2 0.9) (layers F.Cu F.Paste F.Mask)
-      (net 1 GND))
+      (net 18 3V3))
     (model ${KISYS3DMOD}/Resistors_SMD.3dshapes/R_0603.wrl
       (at (xyz 0 0 0))
@@
   (gr_circle (center 122.059 82.337) (end 124.059 82.337) (layer Dwgs.User) (width 0.2))
   (gr_circle (center 147.059 120.837) (end 149.059 120.837) (layer Dwgs.User) (width 0.2))
+  (segment (start 156.45 113.7) (end 156.89934 114.14934) (width 0.25) (layer B.Cu) (net 1))
+  (segment (start 155.6 113.7) (end 156.45 113.7) (width 0.25) (layer B.Cu) (net 1))
+  (segment (start 156.89934 114.14934) (end 156.89934 114.221946) (width 0.25) (layer B.Cu) (net 1))
+  (via (at 156.89934 114.221946) (size 0.6) (drill 0.4) (layers F.Cu B.Cu) (net 1))
   (segment (start 141.2 100.65) (end 141.2 101.352781) (width 0.25) (layer F.Cu) (net 1) (status 10))
   (segment (start 141.325 101.477781) (end 141.276152 101.428933) (width 0.25) (layer F.Cu) (net 1))
@@
   (via (at 155.96108 111.70666) (size 0.6) (drill 0.4) (layers F.Cu B.Cu) (net 1))
   (segment (start 155.95 112.45) (end 155.95 113.1) (width 0.25) (layer F.Cu) (net 1) (status 30))
-  (segment (start 155.6 113.7) (end 156.47106 113.7) (width 0.25) (layer B.Cu) (net 1) (status 10))
-  (segment (start 156.47106 113.7) (end 156.95676 114.1857) (width 0.25) (layer B.Cu) (net 1))
-  (via (at 156.95676 114.1857) (size 0.6) (drill 0.4) (layers F.Cu B.Cu) (net 1))
   (via (at 149.55 115.8) (size 0.6) (drill 0.4) (layers F.Cu B.Cu) (net 1) (status 30))
   (via (at 149.23 112.5) (size 0.6) (drill 0.4) (layers F.Cu B.Cu) (net 1) (status 30))
@@
   (segment (start 118.75 112.6) (end 118.75 113.5) (width 0.25) (layer B.Cu) (net 16) (status 10))
   (segment (start 119.08 113.83) (end 122.35 113.83) (width 0.25) (layer B.Cu) (net 16) (status 20))
+  (segment (start 160.103998 105.55) (end 160.28934 105.55) (width 1) (layer F.Cu) (net 17))
+  (segment (start 157.82544 107.828558) (end 160.103998 105.55) (width 1) (layer F.Cu) (net 17))
+  (segment (start 158.660609 110.456489) (end 157.82544 109.62132) (width 1) (layer F.Cu) (net 17))
+  (segment (start 158.660609 115.243712) (end 158.660609 110.456489) (width 1) (layer F.Cu) (net 17))
+  (segment (start 156.654322 117.249999) (end 158.660609 115.243712) (width 1) (layer F.Cu) (net 17))
+  (segment (start 144.449999 117.249999) (end 156.654322 117.249999) (width 1) (layer F.Cu) (net 17))
+  (segment (start 138.1 110.9) (end 144.449999 117.249999) (width 1) (layer F.Cu) (net 17))
+  (segment (start 160.28934 105.55) (end 161.35 105.55) (width 1) (layer F.Cu) (net 17))
+  (segment (start 157.82544 109.62132) (end 157.82544 107.828558) (width 1) (layer F.Cu) (net 17))
   (segment (start 150.06574 101.98354) (end 150.5966 102.5144) (width 0.25) (layer B.Cu) (net 17))
   (segment (start 150.5966 102.5144) (end 153.750722 102.5144) (width 0.25) (layer B.Cu) (net 17))
@@
   (segment (start 153.750722 102.5144) (end 156.786322 105.55) (width 0.25) (layer B.Cu) (net 17))
   (segment (start 156.786322 105.55) (end 161.35 105.55) (width 0.25) (layer B.Cu) (net 17) (status 20))
-  (segment (start 157.82544 109.62132) (end 157.82544 107.828558) (width 1) (layer F.Cu) (net 17))
-  (segment (start 157.82544 107.828558) (end 160.103998 105.55) (width 1) (layer F.Cu) (net 17))
-  (segment (start 160.103998 105.55) (end 161.35 105.55) (width 1) (layer F.Cu) (net 17) (status 20))
-  (segment (start 158.249999 110.045879) (end 157.82544 109.62132) (width 1) (layer F.Cu) (net 17))
-  (segment (start 158.36646 115.5446) (end 158.249999 115.428139) (width 1) (layer F.Cu) (net 17))
-  (segment (start 158.249999 115.428139) (end 158.249999 110.045879) (width 1) (layer F.Cu) (net 17))
-  (segment (start 156.185091 117.725969) (end 158.36646 115.5446) (width 1) (layer F.Cu) (net 17))
-  (segment (start 138.1 110.9) (end 144.449999 117.249999) (width 1) (layer F.Cu) (net 17) (status 10))
-  (segment (start 144.449999 117.249999) (end 151.181339 117.249999) (width 1) (layer F.Cu) (net 17))
-  (segment (start 151.181339 117.249999) (end 151.657309 117.725969) (width 1) (layer F.Cu) (net 17))
-  (segment (start 151.657309 117.725969) (end 156.185091 117.725969) (width 1) (layer F.Cu) (net 17))
   (segment (start 163.95 105.55) (end 161.35 105.55) (width 0.4) (layer F.Cu) (net 17) (status 30))
   (segment (start 130.90144 84.26704) (end 130.90144 81.75856) (width 0.25) (layer B.Cu) (net 17))
@@
   (segment (start 125.6946 104.15) (end 125.70968 104.13492) (width 1) (layer F.Cu) (net 17))
   (via (at 125.70968 104.13492) (size 1.5) (drill 1) (layers F.Cu B.Cu) (net 17))
+  (via (at 153.5 115.4) (size 0.6) (drill 0.4) (layers F.Cu B.Cu) (net 18))
+  (segment (start 157.33758 115.4) (end 153.5 115.4) (width 0.25) (layer F.Cu) (net 18))
+  (segment (start 154.9097 101.04628) (end 154.9097 101.74628) (width 0.25) (layer F.Cu) (net 18))
+  (segment (start 156.91866 113.08842) (end 157.72384 113.8936) (width 0.25) (layer F.Cu) (net 18))
+  (segment (start 154.9097 101.74628) (end 156.91866 103.75524) (width 0.25) (layer F.Cu) (net 18))
+  (segment (start 156.91866 103.75524) (end 156.91866 113.08842) (width 0.25) (layer F.Cu) (net 18))
+  (segment (start 157.72384 113.8936) (end 157.72384 115.01374) (width 0.25) (layer F.Cu) (net 18))
+  (segment (start 157.72384 115.01374) (end 157.33758 115.4) (width 0.25) (layer F.Cu) (net 18))
+  (segment (start 154.88702 99.18446) (end 154.88702 101.0236) (width 0.25) (layer F.Cu) (net 18))
+  (segment (start 154.88702 101.0236) (end 154.9097 101.04628) (width 0.25) (layer F.Cu) (net 18))
   (segment (start 137.07364 92.87002) (end 140.4082 89.53546) (width 0.5) (layer B.Cu) (net 18))
   (via (at 137.07364 92.87002) (size 1) (drill 0.7) (layers F.Cu B.Cu) (net 18))
@@
   (segment (start 123.1 102.45) (end 126.15 102.45) (width 0.25) (layer F.Cu) (net 26) (status 30))
   (segment (start 126.15 102.45) (end 126.2 102.4) (width 0.25) (layer F.Cu) (net 26) (status 30))
-  (segment (start 152.293 101.31298) (end 150.16226 101.31298) (width 0.25) (layer F.Cu) (net 37))
-  (segment (start 150.16226 101.31298) (end 149.41296 100.56368) (width 0.25) (layer F.Cu) (net 37))
+  (segment (start 151.57776 101.32822) (end 150.1775 101.32822) (width 0.25) (layer F.Cu) (net 37))
+  (segment (start 150.1775 101.32822) (end 149.41296 100.56368) (width 0.25) (layer F.Cu) (net 37))
+  (segment (start 152.7097 101.04628) (end 151.8597 101.04628) (width 0.25) (layer F.Cu) (net 37))
+  (segment (start 151.8597 101.04628) (end 151.57776 101.32822) (width 0.25) (layer F.Cu) (net 37))
   (segment (start 152.7097 101.04628) (end 152.5597 101.04628) (width 0.25) (layer F.Cu) (net 37))
   (segment (start 152.5597 101.04628) (end 152.293 101.31298) (width 0.25) (layer F.Cu) (net 37))

Commit message: update
Parts:
- removed C5: 4.7uF, Capacitors_SMD:C_0603_HandSoldering
- removed C7: C_0.1uF, Capacitors_SMD:C_0603_HandSoldering
- removed Q2: Q_NMOS_GSD, TO_SOT_Packages_SMD:SOT-23
- removed Q3: Q_PMOS_GSD, TO_SOT_Packages_SMD:SOT-23
- removed R14, R15: 1K, Resistors_SMD:R_0603_HandSoldering
- removed U7: OPT3001, Housings_DFN_QFN:DFN-6-1EP_2x2mm_Pitch0.65mm
- added D3: LED, LEDs:LED_0603, F.Cu at (130.8, 87.5)
- added D5: LED, LEDs:LED_0603, F.Cu at (139.6, 87.3)
- added R11: R_10k, Resistors_SMD:R_0603, F.Cu at (126.5, 87.1)
- added REBOOT: SW_PUSH, Buttons_Switches_SMD:SW_SPST_KMR2, F.Cu at (130.7, 82.9)
- C2: footprint open-automation:CAP-RAD-5mm-UVR1H102MHD -> Capacitors_THT:CP_Radial_D10.0mm_P3.50mm
- Q1, R10, R5, R8, R9, U10: moved to B.Cu
- R1: value R_10 -> R_1
- R2, R3: value 1K -> R_10k; footprint Resistors_SMD:R_0603_HandSoldering -> Resistors_SMD:R_0603
- R4: value 50m -> R_10k; footprint Resistors_SMD:R_0805_HandSoldering -> Resistors_SMD:R_0603; moved to F.Cu
- R7: value R_10k -> 1K
- U2: value Power-Monitor-INA219 -> TSL45315CL; footprint TO_SOT_Packages_SMD:SOT-23-8_Handsoldering -> open-automation:LIGHT-SENSOR-TSL45315CL
- U4: footprint footprints:enclosure-25x38 -> open-automation:enclosure-25x38
- moved R2 44.7 mm to (154.3, 85.7), turned to 180 degrees
- moved C8 39.7 mm to (152.7, 112.9), turned to 180 degrees
- moved J1 39.4 mm to (129.4, 122.4)
- moved R4 35.0 mm to (139.6, 85.6)
- moved D4 33.3 mm to (126.5, 89.4), turned to 0 degrees
- moved U2 33.0 mm to (156.4, 118.0), turned to 270 degrees
- moved U5 31.5 mm to (148.0, 114.6), turned to 90 degrees
- moved C3 27.8 mm to (126.6, 91.3), turned to 180 degrees
- moved U11 25.3 mm to (126.3, 97.3), turned to 90 degrees
- moved Q1 20.3 mm to (113.5, 110.4), turned to 0 degrees
- moved C1 18.8 mm to (113.7, 118.6), turned to 180 degrees
- moved L1 18.1 mm to (122.9, 110.8), turned to 0 degrees
- moved R9 17.7 mm to (154.1, 116.9), turned to 270 degrees
- moved PROG 16.5 mm to (139.4, 82.9), turned to 180 degrees
- moved C6 16.3 mm to (145.1, 114.1), turned to 270 degrees
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Connections:
- D2 pad 2: V_USB -> 3V3
- P5 pad 3: Net-(P5-Pad3) -> TXD
- P5 pad 4: Net-(P5-Pad4) -> RXD
- P5 pad 5: Net-(P5-Pad5) -> TXD
- P5 pad 6: Net-(P5-Pad6) -> RXD
- PROG pad 1: EN -> PROG
- Q1 pad 1: BAT_SW -> PANEL_SW
- Q1 pad 2: BATTERY -> V_PANEL
- Q1 pad 3: Net-(Q1-Pad3) -> V_MAIN
- R10 pad 2: 3V3 -> VCC_I2C
- R2 pad 1: Net-(D4-Pad1) -> Net-(D2-Pad1)
- R2 pad 2: GND -> FACTORY
- R3 pad 1: 3V3 -> Net-(D3-Pad1)
- R3 pad 2: BAT_SW -> EN
- R4 pad 1: V_PANEL -> Net-(D5-Pad1)
- R4 pad 2: V_MAIN -> PROG
- R5 pad 1: Net-(Q1-Pad3) -> BATTERY
- R7 pad 1: LIGHT_INT -> 3V3
- R7 pad 2: 3V3 -> PANEL_SW
- R9 pad 2: 3V3 -> VCC_I2C
- U1 pad 27: BAT_SW -> PANEL_SW
- U2 pad 1: V_PANEL -> VCC_I2C
- U2 pad 2: V_MAIN -> GND
- U2 pad 3: GND -> SDA
- U2 pad 4: VCC_I2C -> SCL
- U5 pad 1: Net-(Q1-Pad3) -> BATTERY
- U5 pad 7: 3V3 -> VCC_I2C
Routing:
- net BAT_SW: track 54.2 -> 0.00 mm, vias 4 -> 0
- net BATTERY: track 4.86 -> 51.3 mm, vias 4 -> 6
- net SCL: track 82.7 -> 38.8 mm, vias 2 -> 0
- net PANEL_SW: track 0.00 -> 41.2 mm, vias 0 -> 4
- net VCC_I2C: track 73.1 -> 37.0 mm, vias 7 -> 9
- net 3V3: track 134.8 -> 98.8 mm, vias 9 -> 8
- net PROG: track 41.7 -> 75.8 mm
- net SDA: track 83.6 -> 50.3 mm, vias 4 -> 0
- net FACTORY: track 31.4 -> 64.4 mm, vias 1 -> 5
- net V_USB: track 97.8 -> 65.6 mm, vias 2 -> 1
- net V_MAIN: track 46.3 -> 74.6 mm, vias 3 -> 6
- net Net-(Q1-Pad3): track 16.6 -> 0.00 mm, vias 1 -> 0
- net Net-(D2-Pad1): track 13.1 -> 1.74 mm, vias 2 -> 0
- net Net-(D1-Pad1): track 25.6 -> 14.2 mm, vias 1 -> 0
- net TXD: track 30.4 -> 41.5 mm, vias 0 -> 1
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- removed copper zone on B.Cu, net BATTERY
- removed copper zone on F.Cu, net Net-(Q1-Pad3)
- removed copper zone on B.Cu, net V_MAIN
- removed copper zone on B.Cu, net V_PANEL
Other:
- board text added: "Smart-Regulator v0.3"
- board text removed: "Smart-Regulator v0.2"

Commit message: update
Parts:
- moved U3 0.05 mm to (116.1, 95.3)
Other:
- board text added: "3V3"
- board text added: "FACT"
- board text added: "GND"
- board text added: "PROG"
- board text added: "RX"
- board text added: "SCL"
- board text added: "SDA"
- board text added: "Smart-Regulator v0.4"
- board text added: "TX"
- board text added: "USB"
- board text removed: "Smart-Regulator v0.3"
Changed lines of the file:
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@@
     (area 82.735 68.56 184.875001 142.276666)
     (thickness 1.6)
-    (drawings 21)
-    (tracks 447)
+    (drawings 31)
+    (tracks 446)
     (zones 0)
     (modules 42)
@@
     (44 Edge.Cuts user)
     (45 Margin user hide)
-    (46 B.CrtYd user)
-    (47 F.CrtYd user)
+    (46 B.CrtYd user hide)
+    (47 F.CrtYd user hide)
     (48 B.Fab user hide)
     (49 F.Fab user hide)
@@
     (tags "capacitor 0603")
     (attr smd)
-    (fp_text reference C3 (at -2.9 0 180) (layer F.SilkS)
+    (fp_text reference C3 (at 2.72 -0.21 180) (layer F.SilkS)
       (effects (font (size 0.7 0.7) (thickness 0.15)))
     )
@@
     (tags "smd diode")
     (attr smd)
-    (fp_text reference D4 (at 2.5 0) (layer F.SilkS)
+    (fp_text reference D4 (at -2.26 0.06) (layer F.SilkS)
       (effects (font (size 0.7 0.7) (thickness 0.15)))
     )
@@
     (tags "resistor 0603")
     (attr smd)
-    (fp_text reference R11 (at 1.8 0 90) (layer F.SilkS)
+    (fp_text reference R11 (at -2.37 -0.05 180) (layer F.SilkS)
       (effects (font (size 0.7 0.7) (thickness 0.15)))
     )
@@
       (net 14 FACTORY))
   )
-  (module open-automation:Regulator-LM2576 (layer F.Cu)
-    (at 116.14 95.26 270)
-    (fp_text reference U3 (at 4.722 3.046 360) (layer F.SilkS)
-      (effects (font (size 0.7 0.7) (thickness 0.15)))
-    )
-    (fp_text value LM2576 (at -0.1 -6.25 270) (layer F.Fab)
-      (effects (font (size 1 1) (thickness 0.15)))
-    )
-    (fp_line (start 3.5 -5.55) (end -4.65 -5.55) (layer F.SilkS) (width 0.15))
-    (fp_line (start 3.5 4.6) (end 3.5 -5.55) (layer F.SilkS) (width 0.15))
-    (fp_line (start -4.65 4.6) (end 3.5 4.6) (layer F.SilkS) (width 0.15))
-    (fp_line (start -4.65 -5.55) (end -4.65 4.6) (layer F.SilkS) (width 0.15))
-    (pad 5 smd rect (at 6.65 -3.9 270) (size 2.16 1.07) (layers F.Cu F.Paste F.Mask)
-      (net 17 POWER_EN))
-    (pad 4 smd rect (at 6.65 -2.2 270) (size 2.16 1.07) (layers F.Cu F.Paste F.Mask)
-      (net 11 V_USB))
-    (pad 2 smd rect (at 6.65 1.2 270) (size 2.16 1.07) (layers F.Cu F.Paste F.Mask)
-      (net 2 "Net-(D1-Pad1)"))
-    (pad 3 smd rect (at 6.65 -0.5 270) (size 2.16 1.07) (layers F.Cu F.Paste F.Mask)
-      (net 1 GND))
-    (pad 1 smd rect (at 6.65 2.9 270) (size 2.16 1.07) (layers F.Cu F.Paste F.Mask)
-      (net 10 V_MAIN))
-    (pad 3 smd rect (at -0.65 -0.45 270) (size 6.99 8.33) (layers F.Cu F.Paste F.Mask)
-      (net 1 GND))
-  )
   (module Resistors_SMD:R_0603_HandSoldering (layer B.Cu)
     (at 140.34 114.86 270)
@@
       (net 15 V_PANEL))
   )
-  (gr_text "Smart-Regulator v0.3" (at 124.92736 124.91212) (layer F.SilkS)
+  (module open-automation:Regulator-LM2576 (layer F.Cu)
+    (at 116.13 95.31 270)
+    (fp_text reference U3 (at 4.722 3.046 360) (layer F.SilkS)
+      (effects (font (size 0.7 0.7) (thickness 0.15)))
+    )
+    (fp_text value LM2576 (at -0.1 -6.25 270) (layer F.Fab)
+      (effects (font (size 1 1) (thickness 0.15)))
+    )
+    (fp_line (start 3.5 -5.55) (end -6.44 -5.56) (layer F.SilkS) (width 0.15))
+    (fp_line (start 3.5 4.6) (end 3.5 -5.55) (layer F.SilkS) (width 0.15))
+    (fp_line (start -6.44 4.59) (end 3.5 4.6) (layer F.SilkS) (width 0.15))
+    (fp_line (start -6.44 -5.56) (end -6.44 4.59) (layer F.SilkS) (width 0.15))
+    (pad 5 smd rect (at 6.65 -3.9 270) (size 3 1.07) (layers F.Cu F.Paste F.Mask)
+      (net 17 POWER_EN))
+    (pad 4 smd rect (at 6.65 -2.2 270) (size 3 1.07) (layers F.Cu F.Paste F.Mask)
+      (net 11 V_USB))
+    (pad 2 smd rect (at 6.65 1.2 270) (size 3 1.07) (layers F.Cu F.Paste F.Mask)
+      (net 2 "Net-(D1-Pad1)"))
+    (pad 3 smd rect (at 6.65 -0.5 270) (size 3 1.07) (layers F.Cu F.Paste F.Mask)
+      (net 1 GND))
+    (pad 1 smd rect (at 6.65 2.9 270) (size 3 1.07) (layers F.Cu F.Paste F.Mask)
+      (net 10 V_MAIN))
+    (pad 3 smd rect (at -1.65 -0.46 270) (size 9 8.33) (layers F.Cu F.Paste F.Mask)
+      (net 1 GND))
+  )
+  (gr_text GND (at 129.48 124.37) (layer F.SilkS)
+    (effects (font (size 0.7 0.7) (thickness 0.15)))
+  )
+  (gr_text 3V3 (at 131.85 124.4) (layer F.SilkS)
+    (effects (font (size 0.7 0.7) (thickness 0.15)))
+  )
+  (gr_text PROG (at 134.46 124.33) (layer F.SilkS)
+    (effects (font (size 0.7 0.7) (thickness 0.15)))
+  )
+  (gr_text FACT (at 137.33 124.36) (layer F.SilkS)
+    (effects (font (size 0.7 0.7) (thickness 0.15)))
+  )
+  (gr_text SCL (at 139.82 124.31) (layer F.SilkS)
+    (effects (font (size 0.7 0.7) (thickness 0.15)))
+  )
+  (gr_text SDA (at 139.44 117.98) (layer F.SilkS)
+    (effects (font (size 0.7 0.7) (thickness 0.15)))
+  )
+  (gr_text RX (at 137.03 118) (layer F.SilkS)
+    (effects (font (size 0.7 0.7) (thickness 0.15)))
+  )
+  (gr_text TX (at 134.5 117.97) (layer F.SilkS)
+    (effects (font (size 0.7 0.7) (thickness 0.15)))
+  )
+  (gr_text USB (at 131.85 117.95) (layer F.SilkS)
+    (effects (font (size 0.7 0.7) (thickness 0.15)))
+  )
+  (gr_text GND (at 129.4 117.95) (layer F.SilkS)
+    (effects (font (size 0.7 0.7) (thickness 0.15)))
+  )
+  (gr_text "Smart-Regulator v0.4" (at 124.92736 124.91212) (layer F.SilkS)
     (effects (font (size 1 1) (thickness 0.2)) (justify right))
   )
@@
   (segment (start 125.69 87.11) (end 125.74 87.06) (width 0.25) (layer F.Cu) (net 9) (status 30))
   (segment (start 113.14 104.76) (end 113.14 102.01) (width 2) (layer F.Cu) (net 10))
-  (segment (start 113.14 102.01) (end 113.204999 101.945001) (width 2) (layer F.Cu) (net 10))
   (segment (start 113.46 114.19) (end 113.14 113.87) (width 2) (layer F.Cu) (net 10))
   (segment (start 113.14 113.87) (end 113.14 104.76) (width 2) (layer F.Cu) (net 10))
