File: hardware/smart-regulator.kicad_pcb (KiCad board)
At the start: 2 copper layers, 82.5 x 48.6 mm, 42 parts, among them J1 Conn_02x05_Odd_Even, P5 USB_A_2, Q1 Q_NMOS_GSD_PSMN038-100YLX, U1 ESP-WROOM-32, U10 touchpad, U11 SPX1117M3-L-3-3/TR, U2 TSL45315CL, U3 LM2576, U4 housing-mounts, U5 Power-Monitor-INA219, U6 SI7020-A20

Commit message: update
Parts:
- removed R5: 50m, Resistors_SMD:R_0805_HandSoldering
- C4: value C_100uF -> C_10uF
- Q1: value Q_NMOS_GSD_PSMN038-100YLX -> Q_NMOS_GSD_AOD4184A; footprint open-automation:SOT-669_PSMN038-100YLX -> TO_SOT_Packages_SMD:TO-252-2_Rectifier
- R1: value R_1 -> R_10m; footprint Resistors_SMD:R_0603_HandSoldering -> Resistors_SMD:R_2512_HandSoldering; moved to F.Cu
- R8: moved to F.Cu
- U11: value SPX1117M3-L-3-3/TR -> NCP1117LPST33T3G
- moved R1 38.7 mm to (114.0, 86.5), turned to 0 degrees
- moved D1 5.51 mm to (124.9, 111.2)
- moved R8 4.41 mm to (123.9, 103.2), turned to 0 degrees
- moved Q1 2.26 mm to (115.5, 109.4), turned to 90 degrees
- moved BATTERY 0.36 mm to (106.8, 102.0), turned to 270 degrees
- turned L1 to 90 degrees
Connections:
- C10 pad 1: VCC_I2C -> 3V3
- C4 pad 1: VCC_I2C -> 3V3
- C6 pad 1: VCC_I2C -> 3V3
- C8 pad 2: VCC_I2C -> 3V3
- C9 pad 1: VCC_I2C -> 3V3
- R1 pad 1: VCC_I2C -> BATTERY
- R1 pad 2: 3V3 -> V_MAIN
- R10 pad 2: VCC_I2C -> 3V3
- R9 pad 2: VCC_I2C -> 3V3
- U2 pad 1: VCC_I2C -> 3V3
- U5 pad 4: VCC_I2C -> 3V3
- U5 pad 7: VCC_I2C -> 3V3
- U6 pad 5: VCC_I2C -> 3V3
Routing:
- net 3V3: track 98.8 -> 140.5 mm, vias 8 -> 17
- net VCC_I2C: track 37.0 -> 0.00 mm, vias 9 -> 0
- net V_MAIN: track 74.6 -> 107.2 mm, vias 6 -> 7
- net BATTERY: track 51.3 -> 68.5 mm, vias 6 -> 4
- net Net-(D1-Pad1): track 14.2 -> 19.1 mm
- net POWER_EN: track 39.3 -> 35.5 mm, vias 7 -> 3
- net FACTORY: track 64.4 -> 61.0 mm
- net V_PANEL: track 17.7 -> 21.0 mm
- net PANEL_SW: track 41.2 -> 39.5 mm
- net GND: track 37.5 -> 38.9 mm, vias 12 -> 11
- net V_USB: track 65.6 -> 66.4 mm
Other:
- board text added: "Smart-Regulator v0.5"
- board text removed: "Smart-Regulator v0.4"

Commit message: layout complete bitches
Parts:
- removed BATTERY, PANEL: CONN_01X02, open-automation:XT60
- removed FACTORY, PROG, REBOOT: SW_PUSH, Buttons_Switches_SMD:SW_SPST_KMR2
- removed LOGO: , open-automation:LOGO
- removed P5: USB_A_2, open-automation:USB_A_2
- added BATTERY1: CONN_01X02, open-automation:XT60, F.Cu at (143.9, 39.7)
- added C11: 100uF, Capacitor_THT:CP_Radial_D10.0mm_P3.50mm, F.Cu at (236.4, 48.3)
- added C12: 4.7uF, Capacitor_SMD:C_0603_1608Metric_Pad1.05x0.95mm_HandSolder, F.Cu at (125.5, -18.7)
- added C13: 1000uF, Capacitor_THT:CP_Radial_D10.0mm_P3.50mm, F.Cu at (199.9, -22.9)
- added C14: C_0.1uF, Capacitor_SMD:C_0603_1608Metric_Pad1.05x0.95mm_HandSolder, F.Cu at (271.9, 16.7)
- added C15: C_0.1uF, Capacitor_SMD:C_0603_1608Metric_Pad1.05x0.95mm_HandSolder, F.Cu at (271.8, 19.8)
- added C5: C_10uF, Capacitor_SMD:C_1206_3216Metric_Pad1.42x1.75mm_HandSolder, F.Cu at (150.0, -22.1)
- added C7: C_10uF, Capacitor_SMD:C_1206_3216Metric_Pad1.42x1.75mm_HandSolder, F.Cu at (144.3, -22.2)
- added D6: D, Diode_SMD:D_SMC, F.Cu at (226.7, 28.0)
- added D7: D_Schottky, Diode_SMD:D_SMA, F.Cu at (223.5, 78.0)
- added D8: LED, LED_SMD:LED_0603_1608Metric_Pad0.88x0.95mm_HandSolder, F.Cu at (128.1, -19.5)
- added P1: USB_A_2, open-automation:USB_A_2, F.Cu at (105.6, 106.2)
- added PANEL1: CONN_01X02, open-automation:XT60, F.Cu at (167.7, 16.0)
- added R12: R_10k, Resistor_SMD:R_0603_1608Metric_Pad1.05x0.95mm_HandSolder, F.Cu at (182.3, 6.66)
- added R13: R_10k, Resistor_SMD:R_0603_1608Metric_Pad1.05x0.95mm_HandSolder, F.Cu at (208.6, -25.9)
- added R14: R_10k, Resistor_SMD:R_0603_1608Metric_Pad1.05x0.95mm_HandSolder, F.Cu at (211.9, -27.4)
- added R15: R_10k, Resistor_SMD:R_0603_1608Metric_Pad1.05x0.95mm_HandSolder, F.Cu at (208.6, -24.4)
- added R16: R_10k, Resistor_SMD:R_0603_1608Metric_Pad1.05x0.95mm_HandSolder, F.Cu at (211.9, -25.9)
- added R17: R_1k, Resistor_SMD:R_0603_1608Metric_Pad1.05x0.95mm_HandSolder, F.Cu at (262.0, 19.8)
- added R18: R_1k, Resistor_SMD:R_0603_1608Metric_Pad1.05x0.95mm_HandSolder, F.Cu at (265.4, 16.7)
- added R19: R_10k, Resistor_SMD:R_0603_1608Metric_Pad1.05x0.95mm_HandSolder, F.Cu at (208.6, -22.9)
- added R20: R_10k, Resistor_SMD:R_0603_1608Metric_Pad1.05x0.95mm_HandSolder, F.Cu at (128.3, -17.8)
- added R21: 1K, Resistor_SMD:R_0603_1608Metric_Pad1.05x0.95mm_HandSolder, F.Cu at (134.1, -23.7)
- added R5: R_10k, Resistor_SMD:R_0603_1608Metric_Pad1.05x0.95mm_HandSolder, F.Cu at (220.9, -21.0)
- added SW1: SW_PUSH, Button_Switch_SMD:SW_SPST_KMR2, F.Cu at (157.7, -47.9)
- added SW2: SW_PUSH, Button_Switch_SMD:SW_SPST_KMR2, F.Cu at (157.7, -44.2)
- added SW3: SW_PUSH, Button_Switch_SMD:SW_SPST_KMR2, F.Cu at (163.3, -47.9)
- added U12: ZLDO1117G33TA, Package_TO_SOT_SMD:SOT-223, F.Cu at (125.5, -25.6)
- added U13: LM2576, open-automation:Regulator-LM2576, F.Cu at (214.1, 83.0)
- added U14: SI7006-A20, open-automation:SI7020-A20, F.Cu at (103.0, 62.1)
- added U15: TSL45315CL, open-automation:LIGHT-SENSOR-TSL45315CL, F.Cu at (137.7, 69.4)
- added U7: ACS712ELCTR-05B-T_NRND, open-automation:ACS711, F.Cu at (243.4, 8.16)
- added U8: Power-Monitor-INA219, Package_TO_SOT_SMD:SOT-23-8_Handsoldering, F.Cu at (136.7, -26.3)
- added U9: Power-Monitor-INA219, Package_TO_SOT_SMD:SOT-23-8_Handsoldering, F.Cu at (141.5, -30.0)
- C1: value 100uF -> C_10uF; footprint open-automation:CAP-RAD-5mm-UVR1H102MHD -> Capacitor_SMD:C_0603_1608Metric_Pad1.05x0.95mm_HandSolder
- C10, C8, C9: footprint Capacitors_SMD:C_0603_HandSoldering -> Capacitor_SMD:C_0603_1608Metric_Pad1.05x0.95mm_HandSolder; moved to F.Cu
- C2: value 1000uF -> C_1uF; footprint Capacitors_THT:CP_Radial_D10.0mm_P3.50mm -> Capacitor_SMD:C_0603_1608Metric_Pad1.05x0.95mm_HandSolder
- C3: value 4.7uF -> C_0.1uF; footprint Capacitors_SMD:C_0603_HandSoldering -> Capacitor_SMD:C_0603_1608Metric_Pad1.05x0.95mm_HandSolder
- C4: footprint Capacitors_SMD:C_1206_HandSoldering -> Capacitor_SMD:C_0603_1608Metric_Pad1.05x0.95mm_HandSolder; moved to F.Cu
- C6: value C_1uF -> C_10uF; footprint Capacitors_SMD:C_0603_HandSoldering -> Capacitor_SMD:C_1206_3216Metric_Pad1.42x1.75mm_HandSolder; moved to F.Cu
- D1: value D_Schottky -> LED-0603-R; footprint Diodes_SMD:D_SMA -> LED_SMD:LED_0603_1608Metric_Pad0.88x0.95mm_HandSolder; moved to F.Cu
- D2, D3: value LED -> LED-0603-R; footprint LEDs:LED_0603 -> LED_SMD:LED_0603_1608Metric_Pad0.88x0.95mm_HandSolder
- D4: value LED -> D; footprint Diodes_SMD:D_0603 -> Diode_SMD:D_SMC
- D5: value LED -> D; footprint LEDs:LED_0603 -> Diode_SMD:D_SMC
- J1: footprint Pin_Headers:Pin_Header_Straight_2x05_Pitch2.54mm -> Connector_PinHeader_2.54mm:PinHeader_2x05_P2.54mm_Vertical
- Q1: footprint TO_SOT_Packages_SMD:TO-252-2_Rectifier -> Package_TO_SOT_SMD:TO-252-2; moved to F.Cu
- R1: value R_10m -> R_10k; footprint Resistors_SMD:R_2512_HandSoldering -> Resistor_SMD:R_0603_1608Metric_Pad1.05x0.95mm_HandSolder
- R10: value R_10k -> R_10m; footprint Resistors_SMD:R_0603_HandSoldering -> Resistor_SMD:R_2512_6332Metric_Pad1.52x3.35mm_HandSolder; moved to F.Cu
- R11, R2, R3, R4: footprint Resistors_SMD:R_0603 -> Resistor_SMD:R_0603_1608Metric_Pad1.05x0.95mm_HandSolder
- R6: footprint Resistors_SMD:R_0603_HandSoldering -> Resistor_SMD:R_0603_1608Metric_Pad1.05x0.95mm_HandSolder; moved to F.Cu
- R7: value 1K -> R_10m; footprint Resistors_SMD:R_0603_HandSoldering -> Resistor_SMD:R_2512_6332Metric_Pad1.52x3.35mm_HandSolder; moved to F.Cu
- R8: value R_10k -> R_10m; footprint Resistors_SMD:R_0603_HandSoldering -> Resistor_SMD:R_2512_6332Metric_Pad1.52x3.35mm_HandSolder
- R9: value R_10k -> R_1k; footprint Resistors_SMD:R_0603_HandSoldering -> Resistor_SMD:R_0603_1608Metric_Pad1.05x0.95mm_HandSolder; moved to F.Cu
- U1: moved to F.Cu
- U10: value touchpad -> Power-Monitor-INA219; footprint open-automation:touch-pad -> Package_TO_SOT_SMD:SOT-23-8_Handsoldering; moved to F.Cu
- U11: value NCP1117LPST33T3G -> DAC; footprint open-automation:SPX1117M3 -> Package_DFN_QFN:DFN-14-1EP_3x3mm_P0.4mm_EP1.78x2.35mm
- U2: value TSL45315CL -> housing-mounts; footprint open-automation:LIGHT-SENSOR-TSL45315CL -> open-automation:enclosure-25x38; moved to F.Cu
- U3: value LM2576 -> touchpad; footprint open-automation:Regulator-LM2576 -> open-automation:touch-pad
- U4: value housing-mounts -> LM2576; footprint open-automation:enclosure-25x38 -> open-automation:Regulator-LM2576
- U5: value Power-Monitor-INA219 -> LM2576; footprint TO_SOT_Packages_SMD:SOT-23-8_Handsoldering -> open-automation:Regulator-LM2576; moved to F.Cu
- U6: value SI7020-A20 -> LM2576; footprint open-automation:SI7020-A20 -> open-automation:Regulator-LM2576; moved to F.Cu
- moved U6 196.5 mm to (291.8, -19.6), turned to 270 degrees
- moved R10 184.2 mm to (290.6, -4.73)
- moved J1 170.3 mm to (127.2, -47.9), turned to 0 degrees
- moved U4 169.2 mm to (258.4, -18.0), turned to 270 degrees
- moved R7 164.8 mm to (254.2, -2.51), turned to 180 degrees
- moved D1 161.6 mm to (165.1, -45.3)
- moved C1 157.3 mm to (252.0, 43.8), turned to 0 degrees
- moved R1 156.0 mm to (220.5, -27.4)
- moved C3 154.6 mm to (262.0, 16.7), turned to 0 degrees
- moved R6 147.4 mm to (224.2, -22.6), turned to 0 degrees
- moved R3 146.5 mm to (223.9, -27.4)
- moved L1 140.1 mm to (228.2, 18.2), turned to 0 degrees
- moved C6 140.0 mm to (140.8, -25.9), turned to 0 degrees
- moved D3 136.4 mm to (162.1, -45.3)
- moved C2 136.2 mm to (252.0, 45.3)
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Connections:
- net RXD renamed /RXD
- net TXD renamed /TXD
- C1 pad 1: V_MAIN -> 3V3
- C10 pad 1: 3V3 -> GND
- C10 pad 2: GND -> Net-(C10-Pad2)
- C2 pad 1: V_USB -> 3V3
- C3 pad 1: 3V3 -> +3V3
- C4 pad 1: 3V3 -> /Power/REG_POWER
- C6 pad 1: 3V3 -> /Power/REG3_POST_CURR
- C8 pad 2: 3V3 -> Net-(C8-Pad2)
- C9 pad 1: 3V3 -> GND
- C9 pad 2: GND -> Net-(C9-Pad2)
- D1 pad 2: GND -> 3V3
- D4 pad 1: Net-(D4-Pad1) -> /V_MAIN
- D4 pad 2: 3V3 -> /Power/REG2_POST_CURR
- D5 pad 1: Net-(D5-Pad1) -> /V_MAIN
- D5 pad 2: 3V3 -> /Power/REG3_POST_CURR
- J1 pad 10: SDA -> /SDA
- J1 pad 4: V_USB -> /V_USB
- J1 pad 5: PROG -> /PROG
- J1 pad 7: FACTORY -> /FACTORY
- J1 pad 9: SCL -> /SCL
- L1 pad 1: Net-(D1-Pad1) -> Net-(D7-Pad1)
- L1 pad 2: V_USB -> /V_USB
- Q1 pad 1: PANEL_SW -> /PANEL_SW
- Q1 pad 2: V_PANEL -> /V_PANEL
- Q1 pad 3: V_MAIN -> /V_MAIN
- R1 pad 1: BATTERY -> /SDA
- R1 pad 2: V_MAIN -> 3V3
- R10 pad 1: SCL -> /Power/REG1_PRE
- R10 pad 2: 3V3 -> /Power/REG1_POST_CURR
- R11 pad 1: Net-(D4-Pad1) -> /Power/REG2_POST_CURR
- R11 pad 2: GND -> /Power/OUT2
- R2 pad 1: Net-(D2-Pad1) -> /SCL
- R2 pad 2: FACTORY -> 3V3
- R3 pad 1: Net-(D3-Pad1) -> GND
- R3 pad 2: EN -> /I02
- R4 pad 1: Net-(D5-Pad1) -> Net-(D1-Pad1)
- R4 pad 2: PROG -> /FACTORY
- R6 pad 1: GND -> Net-(D3-Pad1)
- R6 pad 2: IO2 -> /PROG
- R7 pad 1: 3V3 -> /Power/REG2_PRE
- R7 pad 2: PANEL_SW -> /Power/REG2_POST_CURR
- R8 pad 1: POWER_EN -> /Power/REG3_PRE
- R8 pad 2: GND -> /Power/REG3_POST_CURR
- R9 pad 1: SDA -> +3V3
- R9 pad 2: 3V3 -> Net-(R9-Pad2)
- U1 pad 13: FACTORY -> /FACTORY
- U1 pad 24: IO2 -> /I02
- U1 pad 25: PROG -> /PROG
- U1 pad 27: PANEL_SW -> /PANEL_SW
- U1 pad 28: POWER_EN -> /POWER_EN
- U1 pad 3: EN -> /EN
- U1 pad 30: SDA -> /SDA
- U1 pad 31: SCL -> /SCL
- U10 pad 1: FACTORY -> /Power/REG3_PRE
- U11 pad 1: GND -> /SDA
- U11 pad 2: 3V3 -> /SCL
- U11 pad 3: V_MAIN -> GND
- U3 pad 1: V_MAIN -> (no net)
- U5 pad 1: BATTERY -> /Power/REG_POWER
- U5 pad 2: V_MAIN -> /Power/REG3_PRE
- U5 pad 4: 3V3 -> /Power/OUT3
- U5 pad 5: SCL -> Net-(U5-Pad5)
- U6 pad 1: SDA -> /Power/REG_POWER
- U6 pad 2: GND -> /Power/REG1_PRE
- U6 pad 3: (no net) -> GND
- U6 pad 4: (no net) -> /Power/OUT1
- U6 pad 5: 3V3 -> Net-(U6-Pad5)
Routing:
- net 3V3: track 140.5 -> 0.00 mm, vias 17 -> 0
- net V_MAIN: track 107.2 -> 0.00 mm, vias 7 -> 0
- net PROG: track 75.5 -> 0.00 mm, vias 3 -> 0
- net BATTERY: track 68.5 -> 0.00 mm, vias 4 -> 0
- net V_USB: track 66.4 -> 0.00 mm, vias 1 -> 0
- net FACTORY: track 61.0 -> 0.00 mm, vias 5 -> 0
- net SDA: track 50.3 -> 0.00 mm
- net /TXD: track 41.5 -> 0.00 mm, vias 1 -> 0
- net PANEL_SW: track 39.5 -> 0.00 mm, vias 4 -> 0
- net /RXD: track 39.2 -> 0.00 mm, vias 1 -> 0
- net GND: track 38.9 -> 0.00 mm, vias 11 -> 0
- net SCL: track 38.8 -> 0.00 mm
- net POWER_EN: track 35.5 -> 0.00 mm, vias 3 -> 0
- net V_PANEL: track 21.0 -> 0.00 mm
- net EN: track 20.4 -> 0.00 mm, vias 1 -> 0
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
Commit message: multifile update
Parts:
- removed D7: D_Schottky, Diode_SMD:D_SMA
- removed J1: Conn_02x05_Odd_Even, Connector_PinHeader_2.54mm:PinHeader_2x05_P2.54mm_Vertical
- removed L1: 47uH, open-automation:L-RAD-7.4mm
- removed Q1: Q_NMOS_GSD_AOD4184A, Package_TO_SOT_SMD:TO-252-2
- removed U13: LM2576, open-automation:Regulator-LM2576
- added C16: C_10uF, Capacitor_SMD:C_1206_3216Metric_Pad1.42x1.75mm_HandSolder, F.Cu at (224.3, 87.6)
- added J2: Conn_02x20_Top_Bottom, Connector_PinSocket_2.54mm:PinSocket_2x20_P2.54mm_Vertical, F.Cu at (241.2, 77.7)
- added PACK1: CONN_01X02, open-automation:XT60, F.Cu at (241.6, 92.8)
- added PACK2: CONN_01X02, open-automation:XT60, F.Cu at (241.8, 101.2)
- C10, C5, C6, C7, C8, C9, D4, D5, D6, R10, R11, R12, R13, R14, R15, R16, R7, R8, U10, U4, U5, U6, U8, U9: moved to B.Cu
- C11: value 100uF -> C_10uF; footprint Capacitor_THT:CP_Radial_D10.0mm_P3.50mm -> Capacitor_SMD:C_0603_1608Metric_Pad1.05x0.95mm_HandSolder
- C13: value 1000uF -> C_1uF; footprint Capacitor_THT:CP_Radial_D10.0mm_P3.50mm -> Capacitor_SMD:C_0603_1608Metric_Pad1.05x0.95mm_HandSolder
- D8: value LED -> LED-0603-R
- R21: value 1K -> R_10k
- U2: footprint open-automation:enclosure-25x38 -> open-automation:Pi Mount
- U3: value touchpad -> LM2576; footprint open-automation:touch-pad -> open-automation:Regulator-LM2576
- moved U10 186.4 mm to (221.0, 125.8), turned to 270 degrees
- moved U12 186.1 mm to (241.7, 119.7), turned to 0 degrees
- moved D1 178.2 mm to (229.1, 121.1), turned to 180 degrees
- moved D8 178.1 mm to (235.7, 122.4), turned to 90 degrees
- moved SW1 177.4 mm to (227.4, 115.2), turned to 270 degrees
- moved C12 176.4 mm to (234.8, 119.7), turned to 180 degrees
- moved R20 175.7 mm to (233.9, 122.5), turned to 90 degrees
- moved D2 173.5 mm to (216.5, 121.1), turned to 180 degrees
- moved SW2 169.4 mm to (214.8, 115.3), turned to 270 degrees
- moved C6 166.3 mm to (232.2, 113.0), turned to 90 degrees
- moved U9 163.3 mm to (226.4, 109.6), turned to 270 degrees
- moved R11 156.9 mm to (219.8, 108.2), turned to 180 degrees
- moved R13 151.8 mm to (214.4, 125.8), turned to 180 degrees
- moved R14 151.6 mm to (214.4, 124.2)
- moved D3 150.9 mm to (235.3, 86.7), turned to 270 degrees
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- renumbered BATTERY1 to PACK3
Connections:
- C11 pad 1: /V_MAIN -> /Power/REG_POWER
- C13 pad 1: /V_USB -> /Power/REG_POWER
- C5 pad 1: /Power/REG2_POST_CURR -> /PACK2
- C6 pad 1: /Power/REG3_POST_CURR -> /PACK3
- C7 pad 1: /Power/REG1_POST_CURR -> /PACK1
- D4 pad 2: /Power/REG2_POST_CURR -> /Power/REG2_PRE
- D5 pad 2: /Power/REG3_POST_CURR -> /Power/REG3_PRE
- D6 pad 2: /Power/REG1_POST_CURR -> /Power/REG1_PRE
- PACK3 pad 1: /switches/BATTERY -> /PACK3
- PANEL1 pad 1: /switches/V_PANEL -> /V_PANEL
- R10 pad 2: /Power/REG1_POST_CURR -> /PACK1
- R11 pad 1: /Power/REG2_POST_CURR -> /PACK2
- R13 pad 1: /Power/REG3_POST_CURR -> /PACK3
- R15 pad 1: /Power/REG1_POST_CURR -> /PACK1
- R19 pad 1: /POWER_EN -> /V_USB
- R19 pad 2: GND -> Net-(R19-Pad2)
- R21 pad 1: 3V3 -> Net-(R19-Pad2)
- R21 pad 2: /PANEL_SW -> GND
- R7 pad 2: /Power/REG2_POST_CURR -> /PACK2
- R8 pad 2: /Power/REG3_POST_CURR -> /PACK3
- U10 pad 2: /Power/REG3_POST_CURR -> /PACK3
- U11 pad 13: Net-(U11-Pad13) -> 3V3
- U3 pad 1: (no net) -> /Power/REG_POWER
- U4 pad 5: Net-(U4-Pad5) -> GND
- U5 pad 5: Net-(U5-Pad5) -> GND
- U6 pad 5: Net-(U6-Pad5) -> GND
- U7 pad 1: /Power/PANEL -> /V_PANEL
- U8 pad 2: /Power/REG1_POST_CURR -> /PACK1
- U9 pad 2: /Power/REG2_POST_CURR -> /PACK2
Other:
- board size 82.5 x 48.6 mm -> 157 x 56 mm

Commit message: traces complete
Parts:
- added LOGO: , open-automation:LOGO, B.Cu at (130.4, 107.8)
- added R22: R_10k, Resistor_SMD:R_0603_1608Metric_Pad1.05x0.95mm_HandSolder, F.Cu at (151.9, 92.6)
- J2: value Conn_02x20_Top_Bottom -> Conn_02x20_Odd_Even; moved to B.Cu
- moved D3 109.0 mm to (136.2, 132.0), turned to 90 degrees
- moved R6 104.4 mm to (138.1, 132.0), turned to 90 degrees
- moved FACT 99.4 mm to (128.8, 128.2), turned to 0 degrees
- moved PROG 97.9 mm to (142.8, 132.0), turned to 0 degrees
- moved R4 96.7 mm to (132.8, 128.2), turned to 90 degrees
- moved D1 94.9 mm to (134.4, 128.1), turned to 90 degrees
- moved C13 88.2 mm to (125.6, 96.6), turned to 180 degrees
- moved R3 87.0 mm to (153.1, 129.4), turned to 180 degrees
- moved EN 86.5 mm to (128.6, 121.8), turned to 0 degrees
- moved C11 86.3 mm to (125.6, 98.2), turned to 180 degrees
- moved R5 84.1 mm to (132.4, 122.0), turned to 90 degrees
- moved D2 82.2 mm to (134.3, 121.9), turned to 90 degrees
- moved C2 78.5 mm to (132.5, 109.2)
- moved C1 78.4 mm to (132.4, 110.8)
- moved U1 77.0 mm to (137.5, 110.6), turned to 0 degrees
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- renumbered SW2 to EN, SW1 to FACT, SW3 to PROG
Connections:
- net /PANEL_SW renamed Net-(U1-Pad27)
- J2 pad 10: Net-(J2-Pad10) -> /RXD
- J2 pad 13: GND -> Net-(J2-Pad13)
- J2 pad 14: Net-(J2-Pad14) -> GND
- J2 pad 17: Net-(J2-Pad17) -> 3V3
- J2 pad 19: Net-(J2-Pad19) -> /microcontroller/MOSI
- J2 pad 2: /SDA -> /V_USB
- J2 pad 21: /V_USB -> /microcontroller/MISO
- J2 pad 22: /V_USB -> Net-(J2-Pad22)
- J2 pad 23: GND -> /microcontroller/SCLK
- J2 pad 24: /TXD -> Net-(J2-Pad24)
- J2 pad 25: /RXD -> GND
- J2 pad 27: GND -> Net-(J2-Pad27)
- J2 pad 3: /SCL -> /SDA
- J2 pad 34: Net-(J2-Pad34) -> GND
- J2 pad 35: GND -> Net-(J2-Pad35)
- J2 pad 37: GND -> Net-(J2-Pad37)
- J2 pad 39: Net-(J2-Pad39) -> GND
- J2 pad 4: Net-(J2-Pad4) -> /V_USB
- J2 pad 5: GND -> /SCL
- J2 pad 6: Net-(J2-Pad6) -> GND
- J2 pad 8: Net-(J2-Pad8) -> /TXD
- J2 pad 9: 3V3 -> GND
- U1 pad 14: Net-(U1-Pad14) -> /microcontroller/MISO
- U1 pad 16: Net-(U1-Pad16) -> /microcontroller/MOSI
- U1 pad 20: Net-(U1-Pad20) -> /microcontroller/SCLK
- U1 pad 28: /POWER_EN -> /USB_EN
- U3 pad 5: GND -> /USB_EN
Routing:
- net 3V3: track 0.00 -> 233.0 mm, vias 0 -> 22
- net GND: track 0.00 -> 220.7 mm, vias 0 -> 57
- net /SCL: track 0.00 -> 116.6 mm, vias 0 -> 4
- net /SDA: track 0.00 -> 98.9 mm, vias 0 -> 3
- net /Power/REG_POWER: track 0.00 -> 75.7 mm, vias 0 -> 6
- net /TXD: track 0.00 -> 74.4 mm, vias 0 -> 2
- net /RXD: track 0.00 -> 73.6 mm, vias 0 -> 1
- net /Power/OUT3: track 0.00 -> 68.7 mm, vias 0 -> 5
- net /V_USB: track 0.00 -> 67.5 mm, vias 0 -> 2
- net /microcontroller/MISO: track 0.00 -> 54.9 mm, vias 0 -> 7
- net /V_MAIN: track 0.00 -> 49.7 mm, vias 0 -> 4
- net /microcontroller/SCLK: track 0.00 -> 49.1 mm, vias 0 -> 4
- net /USB_EN: track 0.00 -> 47.1 mm, vias 0 -> 2
- net /microcontroller/MOSI: track 0.00 -> 47.0 mm, vias 0 -> 1
- net /Power/OUT2: track 0.00 -> 39.5 mm, vias 0 -> 5
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- added copper zone on B.Cu, net GND
- removed copper zone on F.Cu, net GND
Other:
- board size 157 x 56 mm -> 66 x 56 mm
- net class DELETE removed
- net class Default: trace_width 0.25 -> 0.2
- net class x-small added: clearance 0.2, trace_width 0.2, via_dia 0.6, via_drill 0.4
- rule pad_to_mask_clearance: 0.2 -> 0
- rule trace_min: 0.2 -> 0
- board text added: "Smart-Regulator"
- board text added: "v0.6"
- board text removed: "FACT"
- board text removed: "PROG"
- board text removed: "Smart-Regulator v0.5"

Commit message: re-layout
Parts:
- removed EN, FACT, PROG: SW_PUSH, Button_Switch_SMD:SW_SPST_KMR2
- removed LOGO: , open-automation:LOGO
- added SW1: SW_PUSH, Button_Switch_SMD:SW_SPST_KMR2, F.Cu at (128.5, 128.2)
- added SW2: SW_PUSH, Button_Switch_SMD:SW_SPST_KMR2, F.Cu at (128.4, 121.8)
- added SW3: SW_PUSH, Button_Switch_SMD:SW_SPST_KMR2, F.Cu at (142.7, 132.0)
- C16, C5, C6, C7: footprint Capacitor_SMD:C_1206_3216Metric_Pad1.42x1.75mm_HandSolder -> Capacitor_SMD:C_0603_1608Metric_Pad1.05x0.95mm_HandSolder
- U3: value LM2576 -> MIC29302; moved to B.Cu
- U4, U5: value LM2576 -> MIC29302
- U6: value LM2576 -> MIC29302; moved to F.Cu
- moved U5 31.9 mm to (137.9, 93.0)
- moved U4 21.6 mm to (129.9, 125.7)
- moved C6 20.2 mm to (141.0, 123.7), turned to 180 degrees
- moved C10 16.7 mm to (141.0, 121.9), turned to 0 degrees
- moved C9 14.4 mm to (149.2, 104.8), turned to 0 degrees
- moved C8 13.7 mm to (149.5, 88.3), turned to 0 degrees
- moved U3 13.3 mm to (138.4, 109.3)
- moved C7 12.5 mm to (149.5, 90.1), turned to 180 degrees
- moved R8 12.3 mm to (143.8, 126.7)
- moved C11 11.9 mm to (132.3, 88.3), turned to 90 degrees
- moved D5 11.6 mm to (144.8, 132.6)
- moved C5 11.4 mm to (149.2, 106.4), turned to 180 degrees
- moved U10 11.3 mm to (145.5, 122.4), turned to 0 degrees
- moved U9 11.0 mm to (153.8, 105.9), turned to 0 degrees
- moved U8 10.7 mm to (155.0, 89.2), turned to 0 degrees
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Connections:
- U3 pad 1: /Power/REG_POWER -> GND
- U3 pad 2: /V_USB -> /Power/REG_POWER
- U3 pad 4: Net-(R19-Pad2) -> /Power/REG2_PRE
- U3 pad 5: /USB_EN -> /Power/OUT2
- U4 pad 1: /Power/REG_POWER -> GND
- U4 pad 2: /Power/REG2_PRE -> /Power/REG_POWER
- U4 pad 4: /Power/OUT2 -> /Power/REG3_PRE
- U4 pad 5: GND -> /Power/OUT3
- U5 pad 1: /Power/REG_POWER -> GND
- U5 pad 2: /Power/REG3_PRE -> /Power/REG_POWER
- U5 pad 4: /Power/OUT3 -> /Power/REG1_PRE
- U5 pad 5: GND -> /Power/OUT1
- U6 pad 1: /Power/REG_POWER -> /USB_EN
- U6 pad 2: /Power/REG1_PRE -> /Power/REG_POWER
- U6 pad 4: /Power/OUT1 -> /V_USB
- U6 pad 5: GND -> Net-(R19-Pad2)
Routing:
- net 3V3: track 233.0 -> 0.00 mm, vias 22 -> 0
- net GND: track 220.7 -> 0.00 mm, vias 57 -> 0
- net /SCL: track 116.6 -> 0.00 mm, vias 4 -> 0
- net /SDA: track 98.9 -> 0.00 mm, vias 3 -> 0
- net /Power/REG_POWER: track 75.7 -> 0.00 mm, vias 6 -> 0
- net /TXD: track 74.4 -> 0.00 mm, vias 2 -> 0
- net /RXD: track 73.6 -> 0.00 mm, vias 1 -> 0
- net /Power/OUT3: track 68.7 -> 0.00 mm, vias 5 -> 0
- net /V_USB: track 67.5 -> 0.00 mm, vias 2 -> 0
- net /microcontroller/MISO: track 54.9 -> 0.00 mm, vias 7 -> 0
- net /V_MAIN: track 49.7 -> 0.00 mm, vias 4 -> 0
- net /microcontroller/SCLK: track 49.1 -> 0.00 mm, vias 4 -> 0
- net /USB_EN: track 47.1 -> 0.00 mm, vias 2 -> 0
- net /microcontroller/MOSI: track 47.0 -> 0.00 mm, vias 1 -> 0
- net /Power/OUT2: track 39.5 -> 0.00 mm, vias 5 -> 0
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- added copper zone on F.Cu, net /V_PANEL

Commit message: traces complete
Parts:
- added D7: D, open-automation:SOD128, B.Cu at (155.9, 126.7)
- added D9: D, open-automation:SOD128, B.Cu at (155.9, 130.6)
- added R23: R_10k, Resistor_SMD:R_0603_1608Metric_Pad1.05x0.95mm_HandSolder, B.Cu at (143.8, 87.8)
- added R24: R_10k, Resistor_SMD:R_0603_1608Metric_Pad1.05x0.95mm_HandSolder, B.Cu at (144.2, 104.2)
- added R25: R_10k, Resistor_SMD:R_0603_1608Metric_Pad1.05x0.95mm_HandSolder, B.Cu at (135.6, 121.2)
- D4, D5, D6: footprint Diode_SMD:D_SMC -> open-automation:SOD128
- moved D5 18.8 mm to (154.2, 116.3)
- moved D4 14.9 mm to (145.2, 130.9)
- moved R2 7.19 mm to (170.7, 88.5)
- moved U11 4.72 mm to (163.7, 92.4)
- moved R17 4.58 mm to (164.2, 87.8)
- moved R18 4.55 mm to (164.3, 89.5)
- moved U4 4.50 mm to (125.4, 125.1)
- moved C14 3.48 mm to (170.7, 93.5), turned to 0 degrees
- moved R1 3.47 mm to (170.7, 92.0), turned to 180 degrees
- moved D6 1.95 mm to (154.1, 99.7)
- moved U14 1.16 mm to (174.3, 90.3), turned to 90 degrees
- moved R14 0.38 mm to (137.1, 133.7)
- moved R13 0.23 mm to (137.1, 132.0)
Connections:
- C3 pad 1: +3V3 -> 3V3
- D4 pad 2: /Power/REG2_PRE -> /Power/REG3_PRE
- D5 pad 2: /Power/REG3_PRE -> /Power/REG2_PRE
- R9 pad 1: +3V3 -> 3V3
- U1 pad 6: Net-(U1-Pad6) -> /REG3_EN
- U1 pad 8: Net-(U1-Pad8) -> /REG1_EN
- U1 pad 9: Net-(U1-Pad9) -> /REG2_EN
- U12 pad 1: /V_MAIN -> Net-(D7-Pad1)
- U3 pad 1: GND -> /REG2_EN
- U4 pad 1: GND -> /REG3_EN
- U5 pad 1: GND -> /REG1_EN
- U7 pad 12: +3V3 -> 3V3
Routing:
- net 3V3: track 0.00 -> 245.9 mm, vias 0 -> 37
- net GND: track 0.00 -> 130.5 mm, vias 0 -> 43
- net /Power/REG_POWER: track 0.00 -> 113.1 mm, vias 0 -> 9
- net /SCL: track 0.00 -> 105.0 mm, vias 0 -> 7
- net /SDA: track 0.00 -> 104.5 mm, vias 0 -> 7
- net /RXD: track 0.00 -> 77.5 mm, vias 0 -> 10
- net /V_USB: track 0.00 -> 76.8 mm, vias 0 -> 12
- net /TXD: track 0.00 -> 75.5 mm, vias 0 -> 6
- net /Power/OUT3: track 0.00 -> 74.5 mm, vias 0 -> 5
- net /microcontroller/MISO: track 0.00 -> 72.1 mm, vias 0 -> 8
- net /microcontroller/SCLK: track 0.00 -> 70.2 mm, vias 0 -> 6
- net /PACK3: track 0.00 -> 57.3 mm, vias 0 -> 7
- net /microcontroller/MOSI: track 0.00 -> 54.0 mm, vias 0 -> 6
- net /REG1_EN: track 0.00 -> 45.8 mm, vias 0 -> 3
- net /USB_EN: track 0.00 -> 44.7 mm, vias 0 -> 10
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