File: hardware/environment.sch (KiCad schematic (older format))
At the start: 5 parts, among them U6 SI7020-A20, U7 OPT3001

Commit message: update
Parts:
- removed R7: R_10k, Resistors_SMD:R_0603_HandSoldering, symbol R_10k
- removed U7: OPT3001, Housings_DFN_QFN:DFN-6-1EP_2x2mm_Pitch0.65mm, symbol OPT3001
- added U2: TSL45315CL, open-automation:LIGHT-SENSOR-TSL45315CL, symbol TSL45315CL
Connections:
- net labels removed: 3V3, LIGHT_INT
- wire segments 20 -> 16
Other:
- moved on the sheet: C10, C9, U6
Changed lines of the file:
@@
 Comment4 ""
 $EndDescr
-Text Label 4800 1300 0    197  ~ 0
+Text Label 5125 1950 0    197  ~ 0
 Environment
-Text GLabel 3050 3200 0    60   Input ~ 0
+Text GLabel 3400 3425 0    60   Input ~ 0
 VCC_I2C
 $Comp
-L GND #PWR028
+L GND #PWR023
 U 1 1 59C50BD3
-P 3500 3350
-F 0 "#PWR028" H 3500 3100 50  0001 C CNN
-F 1 "GND" H 3500 3200 50  0000 C CNN
-F 2 "" H 3500 3350 50  0000 C CNN
-F 3 "" H 3500 3350 50  0000 C CNN
-	1    3500 3350
+P 3850 3575
+F 0 "#PWR023" H 3850 3325 50  0001 C CNN
+F 1 "GND" H 3850 3425 50  0000 C CNN
+F 2 "" H 3850 3575 50  0000 C CNN
+F 3 "" H 3850 3575 50  0000 C CNN
+	1    3850 3575
 	1    0    0    -1
 $EndComp
-Text GLabel 4500 3200 2    60   Input ~ 0
+Text GLabel 4850 3425 2    60   Input ~ 0
 SCL
-Text GLabel 4500 3300 2    60   Input ~ 0
+Text GLabel 4850 3525 2    60   Input ~ 0
 SDA
 $Comp
 L SI7020-A20 U6
 U 1 1 59C50BD4
-P 4000 3300
-F 0 "U6" H 4200 3200 60  0000 C CNN
-F 1 "SI7020-A20" H 4000 3500 60  0000 C CNN
-F 2 "open-automation:SI7020-A20" H 4000 3000 60  0001 C CNN
-F 3 "https://www.digikey.com/product-detail/en/silicon-labs/SI7020-A20-GM1R/336-3596-1-ND/5823452" H 4000 3100 60  0001 C CNN
-F 4 "SI7020-A20-GM1R" H 4100 3100 60  0001 C CNN "Part Number"
-	1    4000 3300
+P 4350 3525
+F 0 "U6" H 4550 3425 60  0000 C CNN
+F 1 "SI7020-A20" H 4350 3725 60  0000 C CNN
+F 2 "open-automation:SI7020-A20" H 4350 3225 60  0001 C CNN
+F 3 "https://www.digikey.com/product-detail/en/silicon-labs/SI7020-A20-GM1R/336-3596-1-ND/5823452" H 4350 3325 60  0001 C CNN
+F 4 "SI7020-A20-GM1R" H 4450 3325 60  0001 C CNN "Part Number"
+	1    4350 3525
 	1    0    0    -1
 $EndComp
@@
 L C_0.1uF C9
 U 1 1 59C50BD5
-P 3200 3400
-F 0 "C9" H 3225 3500 50  0000 L CNN
-F 1 "C_0.1uF" H 2900 3300 50  0000 L CNN
-F 2 "Capacitors_SMD:C_0603_HandSoldering" H 3300 3700 50  0001 C CNN
-F 3 "https://www.digikey.com/product-detail/en/kemet/C0603C104K5RACTU/399-5089-1-ND/1465623" H 3200 3150 50  0001 C CNN
-F 4 "C0603C104K5RACTU" H 3325 3600 60  0001 C CNN "Part Number"
-	1    3200 3400
+P 3550 3625
+F 0 "C9" H 3575 3725 50  0000 L CNN
+F 1 "C_0.1uF" H 3250 3525 50  0000 L CNN
+F 2 "Capacitors_SMD:C_0603_HandSoldering" H 3650 3925 50  0001 C CNN
+F 3 "https://www.digikey.com/product-detail/en/kemet/C0603C104K5RACTU/399-5089-1-ND/1465623" H 3550 3375 50  0001 C CNN
+F 4 "C0603C104K5RACTU" H 3675 3825 60  0001 C CNN "Part Number"
+	1    3550 3625
 	1    0    0    -1
 $EndComp
 $Comp
-L GND #PWR029
+L GND #PWR024
 U 1 1 59C50BD6
-P 3200 3600
-F 0 "#PWR029" H 3200 3350 50  0001 C CNN
-F 1 "GND" H 3200 3450 50  0000 C CNN
-F 2 "" H 3200 3600 50  0000 C CNN
-F 3 "" H 3200 3600 50  0000 C CNN
-	1    3200 3600
+P 3550 3825
+F 0 "#PWR024" H 3550 3575 50  0001 C CNN
+F 1 "GND" H 3550 3675 50  0000 C CNN
+F 2 "" H 3550 3825 50  0000 C CNN
+F 3 "" H 3550 3825 50  0000 C CNN
+	1    3550 3825
 	1    0    0    -1
 $EndComp
-Text Label 7150 2700 0    60   ~ 0
+Text Label 7675 3250 0    60   ~ 0
 Light-Level
+Text GLabel 8425 3625 2    60   Input ~ 0
+SDA
+Text GLabel 8425 3500 2    60   Input ~ 0
+SCL
 $Comp
-L OPT3001 U7
-U 1 1 59C50BD7
-P 7500 3200
-F 0 "U7" H 7650 2950 60  0000 C CNN
-F 1 "OPT3001" H 7500 3350 60  0000 C CNN
-F 2 "Housings_DFN_QFN:DFN-6-1EP_2x2mm_Pitch0.65mm" H 7550 2850 60  0001 C CNN
-F 3 "https://www.digikey.com/product-detail/en/texas-instruments/OPT3001DNPR/296-40474-1-ND/5178351" H 7650 2950 60  0001 C CNN
-F 4 "296-40474-1-ND" H 7750 3050 60  0001 C CNN "Part Number"
-	1    7500 3200
+L GND #PWR025
+U 1 1 59C50BD8
+P 7425 3675
+F 0 "#PWR025" H 7425 3425 50  0001 C CNN
+F 1 "GND" H 7425 3525 50  0000 C CNN
+F 2 "" H 7425 3675 50  0000 C CNN
+F 3 "" H 7425 3675 50  0000 C CNN
+	1    7425 3675
 	1    0    0    -1
 $EndComp
-Text GLabel 7900 3100 1    60   Input ~ 0
-SDA
-Text GLabel 7900 3400 3    60   Input ~ 0
-SCL
-$Comp
-L GND #PWR030
-U 1 1 59C50BD8
-P 7150 3400
-F 0 "#PWR030" H 7150 3150 50  0001 C CNN
-F 1 "GND" H 7150 3250 50  0000 C CNN
-F 2 "" H 7150 3400 50  0000 C CNN
-F 3 "" H 7150 3400 50  0000 C CNN
-	1    7150 3400
-	1    0    0    -1
-$EndComp
-Text GLabel 6700 3150 0    60   Input ~ 0
+Text GLabel 7100 3525 0    60   Input ~ 0
 VCC_I2C
 $Comp
 L C_0.1uF C10
 U 1 1 59C50BDA
-P 6850 3350
-F 0 "C10" H 6875 3450 50  0000 L CNN
-F 1 "C_0.1uF" H 6550 3250 50  0000 L CNN
-F 2 "Capacitors_SMD:C_0603_HandSoldering" H 6950 3650 50  0001 C CNN
-F 3 "https://www.digikey.com/product-detail/en/kemet/C0603C104K5RACTU/399-5089-1-ND/1465623" H 6850 3100 50  0001 C CNN
-F 4 "C0603C104K5RACTU" H 6975 3550 60  0001 C CNN "Part Number"
-	1    6850 3350
+P 7200 3700
+F 0 "C10" H 7225 3800 50  0000 L CNN
+F 1 "C_0.1uF" H 6900 3600 50  0000 L CNN
+F 2 "Capacitors_SMD:C_0603_HandSoldering" H 7300 4000 50  0001 C CNN
+F 3 "https://www.digikey.com/product-detail/en/kemet/C0603C104K5RACTU/399-5089-1-ND/1465623" H 7200 3450 50  0001 C CNN
+F 4 "C0603C104K5RACTU" H 7325 3900 60  0001 C CNN "Part Number"
+	1    7200 3700
 	1    0    0    -1
 $EndComp
+Text Label 4050 3200 0    60   ~ 0
+Temp-Humidty
+Wire Wire Line
+	3400 3425 3900 3425
+Wire Wire Line
+	3900 3525 3850 3525
+Wire Wire Line
+	4850 3525 4750 3525
+Wire Wire Line
+	4750 3425 4850 3425
+Wire Wire Line
+	3550 3475 3550 3425
+Connection ~ 3550 3425
+Wire Wire Line
+	3550 3825 3550 3775
+Wire Wire Line
+	3850 3525 3850 3575
+Wire Wire Line
+	7425 3675 7425 3625
+Wire Wire Line
+	7425 3625 7475 3625
+Wire Wire Line
+	7100 3525 7475 3525
+Wire Wire Line
+	7200 3525 7200 3550
 $Comp
-L GND #PWR031
-U 1 1 59C50BDB
-P 6850 3550
-F 0 "#PWR031" H 6850 3300 50  0001 C CNN
-F 1 "GND" H 6850 3400 50  0000 C CNN
-F 2 "" H 6850 3550 50  0000 C CNN
-F 3 "" H 6850 3550 50  0000 C CNN
-	1    6850 3550
+L GND #PWR026
+U 1 1 59E2A131
+P 7200 3900
+F 0 "#PWR026" H 7200 3650 50  0001 C CNN
+F 1 "GND" H 7200 3750 50  0000 C CNN
+F 2 "" H 7200 3900 50  0000 C CNN
+F 3 "" H 7200 3900 50  0000 C CNN
+	1    7200 3900
 	1    0    0    -1
 $EndComp
-Text GLabel 8350 2800 1    60   Input ~ 0
-3V3
-Text Label 3500 2900 0    60   ~ 0
-Temp-Humidty
 Wire Wire Line
-	3050 3200 3550 3200
+	7200 3900 7200 3850
+Connection ~ 7200 3525
 Wire Wire Line
-	3550 3300 3500 3300
+	8425 3625 8325 3625
 Wire Wire Line
-	4500 3300 4400 3300
+	8325 3525 8375 3525
 Wire Wire Line
-	4400 3200 4500 3200
+	8375 3525 8375 3500
 Wire Wire Line
-	3200 3250 3200 3200
-Connection ~ 3200 3200
-Wire Wire Line
-	3200 3600 3200 3550
-Wire Wire Line
-	3500 3300 3500 3350
-Wire Wire Line
-	7900 3100 7900 3150
-Wire Wire Line
-	7900 3150 7850 3150
-Wire Wire Line
-	7900 3400 7900 3350
-Wire Wire Line
-	7900 3350 7850 3350
-Wire Wire Line
-	7150 3250 7150 3400
-Wire Wire Line
-	7150 3350 7200 3350
-Wire Wire Line
-	7200 3250 7150 3250
-Connection ~ 7150 3350
-Wire Wire Line
-	7850 3250 8500 3250
-Wire Wire Line
-	6700 3150 7200 3150
-Wire Wire Line
-	6850 3200 6850 3150
-Connection ~ 6850 3150
-Wire Wire Line
-	6850 3550 6850 3500
-Wire Wire Line
-	8350 2850 8350 2800
-Text GLabel 8500 3250 2    60   Input ~ 0
-LIGHT_INT
-Wire Wire Line
-	8350 3150 8350 3250
-Connection ~ 8350 3250
+	8375 3500 8425 3500
 $Comp
-L R_10k R7
-U 1 1 59C50BD9
-P 8350 3000
-F 0 "R7" V 8350 3000 50  0000 C CNN
-F 1 "R_10k" V 8250 3000 50  0000 C CNN
-F 2 "Resistors_SMD:R_0603_HandSoldering" V 8280 3000 50  0001 C CNN
-F 3 "https://www.digikey.com/product-detail/en/yageo/RC0603JR-0710KL/311-10KGRCT-ND/729647" V 8430 3000 50  0001 C CNN
-F 4 "RC0603JR-0710KL" V 8530 3100 60  0001 C CNN "Part Number"
-	1    8350 3000
-	-1   0    0    1
+L TSL45315CL U2
+U 1 1 59E41F23
+P 7925 3625
+F 0 "U2" H 8125 3525 60  0000 C CNN
+F 1 "TSL45315CL" H 7925 3825 60  0000 C CNN
+F 2 "open-automation:LIGHT-SENSOR-TSL45315CL" H 7925 3325 60  0001 C CNN
+F 3 "https://www.digikey.com/product-detail/en/ams/TSL45315CL/TSL45315-CLCT-ND/3095326" H 7925 3425 60  0001 C CNN
+F 4 "TSL45315CL" H 7925 3225 60  0001 C CNN "Part Number"
+	1    7925 3625
+	1    0    0    -1
 $EndComp
 $EndSCHEMATC

Commit message: update
Connections:
- net VCC_I2C renamed 3V3
Changed lines of the file:
@@
 Environment
 Text GLabel 3400 3425 0    60   Input ~ 0
-VCC_I2C
+3V3
 $Comp
 L GND #PWR023
@@
 $EndComp
 Text GLabel 7100 3525 0    60   Input ~ 0
-VCC_I2C
+3V3
 $Comp
 L C_0.1uF C10

Commit message: regulator ya know
Parts:
- C10, C9: footprint Capacitors_SMD:C_0603_HandSoldering -> Capacitor_SMD:C_0603_1608Metric_Pad0.99x1.00mm_HandSolder; symbol C_0.1uF -> open-automation:C_0.1uF; Part Number C0603C104K5RACTU -> CC0603MRY5V8BB104
- U2: symbol TSL45315CL -> open-automation:TSL45315CL
- U6: symbol SI7020-A20 -> open-automation:SI7020-A20
Changed lines of the file:
@@
-EESchema Schematic File Version 2
-LIBS:power
-LIBS:device
-LIBS:transistors
-LIBS:conn
-LIBS:linear
-LIBS:regul
-LIBS:74xx
-LIBS:cmos4000
-LIBS:adc-dac
-LIBS:memory
-LIBS:xilinx
-LIBS:microcontrollers
-LIBS:dsp
-LIBS:microchip
-LIBS:analog_switches
-LIBS:motorola
-LIBS:texas
-LIBS:intel
-LIBS:audio
-LIBS:interface
-LIBS:digital-audio
-LIBS:philips
-LIBS:display
-LIBS:cypress
-LIBS:siliconi
-LIBS:opto
-LIBS:atmel
-LIBS:contrib
-LIBS:valves
-LIBS:open-automation
+EESchema Schematic File Version 4
 LIBS:smart-regulator-cache
-EELAYER 25 0
+EELAYER 26 0
 EELAYER END
 $Descr A4 11693 8268
@@
 3V3
 $Comp
-L GND #PWR023
-U 1 1 59C50BD3
-P 3850 3575
-F 0 "#PWR023" H 3850 3325 50  0001 C CNN
-F 1 "GND" H 3850 3425 50  0000 C CNN
-F 2 "" H 3850 3575 50  0000 C CNN
-F 3 "" H 3850 3575 50  0000 C CNN
-	1    3850 3575
-	1    0    0    -1
-$EndComp
-Text GLabel 4850 3425 2    60   Input ~ 0
-SCL
-Text GLabel 4850 3525 2    60   Input ~ 0
-SDA
-$Comp
-L SI7020-A20 U6
+L open-automation:SI7020-A20 U6
 U 1 1 59C50BD4
 P 4350 3525
@@
 $EndComp
 $Comp
-L C_0.1uF C9
+L open-automation:C_0.1uF C9
 U 1 1 59C50BD5
 P 3550 3625
 F 0 "C9" H 3575 3725 50  0000 L CNN
 F 1 "C_0.1uF" H 3250 3525 50  0000 L CNN
-F 2 "Capacitors_SMD:C_0603_HandSoldering" H 3650 3925 50  0001 C CNN
+F 2 "Capacitor_SMD:C_0603_1608Metric_Pad0.99x1.00mm_HandSolder" H 3650 3925 50  0001 C CNN
 F 3 "https://www.digikey.com/product-detail/en/kemet/C0603C104K5RACTU/399-5089-1-ND/1465623" H 3550 3375 50  0001 C CNN
-F 4 "C0603C104K5RACTU" H 3675 3825 60  0001 C CNN "Part Number"
+F 4 "CC0603MRY5V8BB104" H 3675 3825 60  0001 C CNN "Part Number"
 	1    3550 3625
-	1    0    0    -1
-$EndComp
-$Comp
-L GND #PWR024
-U 1 1 59C50BD6
-P 3550 3825
-F 0 "#PWR024" H 3550 3575 50  0001 C CNN
-F 1 "GND" H 3550 3675 50  0000 C CNN
-F 2 "" H 3550 3825 50  0000 C CNN
-F 3 "" H 3550 3825 50  0000 C CNN
-	1    3550 3825
 	1    0    0    -1
 $EndComp
 Text Label 7675 3250 0    60   ~ 0
 Light-Level
-Text GLabel 8425 3625 2    60   Input ~ 0
-SDA
-Text GLabel 8425 3500 2    60   Input ~ 0
-SCL
-$Comp
-L GND #PWR025
-U 1 1 59C50BD8
-P 7425 3675
-F 0 "#PWR025" H 7425 3425 50  0001 C CNN
-F 1 "GND" H 7425 3525 50  0000 C CNN
-F 2 "" H 7425 3675 50  0000 C CNN
-F 3 "" H 7425 3675 50  0000 C CNN
-	1    7425 3675
-	1    0    0    -1
-$EndComp
 Text GLabel 7100 3525 0    60   Input ~ 0
 3V3
 $Comp
-L C_0.1uF C10
+L open-automation:C_0.1uF C10
 U 1 1 59C50BDA
 P 7200 3700
 F 0 "C10" H 7225 3800 50  0000 L CNN
 F 1 "C_0.1uF" H 6900 3600 50  0000 L CNN
-F 2 "Capacitors_SMD:C_0603_HandSoldering" H 7300 4000 50  0001 C CNN
+F 2 "Capacitor_SMD:C_0603_1608Metric_Pad0.99x1.00mm_HandSolder" H 7300 4000 50  0001 C CNN
 F 3 "https://www.digikey.com/product-detail/en/kemet/C0603C104K5RACTU/399-5089-1-ND/1465623" H 7200 3450 50  0001 C CNN
-F 4 "C0603C104K5RACTU" H 7325 3900 60  0001 C CNN "Part Number"
+F 4 "CC0603MRY5V8BB104" H 7325 3900 60  0001 C CNN "Part Number"
 	1    7200 3700
 	1    0    0    -1
@@
 Temp-Humidty
 Wire Wire Line
-	3400 3425 3900 3425
+	3400 3425 3550 3425
 Wire Wire Line
 	3900 3525 3850 3525
@@
 	7425 3625 7475 3625
 Wire Wire Line
-	7100 3525 7475 3525
+	7100 3525 7200 3525
 Wire Wire Line
 	7200 3525 7200 3550
-$Comp
-L GND #PWR026
-U 1 1 59E2A131
-P 7200 3900
-F 0 "#PWR026" H 7200 3650 50  0001 C CNN
-F 1 "GND" H 7200 3750 50  0000 C CNN
-F 2 "" H 7200 3900 50  0000 C CNN
-F 3 "" H 7200 3900 50  0000 C CNN
-	1    7200 3900
-	1    0    0    -1
-$EndComp
 Wire Wire Line
 	7200 3900 7200 3850
@@
 	8375 3500 8425 3500
 $Comp
-L TSL45315CL U2
+L open-automation:TSL45315CL U2
 U 1 1 59E41F23
 P 7925 3625
@@
 	1    0    0    -1
 $EndComp
+Wire Wire Line
+	3550 3425 3900 3425
+Wire Wire Line
+	7200 3525 7475 3525
+$Comp
+L open-automation:GND #PWR?
+U 1 1 5B3C6280
+P 3550 3825
+F 0 "#PWR?" H 3550 3575 50  0001 C CNN
+F 1 "GND" H 3555 3652 50  0000 C CNN
+F 2 "" H 3550 3825 50  0000 C CNN
+F 3 "" H 3550 3825 50  0000 C CNN
+	1    3550 3825
+	1    0    0    -1
+$EndComp
+$Comp
+L open-automation:GND #PWR?
+U 1 1 5B3C63A0
+P 3850 3575
+F 0 "#PWR?" H 3850 3325 50  0001 C CNN
+F 1 "GND" H 3855 3402 50  0000 C CNN
+F 2 "" H 3850 3575 50  0000 C CNN
+F 3 "" H 3850 3575 50  0000 C CNN
+	1    3850 3575
+	1    0    0    -1
+$EndComp
+$Comp
+L open-automation:GND #PWR?
+U 1 1 5B3C6890
+P 7425 3675
+F 0 "#PWR?" H 7425 3425 50  0001 C CNN
+F 1 "GND" H 7430 3502 50  0000 C CNN
+F 2 "" H 7425 3675 50  0000 C CNN
+F 3 "" H 7425 3675 50  0000 C CNN
+	1    7425 3675
+	1    0    0    -1
+$EndComp
+$Comp
+L open-automation:GND #PWR?
+U 1 1 5B3C69B5
+P 7200 3900
+F 0 "#PWR?" H 7200 3650 50  0001 C CNN
+F 1 "GND" H 7205 3727 50  0000 C CNN
+F 2 "" H 7200 3900 50  0000 C CNN
+F 3 "" H 7200 3900 50  0000 C CNN
+	1    7200 3900
+	1    0    0    -1
+$EndComp
+Text HLabel 4850 3425 2    50   Input ~ 0
+SCL
+Text HLabel 4850 3525 2    50   Input ~ 0
+SDA
+Text HLabel 8425 3500 2    50   Input ~ 0
+SCL
+Text HLabel 8425 3625 2    50   Input ~ 0
+SDA
 $EndSCHEMATC

Commit message: additional components
Other:
- note added: "ENVIRONMENT"
Changed lines of the file:
@@
 Text HLabel 8425 3625 2    50   Input ~ 0
 SDA
+Text Notes 7050 6900 0    197  ~ 0
+ENVIRONMENT
 $EndSCHEMATC

Commit message: layout complete bitches
Parts:
- C14: renamed from C9; footprint Capacitor_SMD:C_0603_1608Metric_Pad0.99x1.00mm_HandSolder -> Capacitor_SMD:C_0603_1608Metric_Pad1.05x0.95mm_HandSolder
- C15: renamed from C10; footprint Capacitor_SMD:C_0603_1608Metric_Pad0.99x1.00mm_HandSolder -> Capacitor_SMD:C_0603_1608Metric_Pad1.05x0.95mm_HandSolder
- U14: renamed from U6; value SI7020-A20 -> SI7006-A20; Part Number SI7020-A20-GM1R -> SI7006-A20-IM
- renumbered U2 to U15
Changed lines of the file:
@@
 3V3
 $Comp
-L open-automation:SI7020-A20 U6
+L open-automation:SI7020-A20 U14
 U 1 1 59C50BD4
 P 4350 3525
-F 0 "U6" H 4550 3425 60  0000 C CNN
-F 1 "SI7020-A20" H 4350 3725 60  0000 C CNN
+F 0 "U14" H 4550 3425 60  0000 C CNN
+F 1 "SI7006-A20" H 4350 3725 60  0000 C CNN
 F 2 "open-automation:SI7020-A20" H 4350 3225 60  0001 C CNN
-F 3 "https://www.digikey.com/product-detail/en/silicon-labs/SI7020-A20-GM1R/336-3596-1-ND/5823452" H 4350 3325 60  0001 C CNN
-F 4 "SI7020-A20-GM1R" H 4450 3325 60  0001 C CNN "Part Number"
+F 3 "https://www.digikey.com/product-detail/en/silicon-labs/SI7006-A20-IM/336-3124-ND/5050329" H 4350 3325 60  0001 C CNN
+F 4 "SI7006-A20-IM" H 4450 3325 60  0001 C CNN "Part Number"
 	1    4350 3525
 	1    0    0    -1
 $EndComp
 $Comp
-L open-automation:C_0.1uF C9
+L open-automation:C_0.1uF C14
 U 1 1 59C50BD5
 P 3550 3625
-F 0 "C9" H 3575 3725 50  0000 L CNN
+F 0 "C14" H 3575 3725 50  0000 L CNN
 F 1 "C_0.1uF" H 3250 3525 50  0000 L CNN
-F 2 "Capacitor_SMD:C_0603_1608Metric_Pad0.99x1.00mm_HandSolder" H 3650 3925 50  0001 C CNN
+F 2 "Capacitor_SMD:C_0603_1608Metric_Pad1.05x0.95mm_HandSolder" H 3650 3925 50  0001 C CNN
 F 3 "https://www.digikey.com/product-detail/en/kemet/C0603C104K5RACTU/399-5089-1-ND/1465623" H 3550 3375 50  0001 C CNN
 F 4 "CC0603MRY5V8BB104" H 3675 3825 60  0001 C CNN "Part Number"
@@
 3V3
 $Comp
-L open-automation:C_0.1uF C10
+L open-automation:C_0.1uF C15
 U 1 1 59C50BDA
 P 7200 3700
-F 0 "C10" H 7225 3800 50  0000 L CNN
+F 0 "C15" H 7225 3800 50  0000 L CNN
 F 1 "C_0.1uF" H 6900 3600 50  0000 L CNN
-F 2 "Capacitor_SMD:C_0603_1608Metric_Pad0.99x1.00mm_HandSolder" H 7300 4000 50  0001 C CNN
+F 2 "Capacitor_SMD:C_0603_1608Metric_Pad1.05x0.95mm_HandSolder" H 7300 4000 50  0001 C CNN
 F 3 "https://www.digikey.com/product-detail/en/kemet/C0603C104K5RACTU/399-5089-1-ND/1465623" H 7200 3450 50  0001 C CNN
 F 4 "CC0603MRY5V8BB104" H 7325 3900 60  0001 C CNN "Part Number"
@@
 	8375 3500 8425 3500
 $Comp
-L open-automation:TSL45315CL U2
+L open-automation:TSL45315CL U15
 U 1 1 59E41F23
 P 7925 3625
-F 0 "U2" H 8125 3525 60  0000 C CNN
+F 0 "U15" H 8125 3525 60  0000 C CNN
 F 1 "TSL45315CL" H 7925 3825 60  0000 C CNN
 F 2 "open-automation:LIGHT-SENSOR-TSL45315CL" H 7925 3325 60  0001 C CNN
@@
 	7200 3525 7475 3525
 $Comp
-L open-automation:GND #PWR?
+L open-automation:GND #PWR045
 U 1 1 5B3C6280
 P 3550 3825
-F 0 "#PWR?" H 3550 3575 50  0001 C CNN
+F 0 "#PWR045" H 3550 3575 50  0001 C CNN
 F 1 "GND" H 3555 3652 50  0000 C CNN
 F 2 "" H 3550 3825 50  0000 C CNN
@@
 $EndComp
 $Comp
-L open-automation:GND #PWR?
+L open-automation:GND #PWR046
 U 1 1 5B3C63A0
 P 3850 3575
-F 0 "#PWR?" H 3850 3325 50  0001 C CNN
+F 0 "#PWR046" H 3850 3325 50  0001 C CNN
 F 1 "GND" H 3855 3402 50  0000 C CNN
 F 2 "" H 3850 3575 50  0000 C CNN
@@
 $EndComp
 $Comp
-L open-automation:GND #PWR?
+L open-automation:GND #PWR048
 U 1 1 5B3C6890
 P 7425 3675
-F 0 "#PWR?" H 7425 3425 50  0001 C CNN
+F 0 "#PWR048" H 7425 3425 50  0001 C CNN
 F 1 "GND" H 7430 3502 50  0000 C CNN
 F 2 "" H 7425 3675 50  0000 C CNN
@@
 $EndComp
 $Comp
-L open-automation:GND #PWR?
+L open-automation:GND #PWR047
 U 1 1 5B3C69B5
 P 7200 3900
-F 0 "#PWR?" H 7200 3650 50  0001 C CNN
+F 0 "#PWR047" H 7200 3650 50  0001 C CNN
 F 1 "GND" H 7205 3727 50  0000 C CNN
 F 2 "" H 7200 3900 50  0000 C CNN

Commit message: multifile update
Parts:
- C14, C15: Part Number CC0603MRY5V8BB104 -> CC0603ZRY5V9BB104
Changed lines of the file:
@@
 F 2 "Capacitor_SMD:C_0603_1608Metric_Pad1.05x0.95mm_HandSolder" H 3650 3925 50  0001 C CNN
 F 3 "https://www.digikey.com/product-detail/en/kemet/C0603C104K5RACTU/399-5089-1-ND/1465623" H 3550 3375 50  0001 C CNN
-F 4 "CC0603MRY5V8BB104" H 3675 3825 60  0001 C CNN "Part Number"
+F 4 "CC0603ZRY5V9BB104" H 3675 3825 60  0001 C CNN "Part Number"
 	1    3550 3625
 	1    0    0    -1
@@
 F 2 "Capacitor_SMD:C_0603_1608Metric_Pad1.05x0.95mm_HandSolder" H 7300 4000 50  0001 C CNN
 F 3 "https://www.digikey.com/product-detail/en/kemet/C0603C104K5RACTU/399-5089-1-ND/1465623" H 7200 3450 50  0001 C CNN
-F 4 "CC0603MRY5V8BB104" H 7325 3900 60  0001 C CNN "Part Number"
+F 4 "CC0603ZRY5V9BB104" H 7325 3900 60  0001 C CNN "Part Number"
 	1    7200 3700
 	1    0    0    -1

Commit message: parts
Parts:
- C14, C15: Part Number CC0603ZRY5V9BB104 -> GCM188R71C104KA37D
Changed lines of the file:
@@
 F 1 "C_0.1uF" H 3250 3525 50  0000 L CNN
 F 2 "Capacitor_SMD:C_0603_1608Metric_Pad1.05x0.95mm_HandSolder" H 3650 3925 50  0001 C CNN
-F 3 "https://www.digikey.com/product-detail/en/kemet/C0603C104K5RACTU/399-5089-1-ND/1465623" H 3550 3375 50  0001 C CNN
-F 4 "CC0603ZRY5V9BB104" H 3675 3825 60  0001 C CNN "Part Number"
+F 3 "https://www.digikey.com/product-detail/en/murata-electronics-north-america/GCM188R71C104KA37D/490-4774-1-ND/1641693" H 3550 3375 50  0001 C CNN
+F 4 "GCM188R71C104KA37D" H 3675 3825 60  0001 C CNN "Part Number"
 	1    3550 3625
 	1    0    0    -1
@@
 F 1 "C_0.1uF" H 6900 3600 50  0000 L CNN
 F 2 "Capacitor_SMD:C_0603_1608Metric_Pad1.05x0.95mm_HandSolder" H 7300 4000 50  0001 C CNN
-F 3 "https://www.digikey.com/product-detail/en/kemet/C0603C104K5RACTU/399-5089-1-ND/1465623" H 7200 3450 50  0001 C CNN
-F 4 "CC0603ZRY5V9BB104" H 7325 3900 60  0001 C CNN "Part Number"
+F 3 "https://www.digikey.com/product-detail/en/murata-electronics-north-america/GCM188R71C104KA37D/490-4774-1-ND/1641693" H 7200 3450 50  0001 C CNN
+F 4 "GCM188R71C104KA37D" H 7325 3900 60  0001 C CNN "Part Number"
 	1    7200 3700
 	1    0    0    -1
